Commit message: fixed small bugs in track displacement changed wheelbase to 1.2m as is on the real car

File: eufs_description/urdf/wheels/suspension_wheel.urdf.xacro (robot description, xacro)
@@ -15,5 +15,5 @@
        from a U joint to the corresponding hex hub. wheel_travel is the
        vertical wheel travel. -->
-  <xacro:property name="wheelbase" value="1.55"/>
+  <xacro:property name="wheelbase" value="1.2"/>
   <xacro:property name="hex_hub_dist" value="1.360"/>  <!-- track/width of the car -->
   <xacro:property name="axle_length" value="0.120"/>

Commit message: fixed wheelbase and track of the sim model

File: eufs_description/urdf/wheels/suspension_wheel.urdf.xacro (robot description, xacro)
@@ -1,4 +1,16 @@
 <?xml version="1.0"?>
 <robot name="wheel" xmlns:xacro="http://www.ros.org/wiki/xacro">
+<!--
+ADS-DV Specifications as given by IMechE:
+WHEELBASE         :1530mm
+FRONT TRACK       :1201mm
+REAR TRACK        :1201mm
+OVERALL WIDTH     :1430mm
+OVERALL LENGTH    :2814.6mm
+STATIC CASTER     :6 deg
+STATIC CAMBER     :2 deg
+TYRES             : SAE FORMULA STUDENT AVON 7.2/20.0-13
+DRIVEN WHEELS     :4WD
+DIFFERENTIALS     :OPEN DIFF -->
   <!-- hub_dia and tire_dia are the diameters of the hub and tire,
        respectively. hex_hub_depth is the distance that the hex hub is
@@ -15,6 +27,6 @@
        from a U joint to the corresponding hex hub. wheel_travel is the
        vertical wheel travel. -->
-  <xacro:property name="wheelbase" value="1.2"/>
-  <xacro:property name="hex_hub_dist" value="1.360"/>  <!-- track/width of the car -->
+  <xacro:property name="wheelbase" value="1.530"/>
+  <xacro:property name="hex_hub_dist" value="1.201"/>  <!-- track/width of the car -->
   <xacro:property name="axle_length" value="0.120"/>
   <xacro:property name="wheel_travel" value="0.05"/>
