Commit message: carryover to robot model changes from common

File: eufs_description/robots/eufs.urdf.xacro (robot description, xacro)
@@ -19,12 +19,9 @@
     <xacro:property name="wheel_offset_y" value="0.75" />
     <xacro:property name="wheel_offset_z" value="0.0" />
-    <!-- Flag to select the high or low quality model -->
-    <xacro:property name="hq" value="true" />
     <!-- *************** -->
     <!-- Robots Elements -->
     <!-- *************** -->
-    <!-- Here we create the robot elements using the xacro:macros imported at the beggining of this file -->
-    <!-- Summit XL base -->
-    <xacro:eufs_base name="eufs" publish_bf="true" hq="${hq}" />
+    <!-- Chassis of the car -->
+    <xacro:eufs_base name="eufs" publish_bf="true" hq="false" clearance="0.25"/>
     <!-- Gazebo ros control pluggins -->
     <xacro:ros_control/>
