Commit message: remove base_link

File: eufs_description/robots/ads-dv.urdf.xacro (robot description, xacro)
@@ -47,8 +47,8 @@
     LIDAR: 1.700 0.0 -0.150
     STEREO CAM: -0.110 0.0 0.800 -->
-    <xacro:sensor_imu parent="base_link" prefix="imu">
+    <xacro:sensor_imu parent="base_footprint" prefix="imu">
         <origin xyz="-0.0 0.0 0.0" rpy="0 0 0"/>
     </xacro:sensor_imu>
-    <xacro:sensor_gps  parent="base_link" prefix="gps">
+    <xacro:sensor_gps  parent="base_footprint" prefix="gps">
         <origin xyz="0.0 0.0 0.4" rpy="0 0 0"/>
     </xacro:sensor_gps>
@@ -59,8 +59,8 @@
         <origin xyz="1.700 0.0 -0.150" rpy="0 -0.0174533 0"/>
     </xacro:VLP-16> -->
-    <xacro:VLP-16R  parent="base_link" name="velodyne" topic="/velodyne_points" hz="10" samples="800">
+    <xacro:VLP-16R  parent="base_footprint" name="velodyne" topic="/velodyne_points" hz="10" samples="800">
         <origin xyz="1.58 0.0 -0.1" rpy="0 ${1*M_PI/180.0} 0"/>
     </xacro:VLP-16R>
-    <xacro:zed_camera parent="base_link" prefix="zed">
+    <xacro:zed_camera parent="base_footprint" prefix="zed">
         <origin xyz="0.1 0.0 0.52" rpy="0 0 0"/>
     </xacro:zed_camera>

File: eufs_description/sensors/VLP-16.urdf.xacro (robot description, xacro)
@@ -2,5 +2,5 @@
 <robot xmlns:xacro="http://www.ros.org/wiki/xacro" name="VLP-16">
   <xacro:property name="M_PI" value="3.1415926535897931" />
-  <xacro:macro name="VLP-16" params="*origin parent:=base_link name:=velodyne topic:=/velodyne_points hz:=10 lasers:=16 samples:=1875 collision_range:=0.3 min_range:=0.9 max_range:=130.0 noise:=0.008 min_angle:=-${M_PI} max_angle:=${M_PI}">
+  <xacro:macro name="VLP-16" params="*origin parent:=base_footprint name:=velodyne topic:=/velodyne_points hz:=10 lasers:=16 samples:=1875 collision_range:=0.3 min_range:=0.9 max_range:=130.0 noise:=0.008 min_angle:=-${M_PI} max_angle:=${M_PI}">
     <joint name="${name}_base_mount_joint" type="fixed">
       <xacro:insert_block name="origin" />

File: eufs_description/sensors/VLP-16R.urdf.xacro (robot description, xacro)
@@ -2,5 +2,5 @@
 <robot xmlns:xacro="http://www.ros.org/wiki/xacro" name="VLP-16">
   <xacro:property name="M_PI" value="3.1415926535897931" />
-  <xacro:macro name="VLP-16R" params="*origin parent:=base_link name:=velodyne topic:=/velodyne_points hz:=6 lasers:=5 samples:=1200 collision_range:=0.3 min_range:=0.6 max_range:=130.0 noise:=0.008 min_angle:=-2 max_angle:=2">
+  <xacro:macro name="VLP-16R" params="*origin parent:=base_footprint name:=velodyne topic:=/velodyne_points hz:=6 lasers:=5 samples:=1200 collision_range:=0.3 min_range:=0.6 max_range:=130.0 noise:=0.008 min_angle:=-2 max_angle:=2">
     <joint name="${name}_base_mount_joint" type="fixed">
       <xacro:insert_block name="origin" />

File: eufs_description/urdf/ads-dv_base.urdf.xacro (robot description, xacro)
@@ -12,48 +12,37 @@
     <link name="base_footprint">
       <visual>
-          <origin xyz="0 0 0" rpy="0 0 0" />
+        <origin xyz="0 0 ${clearance}" rpy="0 0 0" />  <!-- height is the clearance -->
+        <geometry>
+          <box size="0.001 0.001 0.001" />
+        </geometry>
+        <xacro:if value="${hq}">
           <geometry>
-             <box size="0.001 0.001 0.001" />
+    	      <mesh filename="package://eufs_description/meshes/ads-dv.dae"/>
           </geometry>
+        </xacro:if>
+        <xacro:unless value="${hq}">
+          <geometry>
+    	      <mesh filename="package://eufs_description/meshes/ads-dv.dae"/>
+          </geometry>
+        </xacro:unless>
       </visual>
+      <inertial>
+        <mass value="125.0" />
+        <origin xyz="0 0 0" />
+        <inertia  ixx="16.3"
+                  ixy="0.004"
+                  ixz="0.0"
+                  iyy="33.6"
+                  iyz="0.0"
+                  izz="47.9" />
+      </inertial>
+      <collision>
+        <origin xyz="0 0 0" rpy="0 0 0" />  <!-- might have to adjest height to the clearance -->
+        <geometry>
+          <mesh filename="package://eufs_description/meshes/ads-dv.dae"/>
+        </geometry>
+      </collision>
     </link>
-    <joint name="base_footprint_joint" type="fixed">
-      <origin xyz="0 0 ${clearance}" rpy="0 0 0" />  <!-- height is the clearance -->
-      <parent link="base_footprint"/>
-      <child link="base_link" />
-    </joint>
   </xacro:if>
-  <!-- BASE_LINK -->
-  <link name="base_link">
-    <inertial>
-      <mass value="125.0" />
-      <origin xyz="0 0 0" />
-      <inertia  ixx="16.3"
-                ixy="0.004"
-                ixz="0.0"
-                iyy="33.6"
-                iyz="0.0"
-                izz="47.9" />
-    </inertial>
-    <visual>
-       <origin xyz="0 0 0" rpy="0 0 0" />
-       <xacro:if value="${hq}">
-       <geometry>
-	     <mesh filename="package://eufs_description/meshes/ads-dv.dae"/>
-       </geometry>
-       </xacro:if>
-       <xacro:unless value="${hq}">
-       <geometry>
-	     <mesh filename="package://eufs_description/meshes/ads-dv.dae"/>
-       </geometry>
-       </xacro:unless>
-    </visual>
-    <collision>
-       <origin xyz="0 0 0" rpy="0 0 0 " />
-       <geometry>
-         <mesh filename="package://eufs_description/meshes/ads-dv.dae"/>
-       </geometry>
-    </collision>
-  </link>
   <link name="odom_ground_truth">
     <collision>
@@ -71,5 +60,5 @@
     <axis xyz="0 0 0" />
     <origin xyz="0 0 0" rpy="0 0 0"/>
-    <parent link="base_link"/>
+    <parent link="base_footprint"/>
     <child link="odom_ground_truth"/>
   </joint>

File: eufs_description/urdf/suspension_wheel.urdf.xacro (robot description, xacro)
@@ -85,5 +85,5 @@
                params="lr_prefix fr_prefix lr_reflect fr_reflect child">
     <joint name="${lr_prefix}_${fr_prefix}_shock" type="prismatic">
-      <parent link="base_link"/>
+      <parent link="base_footprint"/>
       <child link="${child}"/>
       <origin xyz="${fr_reflect * wheelbase / 2}

Commit message: update xacro to simulate raw perception sensors only when necessary

File: eufs_description/robots/ads-dv.urdf.xacro (robot description, xacro)
@@ -1,4 +1,5 @@
 <?xml version="1.0"?>
-<robot name="eufs" xmlns:xacro="http://www.ros.org/wiki/xacro">
+<robot name="eufs"
+    xmlns:xacro="http://www.ros.org/wiki/xacro">
     <!-- ***************** -->
     <!-- Imported elements -->
@@ -9,6 +10,6 @@
     <xacro:arg name="simulate_perception" default="false"/>
     <xacro:include filename="$(find eufs_description)/urdf/ads-dv_base.urdf.xacro">
-      <xacro:arg name="publish_tf" value="$(arg publish_tf)"/>
-      <xacro:arg name="simulate_perception" value="$(arg simulate_perception)"/>
+        <xacro:arg name="publish_tf" value="$(arg publish_tf)"/>
+        <xacro:arg name="simulate_perception" value="$(arg simulate_perception)"/>
     </xacro:include>
     <!-- Import Robotnik CAR wheels -->
@@ -21,5 +22,6 @@
     <xacro:property name="PI" value="3.1415926535897931"/>
     <!-- Wheel parameters -->
-    <xacro:property name="wheel_offset_x" value="1.0" />    <!-- x,y,z in translation from base_link to the center of the wheel -->
+    <xacro:property name="wheel_offset_x" value="1.0" />
+    <!-- x,y,z in translation from base_link to the center of the wheel -->
     <xacro:property name="wheel_offset_y" value="0.75" />
     <xacro:property name="wheel_offset_z" value="0.0" />
@@ -34,18 +36,13 @@
     <!-- Gazebo ros control pluggins -->
     <xacro:ros_control/>
-    <!-- Gazebo skid steering pluggins -->
-    <!-- xacro:skid_steering broadcastOdomTF="1"/ -->
     <!-- WHEELS -->
-    <!-- Wheels -->
-    <xacro:front_wheel lr_prefix="left" fr_prefix="front"
-        lr_reflect="1" fr_reflect="1"/>
-    <xacro:front_wheel lr_prefix="right" fr_prefix="front"
-        lr_reflect="-1" fr_reflect="1"/>
-    <xacro:rear_wheel lr_prefix="left" fr_prefix="rear"
-        lr_reflect="1" fr_reflect="-1"/>
-    <xacro:rear_wheel lr_prefix="right" fr_prefix="rear"
-        lr_reflect="-1" fr_reflect="-1"/>
-    <!-- MAIN SENSORS -->
-<!--     LOCATIONS: (XYZ)
+    <xacro:front_wheel lr_prefix="left" fr_prefix="front" lr_reflect="1" fr_reflect="1"/>
+    <xacro:front_wheel lr_prefix="right" fr_prefix="front" lr_reflect="-1" fr_reflect="1"/>
+    <xacro:rear_wheel lr_prefix="left" fr_prefix="rear" lr_reflect="1" fr_reflect="-1"/>
+    <xacro:rear_wheel lr_prefix="right" fr_prefix="rear" lr_reflect="-1" fr_reflect="-1"/>
+    <!-- *********************************************** -->
+    <!--                 MAIN SENSORS                    -->
+    <!-- *********************************************** -->
+    <!--     LOCATIONS: (XYZ)
     IMU: 0.0 0.0 0.170
     GPS: -0.110 0.0 0.9
@@ -55,21 +52,22 @@
         <origin xyz="-0.0 0.0 0.0" rpy="0 0 0"/>
     </xacro:sensor_imu>
-    <xacro:sensor_gps  parent="base_footprint" prefix="gps">
+    <xacro:sensor_gps parent="base_footprint" prefix="gps">
         <origin xyz="0.0 0.0 0.4" rpy="0 0 0"/>
     </xacro:sensor_gps>
-<!--     <xacro:sensor_hokuyo_utm30lx  parent="base_link" prefix="lidar" >
+    <!-- Simulate raw perception sensors only if we're not using the abstracted perception simulation -->
+    <xacro:unless value="$(arg simulate_perception)">
+        <xacro:VLP-16R parent="base_footprint" name="velodyne" topic="/velodyne_points" hz="10" samples="800">
+            <origin xyz="1.58 0.0 -0.1" rpy="0 ${1*M_PI/180.0} 0"/>
+        </xacro:VLP-16R>
+        <xacro:zed_camera parent="base_footprint" prefix="zed">
+            <origin xyz="0.1 0.0 0.52" rpy="0 0 0"/>
+        </xacro:zed_camera>
+    </xacro:unless>
+    <!-- *********************************************** -->
+    <!-- EXTRA SENSORS FROM THE ROBOTNIK SENSORS LIBRARY -->
+    <!-- *********************************************** -->
+    <!--     <xacro:sensor_hokuyo_utm30lx parent="base_link" prefix="lidar">
         <origin xyz="1.700 0.0 -0.080" rpy="0 -0.0174533 0"/>
-    </xacro:sensor_hokuyo_utm30lx> -->
-    <!-- <xacro:VLP-16  parent="base_link" name="velodyne" topic="/velodyne_points" hz="10">
-        <origin xyz="1.700 0.0 -0.150" rpy="0 -0.0174533 0"/>
-    </xacro:VLP-16> -->
-    <xacro:VLP-16R  parent="base_footprint" name="velodyne" topic="/velodyne_points" hz="10" samples="800">
-        <origin xyz="1.58 0.0 -0.1" rpy="0 ${1*M_PI/180.0} 0"/>
-    </xacro:VLP-16R>
-    <xacro:zed_camera parent="base_footprint" prefix="zed">
-        <origin xyz="0.1 0.0 0.52" rpy="0 0 0"/>
-    </xacro:zed_camera>
-    <!-- EXTRA SENSORS FROM THE ROBOTNIK SENSORS LIBRARY -->
-<!--
+    </xacro:sensor_hokuyo_utm30lx>
     <xacro:sensor_hokuyo3d name="hokuyo3d" parent="base_link">
         <origin xyz="0.9 0.0 0.450" rpy="0 0.35 0"/>
@@ -87,12 +85,7 @@
         <origin xyz="0.0 0.0 0.45" rpy="0 0 0"/>
     </xacro:sensor_kinect>
-    <xacro:BB2-08S2C-60  prefix="bee" frame="bee" name="bee"/>
+    <xacro:BB2-08S2C-60 prefix="bee" frame="bee" name="bee"/>
     <xacro:sensor_fotonic name="fotonic" parent="base_link">
         <origin xyz="0.3 0.0 0.24" rpy="0 0 0"/>
     </xacro:sensor_fotonic>   -->
-    <!-- PLUGINS -->
-    <!-- ros control plugin -->
-<!--   <gazebo>
-    <plugin name="gazebo_ros_control" filename="libgazebo_ros_control.so"/>
-</gazebo> -->
 </robot>
