Commit message: Added the vehicle model to the ads car. Wheels are a bit weird for some reason

File: eufs_description/robots/ads-dv.urdf.xacro (robot description, xacro)
@@ -1,4 +1,9 @@
 <?xml version="1.0"?>
 <robot name="eufs" xmlns:xacro="http://www.ros.org/wiki/xacro">
+    <xacro:property name="robot_sensors" value="${load_yaml('$(arg sensors_config_file)')}"/>
+    <xacro:property name="car_settings" value="${load_yaml('$(arg car_config_file)')}"/>
+    <xacro:property name="dist" value="${load_yaml('$(arg car_dimensions_file)')}"/>
+    <xacro:include filename="$(find eufs_description)/urdf/vehicle/inertias.xacro"/>
+    <xacro:include filename="$(find eufs_description)/urdf/vehicle/plugins.gazebo"/>
     <!-- ***************** -->
     <!-- Imported elements -->
@@ -7,6 +12,4 @@
     <!-- Import Robotnik CAR base elements -->
     <xacro:include filename="$(find eufs_description)/urdf/ads-dv_base.urdf.xacro" />
-    <!-- Import Robotnik CAR wheels -->
-    <xacro:include filename="$(find eufs_description)/urdf/suspension_wheel.urdf.xacro" />
     <!-- Import all available sensors -->
     <xacro:include filename="$(find eufs_description)/sensors/all_sensors.urdf.xacro" />
@@ -27,18 +30,198 @@
     <!-- Summit XL base -->
     <xacro:eufs_base name="eufs" publish_bf="true" hq="${hq}" />
-    <!-- Gazebo ros control pluggins -->
-    <xacro:ros_control/>
     <!-- Gazebo skid steering pluggins -->
     <!-- xacro:skid_steering broadcastOdomTF="1"/ -->
     <!-- WHEELS -->
+    <!-- hub_dia and tire_dia are the diameters of the hub and tire,
+     respectively. hex_hub_depth is the distance that the hex hub is
+     inset from the outer edge of the tire. It is set so that each wheel
+     is a "zero offset" wheel. hex_hub_depth = tire_width / 2 -
+     axle_length. -->
+    <xacro:property name="hub_dia" value="0.08"/>
+    <xacro:property name="tire_dia" value="0.505"/>
+    <xacro:property name="tire_width" value="0.2"/>
+    <xacro:property name="hex_hub_depth" value="0.120"/> <!-- or +0.072 -->
+    <xacro:property name="wheel_mass" value="10.0"/>   <!-- check -->
+    <!-- hex_hub_dist is the distance between left and right hex hubs when
+         the shock absorbers are fully extended. axle_length is the distance
+         from a U joint to the corresponding hex hub. wheel_travel is the
+         vertical wheel travel. -->
+    <xacro:property name="wheelbase" value="1.530"/>
+    <xacro:property name="hex_hub_dist" value="1.201"/>  <!-- track/width of the car -->
+    <xacro:property name="axle_length" value="0.120"/>
+    <xacro:property name="wheel_travel" value="0.05"/>
+    <xacro:property name="shock_z_offset" value="0.05"/>
+    <!-- Degree-to-radian conversions -->
+    <xacro:property name="degrees_45" value="0.785398163"/>
+    <xacro:property name="degrees_90" value="1.57079633"/>
+    <xacro:property name="degrees_180" value="3.14159265"/>
+    <!-- shock_eff_limit is 2 * ((shock_stroke / 2) * shock_spring_constant) N. -->
+    <xacro:property name="shock_eff_limit" value="50"/>
+    <xacro:property name="shock_vel_limit" value="500"/>
+    <xacro:property name="wheel_joint_damping" value="0.01" />
+    <xacro:property name="wheel_joint_friction" value="0.1" />
+    <xacro:property name="suspension_joint_damping" value="0.01" />
+    <xacro:property name="suspension_joint_friction" value="0.1" />
     <!-- Wheels -->
-    <xacro:front_wheel lr_prefix="left" fr_prefix="front"
-        lr_reflect="1" fr_reflect="1"/>
-    <xacro:front_wheel lr_prefix="right" fr_prefix="front"
-        lr_reflect="-1" fr_reflect="1"/>
-    <xacro:rear_wheel lr_prefix="left" fr_prefix="rear"
-        lr_reflect="1" fr_reflect="-1"/>
-    <xacro:rear_wheel lr_prefix="right" fr_prefix="rear"
-        lr_reflect="-1" fr_reflect="-1"/>
+    <xacro:macro name="body_left_rear_wheel">
+        <joint name="rear_left_wheel_joint" type="continuous">
+            <origin xyz="${-1 * wheelbase / 2}
+                         ${1 * ((hex_hub_dist / 2) - axle_length)}
+                         ${-wheel_travel}"
+                    rpy="0 0 0"/>
+            <parent link="base_footprint"/>
+            <child link="left_rear_wheel"/>
+            <axis xyz="0 1 0"/>
+        </joint>
+        <link name="left_rear_wheel">
+            <inertial>
+                <xacro:wheels_inertia/>
+            </inertial>
+            <visual>
+                <xacro:wheels_geometry/>
+                <material name="black"/>
+            </visual>
+            <collision name="left_rear_wheel_collision">
+                <geometry>
+                    <sphere radius="0.225"/>
+                </geometry>
+            </collision>
+        </link>
+        <gazebo reference="left_rear_wheel">
+            <material>Gazebo/Black</material>
+        </gazebo>
+    </xacro:macro>
+    <xacro:macro name="body_right_rear_wheel">
+        <joint name="rear_right_wheel_joint" type="continuous">
+            <parent link="base_footprint"/>
+            <child link="right_rear_wheel"/>
+            <origin xyz="${-1 * wheelbase / 2}
+                         ${-1 * ((hex_hub_dist / 2) - axle_length)}
+                         ${-wheel_travel}"
+                    rpy="0 0 0"/>
+            <axis xyz="0 1 0"/>
+        </joint>
+        <link name="right_rear_wheel">
+            <inertial>
+                <xacro:wheels_inertia/>
+            </inertial>
+            <visual>
+                <xacro:wheels_geometry/>
+                <material name="black"/>
+            </visual>
+            <collision name="right_rear_wheel_collision">
+                <geometry>
+                    <sphere radius="0.225"/>
+                </geometry>
+            </collision>
+        </link>
+        <gazebo reference="right_rear_wheel">
+            <material>Gazebo/Black</material>
+        </gazebo>
+    </xacro:macro>
+    <xacro:macro name="body_left_front_wheel">
+        <joint name="left_steering_hinge_joint" type="revolute">
+            <origin xyz="${1 * wheelbase / 2}
+                         ${1 * ((hex_hub_dist / 2) - axle_length)}
+                         ${-wheel_travel}"
+                    rpy="0 0 0"/>
+            <parent link="base_footprint"/>
+            <child link="left_steering_hinge"/>
+            <axis xyz="0 0 1"/>
+            <limit lower="-0.8727" upper="0.8727" effort="10000000" velocity="1000000"/>
+        </joint>
+        <link name="left_steering_hinge">
+            <inertial>
+                <xacro:steering_hinge_inertial_params/>
+            </inertial>
+            <visual>
+                <xacro:steering_hinge_geometry/>
+                <material name="black"/>
+            </visual>
+        </link>
+        <joint name="front_left_wheel_joint" type="continuous">
+            <origin xyz="0 0 0" rpy="0 0 0"/>
+            <parent link="left_steering_hinge"/>
+            <child link="left_front_wheel"/>
+            <axis xyz="0 1 0"/>
+        </joint>
+        <link name="left_front_wheel">
+            <inertial>
+                <xacro:wheels_inertia/>
+            </inertial>
+            <visual>
+                <xacro:wheels_geometry/>
+                <material name="black"/>
+            </visual>
+            <collision name="left_front_wheel_collision">
+                <geometry>
+                    <sphere radius="0.225"/>
+                </geometry>
+            </collision>
+        </link>
+        <gazebo reference="left_front_wheel">
+            <material>Gazebo/Black</material>
+        </gazebo>
+    </xacro:macro>
+    <xacro:macro name="body_right_front_wheel">
+        <joint name="right_steering_hinge_joint" type="revolute">
+            <parent link="base_footprint"/>
+            <child link="right_steering_hinge"/>
+            <axis xyz="0 0 1"/>
+            <origin xyz="${1 * wheelbase / 2}
+                         ${-1 * ((hex_hub_dist / 2) - axle_length)}
+                         ${-wheel_travel}"
+                    rpy="0 0 0"/>
+            <limit lower="-0.8727" upper="0.8727" effort="10000000" velocity="1000000"/>
+        </joint>
+        <link name="right_steering_hinge">
+            <inertial>
+                <xacro:steering_hinge_inertial_params/>
+            </inertial>
+            <visual>
+                <xacro:steering_hinge_geometry/>
+            </visual>
+        </link>
+        <joint name="front_right_wheel_joint" type="continuous">
+            <origin xyz="0 0 0"
+                    rpy="0 0 0"/>
+            <parent link="right_steering_hinge"/>
+            <child link="right_front_wheel"/>
+            <axis xyz="0 1 0"/>
+        </joint>
+        <link name="right_front_wheel">
+            <inertial>
+                <xacro:wheels_inertia/>
+            </inertial>
+            <visual>
+                <xacro:wheels_geometry/>
+                <material name="black"/>
+            </visual>
+            <collision name="right_front_wheel_collision">
+                <geometry>
+                    <sphere radius="0.225"/>
+                </geometry>
+            </collision>
+        </link>
+        <gazebo reference="right_front_wheel">
+            <material>Gazebo/Black</material>
+        </gazebo>
+    </xacro:macro>
+    <!-- ################################################################## -->
+    <!-- #### Add the left rear wheel with its joints and tranmissions #### -->
+    <!-- ################################################################## -->
+    <xacro:body_left_rear_wheel/>
+    <!-- ################################################################### -->
+    <!-- #### Add the right rear wheel with its joints and tranmissions #### -->
+    <!-- ################################################################### -->
+    <xacro:body_right_rear_wheel/>
+    <!-- ############################################################################## -->
+    <!-- #### Add the left front wheel with its joints, steering and tranmissions #### -->
+    <!-- ############################################################################## -->
+    <xacro:body_left_front_wheel/>
+    <!-- ############################################################################## -->
+    <!-- #### Add the right front wheel with its joints, steering and tranmissions #### -->
+    <!-- ############################################################################## -->
+    <xacro:body_right_front_wheel/>
     <!-- MAIN SENSORS -->
 <!--     LOCATIONS: (XYZ)

File: eufs_description/urdf/ads-dv_base.urdf.xacro (robot description, xacro)
@@ -20,12 +20,5 @@
     </visual>
     <inertial>
-      <mass value="125.0" />
-      <origin xyz="0 0 0" />
-      <inertia  ixx="16.3"
-                ixy="0.004"
-                ixz="0.0"
-                iyy="33.6"
-                iyz="0.0"
-                izz="47.9" />
+      <xacro:chassis_inertial_params/>
     </inertial>
     <collision>

File: eufs_description/urdf/eufs_base.gazebo.xacro (robot description, xacro)
@@ -3,18 +3,4 @@
   <xacro:arg name="publish_tf" default="false"/>
   <xacro:arg name="simulate_perception" default="false"/>
-  <!-- ROS control plugin which controls all actuators in the simulation
-  This effectively looks in the namespace of the robot, finds the controller
-  interfaces based on a .yaml file (eufs_gazebo/config/eufs_control.yaml) -->
-  <xacro:macro name="ros_control">
-    <gazebo>
-      <plugin name="ros_control" filename="libgazebo_ros_control.so">
-        <robotNamespace>/eufs</robotNamespace>
-        <robotParam>robot_description</robotParam>
-        <controlPeriod>0.001</controlPeriod>
-        <robotSimType>gazebo_ros_control/DefaultRobotHWSim</robotSimType>
-        <legacyModeNS>true</legacyModeNS>
-      </plugin>
-    </gazebo>
-  </xacro:macro>
   <!-- Custom ROS plugin to simulate ground truth state in simulation.
   This node publishes nav_msgs/Odometry and eufs_msgs/CarState messages

Commit message: Fixed rviz by changing the prefix of the transforms

File: eufs_description/robots/ads-dv.urdf.xacro (robot description, xacro)
@@ -69,5 +69,5 @@
     <xacro:property name="suspension_joint_friction" value="0.1" />
     <!-- Wheels -->
-    <xacro:macro name="body_left_rear_wheel">
+    <xacro:macro name="left_rear_wheel">
         <joint name="rear_left_wheel_joint" type="continuous">
             <origin xyz="${-1 * wheelbase / 2}
@@ -97,5 +97,5 @@
         </gazebo>
     </xacro:macro>
-    <xacro:macro name="body_right_rear_wheel">
+    <xacro:macro name="right_rear_wheel">
         <joint name="rear_right_wheel_joint" type="continuous">
             <parent link="base_footprint"/>
@@ -125,5 +125,5 @@
         </gazebo>
     </xacro:macro>
-    <xacro:macro name="body_left_front_wheel">
+    <xacro:macro name="left_front_wheel">
         <joint name="left_steering_hinge_joint" type="revolute">
             <origin xyz="${1 * wheelbase / 2}
@@ -169,5 +169,5 @@
         </gazebo>
     </xacro:macro>
-    <xacro:macro name="body_right_front_wheel">
+    <xacro:macro name="right_front_wheel">
         <joint name="right_steering_hinge_joint" type="revolute">
             <parent link="base_footprint"/>
@@ -216,17 +216,17 @@
     <!-- #### Add the left rear wheel with its joints and tranmissions #### -->
     <!-- ################################################################## -->
-    <xacro:body_left_rear_wheel/>
+    <xacro:left_rear_wheel/>
     <!-- ################################################################### -->
     <!-- #### Add the right rear wheel with its joints and tranmissions #### -->
     <!-- ################################################################### -->
-    <xacro:body_right_rear_wheel/>
+    <xacro:right_rear_wheel/>
     <!-- ############################################################################## -->
     <!-- #### Add the left front wheel with its joints, steering and tranmissions #### -->
     <!-- ############################################################################## -->
-    <xacro:body_left_front_wheel/>
+    <xacro:left_front_wheel/>
     <!-- ############################################################################## -->
     <!-- #### Add the right front wheel with its joints, steering and tranmissions #### -->
     <!-- ############################################################################## -->
-    <xacro:body_right_front_wheel/>
+    <xacro:right_front_wheel/>
     <!-- *********************************************** -->
     <!--                 MAIN SENSORS                    -->
