Commit message: Refactored wheels in robot description

File: eufs_description/robots/ads-dv.urdf.xacro (robot description, xacro)
@@ -6,4 +6,5 @@
     <xacro:property name="dist" value="${load_yaml('$(arg car_dimensions_file)')}"/>
     <xacro:include filename="$(find eufs_description)/urdf/vehicle/inertias.xacro"/>
+    <xacro:include filename="$(find eufs_description)/urdf/wheels.urdf.xacro"/>
     <xacro:include filename="$(find eufs_description)/urdf/vehicle/plugins.gazebo"/>
     <!-- ***************** -->
@@ -38,195 +39,8 @@
     <xacro:eufs_base name="eufs" publish_bf="true" hq="${hq}" />
     <!-- WHEELS -->
-    <!-- hub_dia and tire_dia are the diameters of the hub and tire,
-     respectively. hex_hub_depth is the distance that the hex hub is
-     inset from the outer edge of the tire. It is set so that each wheel
-     is a "zero offset" wheel. hex_hub_depth = tire_width / 2 -
-     axle_length. -->
-    <xacro:property name="hub_dia" value="0.08"/>
-    <xacro:property name="tire_dia" value="0.505"/>
-    <xacro:property name="tire_width" value="0.2"/>
-    <xacro:property name="hex_hub_depth" value="0.120"/> <!-- or +0.072 -->
-    <xacro:property name="wheel_mass" value="10.0"/>   <!-- check -->
-    <!-- hex_hub_dist is the distance between left and right hex hubs when
-         the shock absorbers are fully extended. axle_length is the distance
-         from a U joint to the corresponding hex hub. wheel_travel is the
-         vertical wheel travel. -->
-    <xacro:property name="wheelbase" value="1.530"/>
-    <xacro:property name="hex_hub_dist" value="1.201"/>  <!-- track/width of the car -->
-    <xacro:property name="axle_length" value="0.120"/>
-    <xacro:property name="wheel_travel" value="0.05"/>
-    <xacro:property name="shock_z_offset" value="0.05"/>
-    <!-- Degree-to-radian conversions -->
-    <xacro:property name="degrees_45" value="0.785398163"/>
-    <xacro:property name="degrees_90" value="1.57079633"/>
-    <xacro:property name="degrees_180" value="3.14159265"/>
-    <!-- shock_eff_limit is 2 * ((shock_stroke / 2) * shock_spring_constant) N. -->
-    <xacro:property name="shock_eff_limit" value="50"/>
-    <xacro:property name="shock_vel_limit" value="500"/>
-    <xacro:property name="wheel_joint_damping" value="0.01" />
-    <xacro:property name="wheel_joint_friction" value="0.1" />
-    <xacro:property name="suspension_joint_damping" value="0.01" />
-    <xacro:property name="suspension_joint_friction" value="0.1" />
-    <!-- Wheels -->
-    <xacro:macro name="left_rear_wheel">
-        <joint name="rear_left_wheel_joint" type="continuous">
-            <origin xyz="${-1 * wheelbase / 2}
-                         ${1 * ((hex_hub_dist / 2) - axle_length)}
-                         ${-wheel_travel}"
-                    rpy="0 0 0"/>
-            <parent link="base_footprint"/>
-            <child link="left_rear_wheel"/>
-            <axis xyz="0 1 0"/>
-        </joint>
-        <link name="left_rear_wheel">
-            <inertial>
-                <xacro:wheels_inertia/>
-            </inertial>
-            <visual>
-                <xacro:wheels_geometry/>
-                <material name="black"/>
-            </visual>
-            <collision name="left_rear_wheel_collision">
-                <geometry>
-                    <sphere radius="0.225"/>
-                </geometry>
-            </collision>
-        </link>
-        <gazebo reference="left_rear_wheel">
-            <material>Gazebo/Black</material>
-        </gazebo>
-    </xacro:macro>
-    <xacro:macro name="right_rear_wheel">
-        <joint name="rear_right_wheel_joint" type="continuous">
-            <parent link="base_footprint"/>
-            <child link="right_rear_wheel"/>
-            <origin xyz="${-1 * wheelbase / 2}
-                         ${-1 * ((hex_hub_dist / 2) - axle_length)}
-                         ${-wheel_travel}"
-                    rpy="0 0 0"/>
-            <axis xyz="0 1 0"/>
-        </joint>
-        <link name="right_rear_wheel">
-            <inertial>
-                <xacro:wheels_inertia/>
-            </inertial>
-            <visual>
-                <xacro:wheels_geometry/>
-                <material name="black"/>
-            </visual>
-            <collision name="right_rear_wheel_collision">
-                <geometry>
-                    <sphere radius="0.225"/>
-                </geometry>
-            </collision>
-        </link>
-        <gazebo reference="right_rear_wheel">
-            <material>Gazebo/Black</material>
-        </gazebo>
-    </xacro:macro>
-    <xacro:macro name="left_front_wheel">
-        <joint name="left_steering_hinge_joint" type="revolute">
-            <origin xyz="${1 * wheelbase / 2}
-                         ${1 * ((hex_hub_dist / 2) - axle_length)}
-                         ${-wheel_travel}"
-                    rpy="0 0 0"/>
-            <parent link="base_footprint"/>
-            <child link="left_steering_hinge"/>
-            <axis xyz="0 0 1"/>
-            <limit lower="-0.8727" upper="0.8727" effort="10000000" velocity="1000000"/>
-        </joint>
-        <link name="left_steering_hinge">
-            <inertial>
-                <xacro:steering_hinge_inertial_params/>
-            </inertial>
-            <visual>
-                <xacro:steering_hinge_geometry/>
-                <material name="black"/>
-            </visual>
-        </link>
-        <joint name="front_left_wheel_joint" type="continuous">
-            <origin xyz="0 0 0" rpy="0 0 0"/>
-            <parent link="left_steering_hinge"/>
-            <child link="left_front_wheel"/>
-            <axis xyz="0 1 0"/>
-        </joint>
-        <link name="left_front_wheel">
-            <inertial>
-                <xacro:wheels_inertia/>
-            </inertial>
-            <visual>
-                <xacro:wheels_geometry/>
-                <material name="black"/>
-            </visual>
-            <collision name="left_front_wheel_collision">
-                <geometry>
-                    <sphere radius="0.225"/>
-                </geometry>
-            </collision>
-        </link>
-        <gazebo reference="left_front_wheel">
-            <material>Gazebo/Black</material>
-        </gazebo>
-    </xacro:macro>
-    <xacro:macro name="right_front_wheel">
-        <joint name="right_steering_hinge_joint" type="revolute">
-            <parent link="base_footprint"/>
-            <child link="right_steering_hinge"/>
-            <axis xyz="0 0 1"/>
-            <origin xyz="${1 * wheelbase / 2}
-                         ${-1 * ((hex_hub_dist / 2) - axle_length)}
-                         ${-wheel_travel}"
-                    rpy="0 0 0"/>
-            <limit lower="-0.8727" upper="0.8727" effort="10000000" velocity="1000000"/>
-        </joint>
-        <link name="right_steering_hinge">
-            <inertial>
-                <xacro:steering_hinge_inertial_params/>
-            </inertial>
-            <visual>
-                <xacro:steering_hinge_geometry/>
-            </visual>
-        </link>
-        <joint name="front_right_wheel_joint" type="continuous">
-            <origin xyz="0 0 0"
-                    rpy="0 0 0"/>
-            <parent link="right_steering_hinge"/>
-            <child link="right_front_wheel"/>
-            <axis xyz="0 1 0"/>
-        </joint>
-        <link name="right_front_wheel">
-            <inertial>
-                <xacro:wheels_inertia/>
-            </inertial>
-            <visual>
-                <xacro:wheels_geometry/>
-                <material name="black"/>
-            </visual>
-            <collision name="right_front_wheel_collision">
-                <geometry>
-                    <sphere radius="0.225"/>
-                </geometry>
-            </collision>
-        </link>
-        <gazebo reference="right_front_wheel">
-            <material>Gazebo/Black</material>
-        </gazebo>
-    </xacro:macro>
-    <!-- ################################################################## -->
-    <!-- #### Add the left rear wheel with its joints and tranmissions #### -->
-    <!-- ################################################################## -->
-    <xacro:left_rear_wheel/>
-    <!-- ################################################################### -->
-    <!-- #### Add the right rear wheel with its joints and tranmissions #### -->
-    <!-- ################################################################### -->
-    <xacro:right_rear_wheel/>
-    <!-- ############################################################################## -->
-    <!-- #### Add the left front wheel with its joints, steering and tranmissions #### -->
-    <!-- ############################################################################## -->
-    <xacro:left_front_wheel/>
-    <!-- ############################################################################## -->
-    <!-- #### Add the right front wheel with its joints, steering and tranmissions #### -->
-    <!-- ############################################################################## -->
-    <xacro:right_front_wheel/>
+    <xacro:front_wheel lr_prefix="left" lr_reflect="1"/>
+    <xacro:front_wheel lr_prefix="right" lr_reflect="-1"/>
+    <xacro:rear_wheel lr_prefix="left" lr_reflect="1" />
+    <xacro:rear_wheel lr_prefix="right" lr_reflect="-1" />
     <!-- *********************************************** -->
     <!--                 MAIN SENSORS                    -->

Commit message: Removed reference to the fssim inertias file and replaced and occurance of a macro with its content

File: eufs_description/robots/ads-dv.urdf.xacro (robot description, xacro)
@@ -5,5 +5,4 @@
     <xacro:property name="car_settings" value="${load_yaml('$(arg car_config_file)')}"/>
     <xacro:property name="dist" value="${load_yaml('$(arg car_dimensions_file)')}"/>
-    <xacro:include filename="$(find eufs_description)/urdf/vehicle/inertias.xacro"/>
     <xacro:include filename="$(find eufs_description)/urdf/wheels.urdf.xacro"/>
     <!-- ***************** -->

File: eufs_description/urdf/ads-dv_base.urdf.xacro (robot description, xacro)
@@ -13,4 +13,8 @@
   <!-- <xacro:property name="clearance" value="${tire_dia/2.0}" /> -->
   <xacro:property name="clearance" value="0.0" />
+  <xacro:property name="base_mass" value="140"/>
+  <xacro:property name="base_x" value="0"/>
+  <xacro:property name="base_y" value="0"/>
+  <xacro:property name="base_z" value="0.1"/>
   <!-- BASE FOOTPRINT -->
   <link name="base_footprint">
@@ -22,5 +26,13 @@
     </visual>
     <inertial>
-      <xacro:chassis_inertial_params/>
+      <origin xyz="${base_x} ${base_y} ${base_z}" rpy="0 0 0" />
+      <mass value="${base_mass}" />
+      <inertia
+          ixx="16.3"
+          ixy="0"
+          ixz="0"
+          iyy="33.6"
+          iyz="0"
+          izz="47.9" />
     </inertial>
     <collision>

Commit message: Created config file for the ads-dv car and use it for the wheels in the robot description

File: eufs_description/robots/ads-dv.urdf.xacro (robot description, xacro)
@@ -5,4 +5,5 @@
     <xacro:property name="car_settings" value="${load_yaml('$(arg car_config_file)')}"/>
     <xacro:property name="dist" value="${load_yaml('$(arg car_dimensions_file)')}"/>
+    <xacro:property name="config" value="${load_yaml('$(arg config_file)')}"/>
     <xacro:include filename="$(find eufs_description)/urdf/wheels.urdf.xacro"/>
     <!-- ***************** -->

File: eufs_description/urdf/wheels.urdf.xacro (robot description, xacro)
@@ -1,12 +1,5 @@
 <?xml version="1.0"?>
 <robot name="wheels" xmlns:xacro="http://www.ros.org/wiki/xacro">
-  <xacro:property name="tire_diameter" value="0.505"/>
-  <xacro:property name="tire_width" value="0.2"/>
-  <xacro:property name="wheel_mass" value="10.0"/>   <!-- check -->
   <xacro:property name="degrees_90" value="1.5708"/>
-  <xacro:property name="wheelbase" value="1.530"/>
-  <xacro:property name="hex_hub_dist" value="1.201"/>  <!-- track/width of the car -->
-  <xacro:property name="axle_length" value="0.120"/>
-  <xacro:property name="wheel_travel" value="0.05"/>
   <!-- Description of the wheel itself -->
   <xacro:macro name="wheel"
@@ -15,12 +8,12 @@
       <inertial>
         <origin xyz="0 0 0" rpy="0 0 0" />
-        <mass value="${wheel_mass}"/>
+        <mass value="${config['wheel']['mass']}"/>
         <inertia
-            ixx="0.3"
-            ixy="0"
-            ixz="0"
-            iyy="0.2"
-            iyz="0"
-            izz="0.2"   />
+            ixx="${config['wheel']['inertia']['ixx']}"
+            ixy="${config['wheel']['inertia']['ixy']}"
+            ixz="${config['wheel']['inertia']['ixz']}"
+            iyy="${config['wheel']['inertia']['iyy']}"
+            iyz="${config['wheel']['inertia']['iyz']}"
+            izz="${config['wheel']['inertia']['izz']}"   />
       </inertial>
       <visual>
@@ -32,7 +25,7 @@
       </visual>
       <collision>
-        <origin xyz="0 0 0" rpy="0 0 0"/>
+        <origin xyz="0 0 0" rpy="${degrees_90} 0 0"/>
         <geometry>
-          <cylinder radius="${tire_diameter / 2}" length="${tire_width}"/>
+          <cylinder radius="${config['wheel']['diameter'] / 2}" length="${config['wheel']['width']}"/>
         </geometry>
       </collision>
@@ -46,24 +39,24 @@
                params="lr_prefix lr_reflect">
     <joint name="${lr_prefix}_steering_hinge_joint" type="revolute">
-      <origin xyz="${1 * wheelbase / 2}
-                   ${lr_reflect * ((hex_hub_dist / 2) - axle_length)}
-                   ${-wheel_travel}"
+      <origin xyz="${1 * config['wheel']['wheelbase'] / 2}
+                   ${lr_reflect * ((config['wheel']['hex_hub_dist'] / 2) - config['wheel']['axle_length'])}
+                   ${-config['wheel']['wheel_travel']}"
               rpy="0 0 0"/>
       <parent link="base_footprint"/>
       <child link="${lr_prefix}_steering_hinge"/>
       <axis xyz="0 0 1"/>
-      <limit lower="-0.8727" upper="0.8727" effort="10000000" velocity="1000000"/>
+      <limit lower="${config['wheel']['wheelbase'] * -1}" upper="${config['wheel']['wheelbase']}" effort="10000000" velocity="1000000"/>
     </joint>
     <link name="${lr_prefix}_steering_hinge">
       <inertial>
         <origin xyz="0 0 0" rpy="0 0 0" />
-        <mass value="1" />
+        <mass value="${config['steering_hinge']['mass']}"/>
         <inertia
-            ixx="0.004"
-            ixy="0"
-            ixz="0"
-            iyy="0.004"
-            iyz="0"
-            izz="0.004"   />
+            ixx="${config['steering_hinge']['inertia']['ixx']}"
+            ixy="${config['steering_hinge']['inertia']['ixy']}"
+            ixz="${config['steering_hinge']['inertia']['ixz']}"
+            iyy="${config['steering_hinge']['inertia']['iyy']}"
+            iyz="${config['steering_hinge']['inertia']['iyz']}"
+            izz="${config['steering_hinge']['inertia']['izz']}"   />
       </inertial>
     </link>
@@ -74,4 +67,5 @@
       <child link="${lr_prefix}_front_wheel"/>
       <axis xyz="0 1 0"/>
+      <limit lower="0" upper="0" effort="10000000" velocity="1000000"/>
     </joint>
     <xacro:wheel lr_prefix="${lr_prefix}" fr_prefix="front"/>
@@ -81,11 +75,12 @@
                params="lr_prefix lr_reflect">
     <joint name="rear_${lr_prefix}_wheel_joint" type="continuous">
-      <origin xyz="${-1 * wheelbase / 2}
-                   ${lr_reflect * ((hex_hub_dist / 2) - axle_length)}
-                   ${-wheel_travel}"
+      <origin xyz="${-1 * config['wheel']['wheelbase'] / 2}
+                   ${lr_reflect * ((config['wheel']['hex_hub_dist'] / 2) - config['wheel']['axle_length'])}
+                   ${-config['wheel']['wheel_travel']}"
               rpy="0 0 0"/>
       <parent link="base_footprint"/>
       <child link="${lr_prefix}_rear_wheel"/>
       <axis xyz="0 1 0"/>
+      <limit lower="0" upper="0" effort="10000000" velocity="1000000"/>
     </joint>
     <xacro:wheel lr_prefix="${lr_prefix}" fr_prefix="rear"/>

Commit message: Removed all the fssim car files and added all the config to the ads-dv config file

File: eufs_description/robots/ads-dv.urdf.xacro (robot description, xacro)
@@ -2,7 +2,4 @@
 <robot name="eufs"
     xmlns:xacro="http://www.ros.org/wiki/xacro">
-    <xacro:property name="robot_sensors" value="${load_yaml('$(arg sensors_config_file)')}"/>
-    <xacro:property name="car_settings" value="${load_yaml('$(arg car_config_file)')}"/>
-    <xacro:property name="dist" value="${load_yaml('$(arg car_dimensions_file)')}"/>
     <xacro:property name="config" value="${load_yaml('$(arg config_file)')}"/>
     <xacro:include filename="$(find eufs_description)/urdf/wheels.urdf.xacro"/>

File: eufs_description/urdf/eufs_base.gazebo.xacro (robot description, xacro)
@@ -20,8 +20,4 @@
   <gazebo>
     <plugin name="race_car" filename="libgazebo_race_car_model.so">
-      <chassis>base_link</chassis>
-      <base_link>base_link</base_link>
-      <cog_link>cog</cog_link>
-      <robot_name>$(arg robot_name)</robot_name>
       <vehicle_model>$(arg vehicle_model)</vehicle_model>
       <front_left_wheel>front_left_wheel_joint</front_left_wheel>
@@ -31,6 +27,5 @@
       <rear_left_wheel>rear_left_wheel_joint</rear_left_wheel>
       <rear_right_wheel>rear_right_wheel_joint</rear_right_wheel>
-      <yaml_config>$(arg car_config_file)</yaml_config>
-      <yaml_sensors>$(arg sensors_config_file)</yaml_sensors>
+      <yaml_config>$(arg config_file)</yaml_config>
     </plugin>
   </gazebo>

File: eufs_description/urdf/wheels.urdf.xacro (robot description, xacro)
@@ -33,4 +33,8 @@
     <gazebo reference="${lr_prefix}_${fr_prefix}_wheel">
       <material>Gazebo/Black</material>
+      <mu1>${config['wheel']['friction']}</mu1>
+      <mu2>${config['wheel']['friction']}</mu2>
+      <!-- <minDepth>0.005</minDepth> -->
+      <kp>${config['wheel']['kp']}</kp>
     </gazebo>
   </xacro:macro>
