Commit message: Refactored urdf files

File: eufs_description/robots/ads-dv.urdf.xacro (robot description, xacro)
@@ -1,15 +1,11 @@
 <?xml version="1.0"?>
-<robot name="eufs"
-    xmlns:xacro="http://www.ros.org/wiki/xacro">
-    <xacro:property name="config" value="${load_yaml('$(arg config_file)')}"/>
-    <xacro:include filename="$(find eufs_description)/urdf/wheels.urdf.xacro"/>
+<robot name="eufs" xmlns:xacro="http://www.ros.org/wiki/xacro">
     <!-- ***************** -->
     <!-- Imported elements -->
     <!-- ***************** -->
-    <!-- First we import all posible elements defined in the urdf.xacro files. All these elements are defined as macro:xacros -->
-    <!-- Import Robotnik CAR base elements -->
-    <xacro:arg name="publish_tf" default="false"/>
-    <xacro:arg name="simulate_perception" default="false"/>
-    <xacro:include filename="$(find eufs_description)/urdf/ads-dv_base.urdf.xacro">
+    <!--  Import the wheels  -->
+    <xacro:include filename="$(find eufs_description)/urdf/wheels.urdf.xacro"/>
+    <!-- Import EUFS base element with the chassis -->
+    <xacro:include filename="$(find eufs_description)/urdf/eufs_base.urdf.xacro">
         <xacro:arg name="publish_tf" value="$(arg publish_tf)"/>
         <xacro:arg name="simulate_perception" value="$(arg simulate_perception)"/>
@@ -17,26 +13,27 @@
     <!-- Import all available sensors -->
     <xacro:include filename="$(find eufs_description)/sensors/all_sensors.urdf.xacro" />
+    <!--  Include the plugins  -->
+    <xacro:arg name="publish_tf" default="false"/>
+    <xacro:arg name="simulate_perception" default="true"/>
+    <xacro:include filename="$(find eufs_description)/urdf/eufs_plugins.gazebo.xacro">
+        <xacro:arg name="publish_tf" value="$(arg publish_tf)"/>
+        <xacro:arg name="simulate_perception" value="$(arg simulate_perception)"/>
+    </xacro:include>
+    <!-- ***************** -->
+    <!-- Config parameters -->
+    <!-- ***************** -->
+    <!--  Load the config file  -->
+    <xacro:property name="config" value="${load_yaml('$(arg config_file)')}"/>
     <!-- ***************** -->
     <!-- Global parameters -->
     <!-- ***************** -->
     <xacro:property name="PI" value="3.1415926535897931"/>
-    <!-- Wheel parameters -->
-    <xacro:property name="wheel_offset_x" value="1.0" />
-    <!-- x,y,z in translation from base_link to the center of the wheel -->
-    <xacro:property name="wheel_offset_y" value="0.75" />
-    <xacro:property name="wheel_offset_z" value="0.0" />
-    <!-- Flag to select the high or low quality model -->
-    <xacro:property name="hq" value="true" />
     <!-- *************** -->
     <!-- Robots Elements -->
     <!-- *************** -->
-    <!-- Here we create the robot elements using the xacro:macros imported at the beggining of this file -->
-    <!-- Summit XL base -->
-    <xacro:eufs_base name="eufs" publish_bf="true" hq="${hq}" />
-    <!-- WHEELS -->
-    <xacro:front_wheel lr_prefix="left" lr_reflect="1"/>
-    <xacro:front_wheel lr_prefix="right" lr_reflect="-1"/>
-    <xacro:rear_wheel lr_prefix="left" lr_reflect="1" />
-    <xacro:rear_wheel lr_prefix="right" lr_reflect="-1" />
+    <!-- Chassis of the car -->
+    <xacro:eufs_base chassis_mesh="package://eufs_description/meshes/ads-dv.dae"/>
+    <!-- Wheels -->
+    <xacro:wheels chassis_width="0.98" wheelbase="1.530"></xacro:wheels>
     <!-- *********************************************** -->
     <!--                 MAIN SENSORS                    -->
@@ -47,6 +44,7 @@
     LIDAR: 1.700 0.0 -0.150
     STEREO CAM: -0.110 0.0 0.800 -->
+    <!--  TODO: Check the locations of these are correct  -->
     <xacro:sensor_imu parent="base_footprint" prefix="imu">
-        <origin xyz="-0.0 0.0 0.0" rpy="0 0 0"/>
+        <origin xyz="0.0 0.0 0.0" rpy="0 0 0"/>
     </xacro:sensor_imu>
     <xacro:sensor_gps parent="base_footprint" prefix="gps">
@@ -62,28 +60,3 @@
         </xacro:zed_camera>
     </xacro:unless>
-    <!-- *********************************************** -->
-    <!-- EXTRA SENSORS FROM THE ROBOTNIK SENSORS LIBRARY -->
-    <!-- *********************************************** -->
-    <!--     <xacro:sensor_hokuyo_utm30lx parent="base_link" prefix="lidar">
-        <origin xyz="1.700 0.0 -0.080" rpy="0 -0.0174533 0"/>
-    </xacro:sensor_hokuyo_utm30lx>
-    <xacro:sensor_hokuyo3d name="hokuyo3d" parent="base_link">
-        <origin xyz="0.9 0.0 0.450" rpy="0 0.35 0"/>
-    </xacro:sensor_hokuyo3d>
-    <xacro:sensor_hokuyo_urg04lx name="hokuyo1" parent="base_link">
-        <origin xyz="-0.1 0.0 0.33" rpy="0 0 0"/>
-    </xacro:sensor_hokuyo_urg04lx>
-    <xacro:sensor_axis name="camera" parent="base_link">
-        <origin xyz="0.19 0 0.17" rpy="0 ${15*PI/180} 0"/>
-    </xacro:sensor_axis>
-    <xacro:sensor_asus_xtion_pro name="xtion_pro" parent="base_link">
-        <origin xyz="0.3 0.0 0.3" rpy="0 0 0"/>
-    </xacro:sensor_asus_xtion_pro>
-    <xacro:sensor_kinect parent="base_link" prefix="kinect">
-        <origin xyz="0.0 0.0 0.45" rpy="0 0 0"/>
-    </xacro:sensor_kinect>
-    <xacro:BB2-08S2C-60 prefix="bee" frame="bee" name="bee"/>
-    <xacro:sensor_fotonic name="fotonic" parent="base_link">
-        <origin xyz="0.3 0.0 0.24" rpy="0 0 0"/>
-    </xacro:sensor_fotonic>   -->
 </robot>

File: eufs_description/robots/eufs.urdf.xacro (robot description, xacro)
@@ -4,81 +4,59 @@
     <!-- Imported elements -->
     <!-- ***************** -->
-    <!-- First we import all posible elements defined in the urdf.xacro files. All these elements are defined as macro:xacros -->
-    <!-- Import Robotnik CAR base elements -->
-    <xacro:include filename="$(find eufs_description)/urdf/eufs_base.urdf.xacro" />
-    <!-- Import Robotnik CAR wheels -->
-    <xacro:include filename="$(find eufs_description)/urdf/suspension_wheel.urdf.xacro" />
+    <!--  Import the wheels  -->
+    <xacro:include filename="$(find eufs_description)/urdf/wheels.urdf.xacro"/>
+    <!-- Import EUFS base element with the chassis -->
+    <xacro:include filename="$(find eufs_description)/urdf/eufs_base.urdf.xacro">
+        <xacro:arg name="publish_tf" value="$(arg publish_tf)"/>
+        <xacro:arg name="simulate_perception" value="$(arg simulate_perception)"/>
+    </xacro:include>
     <!-- Import all available sensors -->
     <xacro:include filename="$(find eufs_description)/sensors/all_sensors.urdf.xacro" />
+    <!--  Include the plugins  -->
+    <xacro:arg name="publish_tf" default="false"/>
+    <xacro:arg name="simulate_perception" default="true"/>
+    <xacro:include filename="$(find eufs_description)/urdf/eufs_plugins.gazebo.xacro">
+        <xacro:arg name="publish_tf" value="$(arg publish_tf)"/>
+        <xacro:arg name="simulate_perception" value="$(arg simulate_perception)"/>
+    </xacro:include>
+    <!-- ***************** -->
+    <!-- Config parameters -->
+    <!-- ***************** -->
+    <!--  Load the config file  -->
+    <xacro:property name="config" value="${load_yaml('$(arg config_file)')}"/>
     <!-- ***************** -->
     <!-- Global parameters -->
     <!-- ***************** -->
     <xacro:property name="PI" value="3.1415926535897931"/>
-    <!-- Wheel parameters -->
-    <xacro:property name="wheel_offset_x" value="1.0" />    <!-- x,y,z in translation from base_link to the center of the wheel -->
-    <xacro:property name="wheel_offset_y" value="0.75" />
-    <xacro:property name="wheel_offset_z" value="0.0" />
     <!-- *************** -->
     <!-- Robots Elements -->
     <!-- *************** -->
     <!-- Chassis of the car -->
-    <xacro:eufs_base name="eufs" publish_bf="true" hq="false" clearance="0.25"/>
-    <!-- Gazebo ros control pluggins -->
-    <xacro:ros_control/>
-    <!-- Gazebo skid steering pluggins -->
-    <!-- xacro:skid_steering broadcastOdomTF="1"/ -->
-    <!-- WHEELS -->
-    <xacro:front_wheel lr_prefix="left" fr_prefix="front"
-        lr_reflect="1" fr_reflect="1"/>
-    <xacro:front_wheel lr_prefix="right" fr_prefix="front"
-        lr_reflect="-1" fr_reflect="1"/>
-    <xacro:rear_wheel lr_prefix="left" fr_prefix="rear"
-        lr_reflect="1" fr_reflect="-1"/>
-    <xacro:rear_wheel lr_prefix="right" fr_prefix="rear"
-        lr_reflect="-1" fr_reflect="-1"/>
-    <!-- MAIN SENSORS -->
-    <xacro:sensor_imu parent="base_link" prefix="imu">
-        <origin xyz="0.0 0.0 0.170" rpy="0 0 0"/>
+    <xacro:eufs_base chassis_mesh="package://eufs_description/meshes/chassis.dae"/>
+    <!-- Wheels -->
+    <xacro:wheels chassis_width="1.35" wheelbase="1.530"></xacro:wheels>
+    <!-- *********************************************** -->
+    <!--                 MAIN SENSORS                    -->
+    <!-- *********************************************** -->
+    <!--     LOCATIONS: (XYZ)
+    IMU: 0.0 0.0 0.170
+    GPS: -0.110 0.0 0.9
+    LIDAR: 1.700 0.0 -0.150
+    STEREO CAM: -0.110 0.0 0.800 -->
+    <!--  TODO: Check the locations of these are correct  -->
+    <xacro:sensor_imu parent="base_footprint" prefix="imu">
+        <origin xyz="0.0 0.0 0.0" rpy="0 0 0"/>
     </xacro:sensor_imu>
-    <xacro:sensor_gps  parent="base_link" prefix="gps">
-        <origin xyz="-0.110 0.0 0.9" rpy="0 0 0"/>
+    <xacro:sensor_gps parent="base_footprint" prefix="gps">
+        <origin xyz="0.0 0.0 0.4" rpy="0 0 0"/>
     </xacro:sensor_gps>
-<!--     <xacro:sensor_hokuyo_utm30lx  parent="base_link" prefix="lidar" >
-        <origin xyz="1.700 0.0 -0.080" rpy="0 -0.0174533 0"/>
-    </xacro:sensor_hokuyo_utm30lx> -->
-    <!-- <xacro:VLP-16  parent="base_link" name="velodyne" topic="/velodyne_points" hz="10">
-        <origin xyz="1.700 0.0 -0.150" rpy="0 -0.0174533 0"/>
-    </xacro:VLP-16> -->
-    <xacro:VLP-16  parent="base_link" name="velodyne" topic="/velodyne_points" hz="10" samples="1200">
-        <origin xyz="1.700 0.0 -0.150" rpy="0 -${1.5*M_PI/180.0} 0"/>
-    </xacro:VLP-16>
-    <xacro:zed_camera parent="base_link" prefix="zed">
-        <origin xyz="-0.110 0.0 0.84" rpy="0 0 0"/>
-    </xacro:zed_camera>
-    <!-- EXTRA SENSORS FROM THE ROBOTNIK SENSORS LIBRARY -->
-<!--
-    <xacro:sensor_hokuyo3d name="hokuyo3d" parent="base_link">
-        <origin xyz="0.9 0.0 0.450" rpy="0 0.35 0"/>
-    </xacro:sensor_hokuyo3d>
-    <xacro:sensor_hokuyo_urg04lx name="hokuyo1" parent="base_link">
-        <origin xyz="-0.1 0.0 0.33" rpy="0 0 0"/>
-    </xacro:sensor_hokuyo_urg04lx>
-    <xacro:sensor_axis name="camera" parent="base_link">
-        <origin xyz="0.19 0 0.17" rpy="0 ${15*PI/180} 0"/>
-    </xacro:sensor_axis>
-    <xacro:sensor_asus_xtion_pro name="xtion_pro" parent="base_link">
-        <origin xyz="0.3 0.0 0.3" rpy="0 0 0"/>
-    </xacro:sensor_asus_xtion_pro>
-    <xacro:sensor_kinect parent="base_link" prefix="kinect">
-        <origin xyz="0.0 0.0 0.45" rpy="0 0 0"/>
-    </xacro:sensor_kinect>
-    <xacro:BB2-08S2C-60  prefix="bee" frame="bee" name="bee"/>
-    <xacro:sensor_fotonic name="fotonic" parent="base_link">
-        <origin xyz="0.3 0.0 0.24" rpy="0 0 0"/>
-    </xacro:sensor_fotonic>   -->
-    <!-- PLUGINS -->
-    <!-- ros control plugin -->
-<!--   <gazebo>
-    <plugin name="gazebo_ros_control" filename="libgazebo_ros_control.so"/>
-</gazebo> -->
+    <!-- Simulate raw perception sensors only if we're not using the abstracted perception simulation -->
+    <xacro:unless value="$(arg simulate_perception)">
+        <xacro:VLP-16R parent="base_footprint" name="velodyne" topic="/velodyne_points" hz="10" samples="800">
+            <origin xyz="1.58 0.0 -0.1" rpy="0 ${1*M_PI/180.0} 0"/>
+        </xacro:VLP-16R>
+        <xacro:zed_camera parent="base_footprint" prefix="zed">
+            <origin xyz="0.1 0.0 0.52" rpy="0 0 0"/>
+        </xacro:zed_camera>
+    </xacro:unless>
 </robot>

File: eufs_description/robots/wheelchair.urdf.xacro (robot description, xacro)
@@ -4,9 +4,25 @@
     <!-- Imported elements -->
     <!-- ***************** -->
-    <!-- First we import all posible elements defined in the urdf.xacro files. All these elements are defined as macro:xacros -->
-    <!-- Import Robotnik CAR base elements -->
-    <xacro:include filename="$(find eufs_description)/urdf/eufs_base.urdf.xacro" />
+    <!--  Import the wheels  -->
+    <xacro:include filename="$(find eufs_description)/urdf/wheels.urdf.xacro"/>
+    <!-- Import EUFS base element with the chassis -->
+    <xacro:include filename="$(find eufs_description)/urdf/eufs_base.urdf.xacro">
+        <xacro:arg name="publish_tf" value="$(arg publish_tf)"/>
+        <xacro:arg name="simulate_perception" value="$(arg simulate_perception)"/>
+    </xacro:include>
     <!-- Import all available sensors -->
     <xacro:include filename="$(find eufs_description)/sensors/all_sensors.urdf.xacro" />
+    <!--  Include the plugins  -->
+    <xacro:arg name="publish_tf" default="false"/>
+    <xacro:arg name="simulate_perception" default="true"/>
+    <xacro:include filename="$(find eufs_description)/urdf/eufs_plugins.gazebo.xacro">
+        <xacro:arg name="publish_tf" value="$(arg publish_tf)"/>
+        <xacro:arg name="simulate_perception" value="$(arg simulate_perception)"/>
+    </xacro:include>
+    <!-- ***************** -->
+    <!-- Config parameters -->
+    <!-- ***************** -->
+    <!--  Load the config file  -->
+    <xacro:property name="config" value="${load_yaml('$(arg config_file)')}"/>
     <!-- ***************** -->
     <!-- Global parameters -->
@@ -16,22 +32,26 @@
     <!-- Robots Elements -->
     <!-- *************** -->
-    <!-- Here we create the robot elements using the xacro:macros imported at the beggining of this file -->
-    <!-- Chassis of the car -->
-    <xacro:eufs_base name="eufs" publish_bf="true" hq="false" clearance="0"/>
-    <!-- MAIN SENSORS -->
-    <!-- all sensor frames below are relative to base_footprint -->
-    <xacro:sensor_imu parent="base_link" prefix="imu">
+    <!-- Chassis of the wheelchair -->
+    <!--  NOTE: This is not the chassis of the wheelchair because at the time there is no mesh for it  -->
+    <xacro:eufs_base chassis_mesh="package://eufs_description/meshes/ads-dv.dae"/>
+    <!-- Wheels -->
+    <xacro:wheels chassis_width="1" wheelbase="1.530"></xacro:wheels>
+    <!-- *********************************************** -->
+    <!--                 MAIN SENSORS                    -->
+    <!-- *********************************************** -->
+    <xacro:sensor_imu parent="base_footprint" prefix="imu">
         <origin xyz="0.20 0.0 0.46" rpy="0 0 0"/>
     </xacro:sensor_imu>
-    <xacro:sensor_gps  parent="base_link" prefix="gps">
+    <xacro:sensor_gps  parent="base_footprint" prefix="gps">
         <origin xyz="0.0 0.0 1.095" rpy="0 0 0"/>
     </xacro:sensor_gps>
-    <xacro:VLP-16R  parent="base_link" name="velodyne" topic="/velodyne_points" hz="10" samples="1200">
-        <origin xyz="0.54 0.0 0.13" rpy="0 -${1.7*M_PI/180.0} 0"/>
-    </xacro:VLP-16R>
-    <xacro:zed_camera parent="base_link" prefix="zed">
-        <origin xyz="0.175 -0.01 0.785" rpy="0 0 0"/>
-    </xacro:zed_camera>
-    <!-- We don't have URDFs for the wheels but we're putting the frames here anyway -->
-    <!-- -0.29 +/-0.275 0.155 -->
+    <!-- Simulate raw perception sensors only if we're not using the abstracted perception simulation -->
+    <xacro:unless value="$(arg simulate_perception)">
+        <xacro:VLP-16R parent="base_footprint" name="velodyne" topic="/velodyne_points" hz="10" samples="800">
+            <origin xyz="0.54 0.0 0.13" rpy="0 ${1*M_PI/180.0} 0"/>
+        </xacro:VLP-16R>
+        <xacro:zed_camera parent="base_footprint" prefix="zed">
+            <origin xyz="0.175 -0.01 0.785" rpy="0 0 0"/>
+        </xacro:zed_camera>
+    </xacro:unless>
 </robot>

File: eufs_description/urdf/eufs_base.urdf.xacro (robot description, xacro)
@@ -1,75 +1,39 @@
 <?xml version="1.0"?>
 <robot name="eufs" xmlns:xacro="http://www.ros.org/wiki/xacro">
-  <xacro:arg name="publish_tf" default="false"/>
-  <xacro:arg name="simulate_perception" default="false"/>
-  <xacro:include filename="$(find eufs_description)/urdf/eufs_base.gazebo.xacro">
-    <xacro:arg name="publish_tf" value="$(arg publish_tf)"/>
-    <xacro:arg name="simulate_perception" value="$(arg simulate_perception)"/>
-  </xacro:include>
-  <xacro:macro name="eufs_base" params="name publish_bf hq clearance">
-  <!-- Robot mechanical and motor parameters -->
-  <xacro:property name="PI" value="3.1415926535897931"/>
-  <xacro:property name="wheel_width" value="0.175" />
-  <!-- BASE FOOTPRINT -->
-  <xacro:if value="${publish_bf}">
-    <link name="base_footprint">
+  <xacro:macro name="eufs_base" params="chassis_mesh">
+    <!-- BASE FOOTPRINT -->
+    <link name="base_footprint"/>
+    <joint name="chassis_joint" type="fixed">
+      <parent link="base_footprint"/>
+      <child link="chassis"/>
+      <origin xyz="0 0 0"
+              rpy="0 0 0"/>
+      <axis xyz="1 0 0"/>
+    </joint>
+    <link name="chassis">
       <visual>
-          <origin xyz="0 0 0" rpy="0 0 0" />
-          <geometry>
-             <box size="0.001 0.001 0.001" />
-          </geometry>
+        <origin xyz="0 0 0" rpy="0 0 0" />
+        <geometry>
+          <mesh filename="${chassis_mesh}"/>
+        </geometry>
       </visual>
+      <inertial>
+        <origin xyz="0 0 0" rpy="0 0 0" />
+        <mass value="140" />
+        <inertia
+            ixx="16.3"
+            ixy="0"
+            ixz="0"
+            iyy="33.6"
+            iyz="0"
+            izz="47.9" />
+      </inertial>
+      <collision>
+        <origin xyz="0 0 0" rpy="0 0 0" />
+        <geometry>
+          <mesh filename="${chassis_mesh}"/>
+        </geometry>
+      </collision>
     </link>
-    <joint name="base_footprint_joint" type="fixed">
-      <origin xyz="0 0 ${clearance}" rpy="0 0 0" />  <!-- height is the clearance -->
-      <parent link="base_footprint"/>
-      <child link="base_link" />
-    </joint>
-  </xacro:if>
-  <!-- BASE_LINK -->
-  <link name="base_link">
-    <inertial>
-      <mass value="125.0" />
-      <origin xyz="0 0 0" />
-      <inertia  ixx="1.391" ixy="0.004"  ixz="0.0"  iyy="6.853"  iyz="0.0"  izz="6.125" />
-    </inertial>
-    <visual>
-       <origin xyz="0 0 0" rpy="0 0 0" />
-       <xacro:if value="${hq}">
-       <geometry>
-	     <mesh filename="package://eufs_description/meshes/chassis.dae"/>
-       </geometry>
-       </xacro:if>
-       <xacro:unless value="${hq}">
-       <geometry>
-	     <mesh filename="package://eufs_description/meshes/chassis.dae"/>
-       </geometry>
-       </xacro:unless>
-    </visual>
-    <collision>
-       <origin xyz="0 0 0" rpy="0 0 0 " />
-       <geometry>
-         <mesh filename="package://eufs_description/meshes/chassis_collision.dae"/>
-       </geometry>
-    </collision>
-  </link>
-  <link name="odom_ground_truth">
-    <collision>
-      <geometry>
-        <box size="0.1 0.1 0.1"/>
-      </geometry>
-    </collision>
-    <inertial>
-      <mass value="1e-5" />
-      <origin xyz="0 0 0" rpy="0 0 0"/>
-      <inertia ixx="1e-6" ixy="0" ixz="0" iyy="1e-6" iyz="0" izz="1e-6" />
-    </inertial>
-  </link>
-  <joint name="odom_ground_truth_joint" type="fixed">
-    <axis xyz="0 0 0" />
-    <origin xyz="0 0 0" rpy="0 0 0"/>
-    <parent link="base_link"/>
-    <child link="odom_ground_truth"/>
-  </joint>
   </xacro:macro>
 </robot>

File: eufs_description/urdf/eufs_plugins.gazebo.xacro (robot description, xacro)
@@ -3,16 +3,4 @@
   <xacro:arg name="publish_tf" default="false"/>
   <xacro:arg name="simulate_perception" default="false"/>
-  <!-- Plugin which publishes the state of the given joint
-   The given joint are use in the race_car plugin-->
-  <gazebo>
-    <plugin filename="libgazebo_ros_joint_state_publisher.so" name="joint_state_publisher">
-      <jointName>front_right_wheel_joint, front_left_wheel_joint, rear_right_wheel_joint, rear_left_wheel_joint,
-        right_steering_hinge_joint, left_steering_hinge_joint
-      </jointName>
-      <updateRate>500.0</updateRate>
-      <robotNamespace>/eufs</robotNamespace>
-      <alwaysOn>true</alwaysOn>
-    </plugin>
-  </gazebo>
   <!-- Custom plugin which controls the car using a given vehicle model.
    It controls the car by setting its velocity and position
