Commit message: Update noise based on gps data sheet

File: eufs_description/sensors/gps.urdf.xacro (robot description, xacro)
@@ -27,19 +27,19 @@
                 </geometry>
             </collision>
-            <!--            <visual>-->
-<!--                <origin rpy="0 0 0" xyz="0 0 0"/>-->
-<!--                <material name="gps_color">-->
-<!--                    <color rgba="1 1 1 1"/>-->
-<!--                </material>-->
-<!--                <geometry>-->
-<!--                    <mesh filename="file://$(find eufs_description)/meshes/antenna_3GO16.stl" scale="1.0 1.0 1.0"/>-->
-<!--                </geometry>-->
-<!--            </visual>-->
-<!--            <collision>-->
-<!--                <origin rpy="0 0 0" xyz="0 0 0"/>-->
-<!--                <geometry>-->
-<!--                    <mesh filename="file://$(find eufs_description)/meshes/antenna_3GO16.stl" scale="1.0 1.0 1.0"/>-->
-<!--                </geometry>-->
-<!--            </collision>-->
+<!--        <visual>-->
+<!--            <origin rpy="0 0 0" xyz="0 0 0"/>-->
+<!--            <material name="gps_color">-->
+<!--                <color rgba="1 1 1 1"/>-->
+<!--            </material>-->
+<!--            <geometry>-->
+<!--                <mesh filename="file://$(find eufs_description)/meshes/antenna_3GO16.stl" scale="1.0 1.0 1.0"/>-->
+<!--            </geometry>-->
+<!--        </visual>-->
+<!--        <collision>-->
+<!--            <origin rpy="0 0 0" xyz="0 0 0"/>-->
+<!--            <geometry>-->
+<!--                <mesh filename="file://$(find eufs_description)/meshes/antenna_3GO16.stl" scale="1.0 1.0 1.0"/>-->
+<!--            </geometry>-->
+<!--        </collision>-->
         </link>
         <gazebo reference="${prefix}_base_link">
@@ -50,5 +50,5 @@
             <sensor name="gps" type="gps">
                 <always_on>true</always_on>
-                <update_rate>10</update_rate>
+                <update_rate>5</update_rate>
                 <gps>
                     <position_sensing>
@@ -56,5 +56,5 @@
                             <noise type="gaussian">
                                 <mean>0.0</mean>
-                                <stddev>3</stddev>
+                                <stddev>2</stddev>
                             </noise>
                         </horizontal>
@@ -62,5 +62,5 @@
                             <noise type="gaussian">
                                 <mean>0.0</mean>
-                                <stddev>3</stddev>
+                                <stddev>2.5</stddev>
                             </noise>
                         </vertical>
@@ -70,5 +70,5 @@
                             <noise type="gaussian">
                                 <mean>0.0</mean>
-                                <stddev>0.2</stddev>
+                                <stddev>0.1</stddev>
                             </noise>
                         </horizontal>
@@ -76,5 +76,5 @@
                             <noise type="gaussian">
                                 <mean>0.0</mean>
-                                <stddev>0.2</stddev>
+                                <stddev>0.1</stddev>
                             </noise>
                         </vertical>
