Commit message: Add lidar sensor

File: eufs_description/sensors/VLP-16R.urdf.xacro (robot description, xacro)
@@ -2,5 +2,5 @@
 <robot xmlns:xacro="http://www.ros.org/wiki/xacro" name="VLP-16">
   <xacro:property name="M_PI" value="3.1415926535897931" />
-  <xacro:macro name="VLP-16R" params="*origin parent:=base_footprint name:=velodyne active topic:=/velodyne_points hz:=6 lasers:=5 samples:=1200 collision_range:=0.3 min_range:=0.6 max_range:=130.0 noise:=0.008 min_angle:=-2 max_angle:=2">
+  <xacro:macro name="VLP-16R" params="*origin parent:=base_footprint name:=velodyne active topic:=/velodyne_points hz:=6 lasers:=5 samples:=1200 min_range:=0.6 max_range:=130.0 noise:=0.008 min_angle:=-2 max_angle:=2">
     <joint name="${name}_base_mount_joint" type="fixed">
       <xacro:insert_block name="origin" />
@@ -56,4 +56,5 @@
       <gazebo reference="${name}">
         <sensor type="ray" name="${name}-VLP16">
+          <always_on>true</always_on>
           <pose>0 0 0 0 0 0</pose>
           <visualize>false</visualize>
@@ -63,5 +64,5 @@
               <horizontal>
                 <samples>${samples}</samples>
-                <resolution>1</resolution>
+                <resolution>1.0</resolution>
                 <min_angle>${min_angle}</min_angle>
                 <max_angle>${max_angle}</max_angle>
@@ -69,5 +70,5 @@
               <vertical>
                 <samples>${lasers}</samples>
-                <resolution>1</resolution>
+                <resolution>1.0</resolution>
                 <min_angle>-${7.0*M_PI/180.0}</min_angle>
                 <max_angle> ${1.0*M_PI/180.0}</max_angle>
@@ -75,6 +76,6 @@
             </scan>
             <range>
-              <min>${collision_range}</min>
-              <max>${max_range+1}</max>
+              <min>${min_range}</min>
+              <max>${max_range}</max>
               <resolution>0.001</resolution>
             </range>
@@ -82,16 +83,15 @@
               <type>gaussian</type>
               <mean>0.0</mean>
-              <stddev>0.0</stddev>
+              <stddev>${noise}</stddev>
             </noise>
           </ray>
-          <!--
-          <plugin name="gazebo_ros_laser_controller" filename="libgazebo_ros_velodyne_laser.so">
-            <topicName>${topic}</topicName>
-            <frameName>${name}</frameName>
-            <min_range>${min_range}</min_range>
-            <max_range>${max_range}</max_range>
-            <gaussianNoise>${noise}</gaussianNoise>
+          <plugin name="gazebo_ros_laser_controller" filename="libgazebo_ros_ray_sensor.so">
+            <ros>
+              <remapping>~/out:=${topic}</remapping>
+            </ros>
+            <frame_name>${name}</frame_name>
+            <radiation_type>infrared</radiation_type>
+            <output_type>sensor_msgs/PointCloud2</output_type>
           </plugin>
-          -->
         </sensor>
       </gazebo>

Commit message: Rename hsamples to samples

File: eufs_description/sensors/VLP-16R.urdf.xacro (robot description, xacro)
@@ -2,5 +2,5 @@
 <robot xmlns:xacro="http://www.ros.org/wiki/xacro" name="VLP-16">
   <xacro:property name="M_PI" value="3.1415926535897931" />
-  <xacro:macro name="VLP-16R" params="*origin parent:=base_footprint name:=velodyne active topic:=/velodyne_points hz:=10 lasers:=40 hsamples:=350 min_range:=0.2 max_range:=100.0 noise:=0.008 min_angle:=-2 max_angle:=2">
+  <xacro:macro name="VLP-16R" params="*origin parent:=base_footprint name:=velodyne active topic:=/velodyne_points hz:=10 lasers:=40 samples:=350 min_range:=0.2 max_range:=100.0 noise:=0.008 min_angle:=-2 max_angle:=2">
     <joint name="${name}_base_mount_joint" type="fixed">
       <xacro:insert_block name="origin" />
@@ -63,5 +63,5 @@
             <scan>
               <horizontal>
-                <samples>${hsamples}</samples>
+                <samples>${samples}</samples>
                 <resolution>1.0</resolution>
                 <min_angle>${min_angle}</min_angle>
