Commit message: Feature/camera depth

File: eufs_description/sensors/zed.urdf.xacro (robot description, xacro)
@@ -20,4 +20,5 @@
       </visual>
     </link>
+    <!-- Left and right frames -->
     <link name="${prefix}_left_camera"/>
     <link name="${prefix}_right_camera"/>
@@ -43,4 +44,11 @@
       <parent link="${prefix}_right_camera" />
       <child link="${prefix}_right_camera_optical"/>
+    </joint>
+    <!-- depth frame -->
+    <link name="${prefix}_depth_camera"/>
+    <joint name="${prefix}_depth_camera" type="fixed">
+      <parent link="${prefix}_center"/>
+      <child link="${prefix}_depth_camera"/>
+      <origin xyz="0 0.06 0" rpy="-${0.5*pi} 0 -${0.5*pi}" />
     </joint>
     <gazebo reference="${prefix}_left_camera_optical">
@@ -126,5 +134,5 @@
           <cameraInfoTopicName>rgb/camera_info</cameraInfoTopicName>
           <depthImageCameraInfoTopicName>depth/camera_info</depthImageCameraInfoTopicName>
-          <frameName>${prefix}_left_camera_optical</frameName>
+          <frameName>${prefix}_depth_camera</frameName>
           <baseline>0.12</baseline>
           <distortion_k1>0.0</distortion_k1>

Commit message: Update zed frames in zed urdf

File: eufs_description/sensors/zed.urdf.xacro (robot description, xacro)
@@ -21,38 +21,38 @@
     </link>
     <!-- Left and right frames -->
-    <link name="${prefix}_left_camera"/>
-    <link name="${prefix}_right_camera"/>
-    <link name="${prefix}_left_camera_optical"/>
-    <link name="${prefix}_right_camera_optical"/>
+    <link name="${prefix}_left_camera_frame"/>
+    <link name="${prefix}_right_camera_frame"/>
+    <link name="${prefix}_left_camera_optical_frame"/>
+    <link name="${prefix}_right_camera_optical_frame"/>
     <joint name="${prefix}_left_camera_joint" type="fixed">
       <parent link="${prefix}_center"/>
-      <child link="${prefix}_left_camera"/>
+      <child link="${prefix}_left_camera_frame"/>
       <origin xyz="0 0.06 0" rpy="0 0 0" />
     </joint>
     <joint name="${prefix}_right_camera_joint" type="fixed">
       <parent link="${prefix}_center"/>
-      <child link="${prefix}_right_camera"/>
+      <child link="${prefix}_right_camera_frame"/>
       <origin xyz="0 -0.06 0" rpy="0 0 0" />
     </joint>
     <joint name="left_camera_optical_joint" type="fixed">
       <origin xyz="0 0 0" rpy="0.0 0.0 0.0" />
-      <parent link="${prefix}_left_camera" />
-      <child link="${prefix}_left_camera_optical"/>
+      <parent link="${prefix}_left_camera_frame" />
+      <child link="${prefix}_left_camera_optical_frame"/>
     </joint>
     <joint name="right_camera_optical_joint" type="fixed">
       <origin xyz="0 0 0" rpy="0.0 0.0 0.0" />
-      <parent link="${prefix}_right_camera" />
-      <child link="${prefix}_right_camera_optical"/>
+      <parent link="${prefix}_right_camera_frame" />
+      <child link="${prefix}_right_camera_optical_frame"/>
     </joint>
     <!-- depth frame -->
-    <link name="${prefix}_depth_camera"/>
+    <link name="${prefix}_depth_camera_frame"/>
     <joint name="${prefix}_depth_camera" type="fixed">
       <parent link="${prefix}_center"/>
-      <child link="${prefix}_depth_camera"/>
+      <child link="${prefix}_depth_camera_frame"/>
       <origin xyz="0 0.06 0" rpy="-${0.5*pi} 0 -${0.5*pi}" />
     </joint>
     <!-- Simulate raw perception sensors only if we're not using the abstracted perception simulation -->
     <xacro:unless value="${active}">
-      <gazebo reference="${prefix}_left_camera_optical">
+      <gazebo reference="${prefix}_left_camera_optical_frame">
         <sensor type="multicamera" name="stereo_camera">
           <!-- see MultiSenseSLPlugin.h for available modes -->

Commit message: Comp

File: eufs_description/sensors/zed.urdf.xacro (robot description, xacro)
@@ -7,7 +7,7 @@
       <xacro:insert_block name="origin"/>
       <parent link="${parent}"/>
-      <child link="${prefix}_center"/>
+      <child link="${prefix}_camera_center"/>
     </joint>
-    <link name="${prefix}_center">
+    <link name="${prefix}_camera_center">
       <visual>
         <origin xyz="0 0 0" rpy="0 0 0"/>
@@ -26,10 +26,10 @@
     <link name="${prefix}_right_camera_optical_frame"/>
     <joint name="${prefix}_left_camera_joint" type="fixed">
-      <parent link="${prefix}_center"/>
+      <parent link="${prefix}_camera_center"/>
       <child link="${prefix}_left_camera_frame"/>
       <origin xyz="0 0.06 0" rpy="0 0 0" />
     </joint>
     <joint name="${prefix}_right_camera_joint" type="fixed">
-      <parent link="${prefix}_center"/>
+      <parent link="${prefix}_camera_center"/>
       <child link="${prefix}_right_camera_frame"/>
       <origin xyz="0 -0.06 0" rpy="0 0 0" />
@@ -48,5 +48,5 @@
     <link name="${prefix}_depth_camera_frame"/>
     <joint name="${prefix}_depth_camera" type="fixed">
-      <parent link="${prefix}_center"/>
+      <parent link="${prefix}_camera_center"/>
       <child link="${prefix}_depth_camera_frame"/>
       <origin xyz="0 0.06 0" rpy="-${0.5*pi} 0 -${0.5*pi}" />
