Commit message: make sim use new state ground truth plugin

File: eufs_description/urdf/eufs_base.gazebo.xacro (robot description, xacro)
@@ -7,5 +7,4 @@
         <robotNamespace>/eufs</robotNamespace>
         <robotParam>robot_description</robotParam>
-        <!-- controlPeriod>0.003</controlPeriod -->
         <controlPeriod>0.001</controlPeriod>
 	    <robotSimType>gazebo_ros_control/DefaultRobotHWSim</robotSimType>
@@ -15,5 +14,5 @@
 	</xacro:macro>
   <gazebo>
-    <plugin name="p3d_base_controller" filename="libgazebo_ros_p3d.so">
+    <plugin name="state_ground_truth" filename="libgazebo_state_ground_truth.so">
         <alwaysOn>true</alwaysOn>
         <updateRate>200.0</updateRate>
@@ -22,12 +21,7 @@
         <gaussianNoise>0.00</gaussianNoise>
         <frameName>world</frameName>
-        <!-- origin is at spawn location -->
         <xyzOffset>0.0 0.0 0</xyzOffset>
         <rpyOffset>0 0 0</rpyOffset>
     </plugin>
   </gazebo>
-  <!-- No Ackermann steering plugin -->
-  <!-- <gazebo reference="base_footprint">
-    <material>Gazebo/Green</material>
-  </gazebo> -->
 </robot>

Commit message: add comments and explanation to plugins

File: eufs_description/urdf/eufs_base.gazebo.xacro (robot description, xacro)
@@ -1,6 +1,8 @@
 <?xml version="1.0"?>
 <robot xmlns:xacro="http://www.ros.org/wiki/xacro">
-<arg name="publish_tf" default="false"/>
-  <!-- ros control plugin -->
+  <xacro:arg name="publish_tf" default="false"/>
+  <!-- ROS control plugin which controls all actuators in the simulation
+  This effectively looks in the namespace of the robot, finds the controller
+  interfaces based on a .yaml file (eufs_gazebo/config/eufs_control.yaml) -->
   <xacro:macro name="ros_control">
     <gazebo>
@@ -9,22 +11,26 @@
         <robotParam>robot_description</robotParam>
         <controlPeriod>0.001</controlPeriod>
-	    <robotSimType>gazebo_ros_control/DefaultRobotHWSim</robotSimType>
-      <legacyModeNS>true</legacyModeNS>
+        <robotSimType>gazebo_ros_control/DefaultRobotHWSim</robotSimType>
+        <legacyModeNS>true</legacyModeNS>
       </plugin>
     </gazebo>
-	</xacro:macro>
+  </xacro:macro>
+  <!-- Custom ROS plugin to simulate ground truth state in simulation.
+  This node publishes nav_msgs/Odometry and eufs_msgs/CarState messages
+  with added noise via parameters below. This node can additionally publish
+  a transfrom from referenceFrame to robotFrame -->
   <gazebo>
     <plugin name="state_ground_truth" filename="libgazebo_state_ground_truth.so">
-        <alwaysOn>true</alwaysOn>
-        <updateRate>200.0</updateRate>
-        <referenceFrame>map</referenceFrame>
-        <robotFrame>base_footprint</robotFrame>
-        <publishTransform>$(arg publish_tf)</publishTransform> <!-- TODO: Parametarise from launch file -->
-        <odometryTopicName>/ground_truth/odom</odometryTopicName>
-        <stateTopicName>/ground_truth/state</stateTopicName>
-        <positionNoise>0.0 0.0 0.0</positionNoise>
-        <orientationNoise>0.0 0.0 0.0</orientationNoise>
-        <linearVelocityNoise>0.0 0.0 0.0</linearVelocityNoise>
-        <angularVelocityNoise>0.0 0.0 0.0</angularVelocityNoise>
+      <alwaysOn>true</alwaysOn>
+      <updateRate>200.0</updateRate>
+      <referenceFrame>map</referenceFrame>
+      <robotFrame>base_footprint</robotFrame>
+      <publishTransform>$(arg publish_tf)</publishTransform>
+      <odometryTopicName>/ground_truth/odom</odometryTopicName>
+      <stateTopicName>/ground_truth/state</stateTopicName>
+      <positionNoise>0.0 0.0 0.0</positionNoise>
+      <orientationNoise>0.0 0.0 0.0</orientationNoise>
+      <linearVelocityNoise>0.0 0.0 0.0</linearVelocityNoise>
+      <angularVelocityNoise>0.0 0.0 0.0</angularVelocityNoise>
     </plugin>
   </gazebo>
