Commit message: fixed inertias of speed model

File: eufs_description/urdf/ads-dv_base.urdf.xacro (robot description, xacro)
@@ -1,5 +1,5 @@
 <?xml version="1.0"?>
 <robot name="eufs" xmlns:xacro="http://www.ros.org/wiki/xacro">
-  <xacro:include filename="$(find eufs_description)/urdf/bases/eufs_base.gazebo.xacro" />
+  <xacro:include filename="$(find eufs_description)/urdf/eufs_base.gazebo.xacro" />
   <xacro:macro name="eufs_base" params="name publish_bf hq">
   <!-- Robot mechanical and motor parameters -->
@@ -17,12 +17,4 @@
           </geometry>
       </visual>
-<!--
-      <collision>
-          <origin xyz="0 0 0" rpy="0 0 0" />
-          <geometry>
-            <box size="0.001 0.001 0.001" />
-          </geometry>
-      </collision>
--->
     </link>
     <joint name="base_footprint_joint" type="fixed">
@@ -37,5 +29,10 @@
       <mass value="125.0" />
       <origin xyz="0 0 0" />
-      <inertia  ixx="1.391" ixy="0.004"  ixz="0.0"  iyy="6.853"  iyz="0.0"  izz="6.125" />
+      <inertia  ixx="16.3"
+                ixy="0.004"
+                ixz="0.0"
+                iyy="33.6"
+                iyz="0.0"
+                izz="47.9" />
     </inertial>
     <visual>

File: eufs_description/urdf/suspension_wheel.urdf.xacro (robot description, xacro)
@@ -59,23 +59,20 @@
   <xacro:property name="servo_stall_torque" value="50"/>  <!-- check -->
   <xacro:property name="servo_no_load_speed" value="25"/> <!-- check -->
-  <!-- Inertia of a thick-walled cylindrical tube with open ends. Height is
-       measured along the z axis, which is the tube's axis. inner_rad and
-       outer_rad are the tube's inner and outer radii, respectively. -->
-  <xacro:macro name="thick_walled_tube_inertial"
-               params="inner_rad outer_rad height mass">
+  <!-- Inertia of a thick-walled cylindrical tube with open ends.
+       Empirically validated in simulation. Tweaked until the car
+       could stay in place without drifting. -->
+  <xacro:macro name="wheel_inertia"
+               params="mass">
     <inertial>
       <mass value="${mass}"/>
-      <inertia ixx="${(1 / 12) * mass * (3 * (inner_rad * inner_rad +
-                    outer_rad * outer_rad) + height * height)}"
-               ixy="0" ixz="0"
-               iyy="${(1 / 12) * mass * (3 * (inner_rad * inner_rad +
-                    outer_rad * outer_rad) + height * height)}"
+      <inertia ixx="0.25"
+               ixy="0"
+               ixz="0"
+               iyy="0.3"
                iyz="0"
-               izz="${mass * (inner_rad * inner_rad +
-                    outer_rad * outer_rad) / 2}"/>
+               izz="0.25"/>
     </inertial>
   </xacro:macro>
-  <!-- Null inertial element. This is needed to make the model work with
-       Gazebo. -->
+  <!-- Null inertial element. This is needed to make the model work with Gazebo. -->
   <xacro:macro name="null_inertial">
     <inertial>
@@ -93,5 +90,4 @@
                    ${lr_reflect * ((hex_hub_dist / 2) - axle_length)}
                    ${-wheel_travel}"/>
-                  <!-- ${(wheel_travel / 2) - shock_z_offset}"/-->
       <axis xyz="0 0 -1"/>
       <limit lower="${-wheel_travel / 2}" upper="${wheel_travel / 2}"
@@ -112,16 +108,4 @@
   <xacro:macro name="wheel" params="lr_prefix fr_prefix lr_reflect">
     <link name="${lr_prefix}_${fr_prefix}_axle_carrier">
-	  <!-- visual>
-        <origin xyz="0 0 0"/>
-        <geometry>
-          <cylinder radius="0.1" length="0.1"/>
-        </geometry>
-	  </visual>
-	  <collision>
-        <origin xyz="0 0 0"/>
-        <geometry>
-          <cylinder radius="0.1" length="0.1"/>
-        </geometry>
-	  </collision -->
       <xacro:null_inertial/>
     </link>
@@ -139,5 +123,4 @@
       <type>transmission_interface/SimpleTransmission</type>
       <joint name="${lr_prefix}_${fr_prefix}_axle">
-        <!-- hardwareInterface>hardware_interface/EffortJointInterface</hardwareInterface -->
         <hardwareInterface>hardware_interface/VelocityJointInterface</hardwareInterface>
       </joint>
@@ -167,7 +150,5 @@
         </geometry>
       </collision>
-      <xacro:thick_walled_tube_inertial
-          inner_rad="${hub_dia / 2}" outer_rad="${tire_dia / 2}"
-          height="${tire_width}" mass="${wheel_mass}"/>
+      <xacro:wheel_inertia mass="${wheel_mass}"/>
     </link>
     <gazebo reference="${lr_prefix}_${fr_prefix}_wheel">
@@ -182,16 +163,4 @@
                  child="${lr_prefix}_steering_link"/>
     <link name="${lr_prefix}_steering_link">
-	  <!-- visual>
-		<origin xyz="0 0 0"/>
-        <geometry>
-          <cylinder radius="0.1" length="0.1"/>
-        </geometry>
-	  </visual>
-	  <collision>
-		<origin xyz="0 0 0"/>
-        <geometry>
-          <cylinder radius="0.1" length="0.1"/>
-        </geometry>
-	  </collision -->
       <xacro:null_inertial/>
     </link>

Commit message: Fix green chassis

File: eufs_description/urdf/ads-dv_base.urdf.xacro (robot description, xacro)
@@ -7,5 +7,5 @@
   <xacro:property name="wheel_width" value="0.175" />
   <!-- <xacro:property name="clearance" value="${tire_dia/2.0}" /> -->
-  <xacro:property name="clearance" value="0.25" />
+  <xacro:property name="clearance" value="0.15" />
   <!-- BASE FOOTPRINT -->
   <xacro:if value="${publish_bf}">
@@ -13,17 +13,7 @@
       <visual>
         <origin xyz="0 0 ${clearance}" rpy="0 0 0" />  <!-- height is the clearance -->
-        <geometry>
-          <box size="0.001 0.001 0.001" />
-        </geometry>
-        <xacro:if value="${hq}">
           <geometry>
-    	      <mesh filename="package://eufs_description/meshes/ads-dv.dae"/>
+            <mesh filename="package://eufs_description/meshes/ads-dv.dae"/>
           </geometry>
-        </xacro:if>
-        <xacro:unless value="${hq}">
-          <geometry>
-    	      <mesh filename="package://eufs_description/meshes/ads-dv.dae"/>
-          </geometry>
-        </xacro:unless>
       </visual>
       <inertial>

Commit message: temp

File: eufs_description/urdf/ads-dv_base.urdf.xacro (robot description, xacro)
@@ -9,40 +9,29 @@
   <xacro:property name="clearance" value="0.25" />
   <!-- BASE FOOTPRINT -->
-  <xacro:if value="${publish_bf}">
-    <link name="base_footprint">
-      <visual>
-        <origin xyz="0 0 ${clearance}" rpy="0 0 0" />  <!-- height is the clearance -->
-        <geometry>
-          <box size="0.001 0.001 0.001" />
-        </geometry>
-        <xacro:if value="${hq}">
-          <geometry>
-    	      <mesh filename="package://eufs_description/meshes/ads-dv.dae"/>
-          </geometry>
-        </xacro:if>
-        <xacro:unless value="${hq}">
-          <geometry>
-    	      <mesh filename="package://eufs_description/meshes/ads-dv.dae"/>
-          </geometry>
-        </xacro:unless>
-      </visual>
-      <inertial>
-        <mass value="125.0" />
-        <origin xyz="0 0 0" />
-        <inertia  ixx="16.3"
-                  ixy="0.004"
-                  ixz="0.0"
-                  iyy="33.6"
-                  iyz="0.0"
-                  izz="47.9" />
-      </inertial>
-      <collision>
-        <origin xyz="0 0 0" rpy="0 0 0" />  <!-- might have to adjest height to the clearance -->
-        <geometry>
-          <mesh filename="package://eufs_description/meshes/ads-dv.dae"/>
-        </geometry>
-      </collision>
-    </link>
-  </xacro:if>
+  <link name="base_footprint">
+    <visual>
+      <origin xyz="0 0 ${clearance}" rpy="0 0 0" />  <!-- height is the clearance -->
+      <geometry>
+        <box size="0.001 0.001 0.001" />
+        <mesh filename="package://eufs_description/meshes/ads-dv.dae"/>
+      </geometry>
+    </visual>
+    <inertial>
+      <mass value="125.0" />
+      <origin xyz="0 0 0" />
+      <inertia  ixx="16.3"
+                ixy="0.004"
+                ixz="0.0"
+                iyy="33.6"
+                iyz="0.0"
+                izz="47.9" />
+    </inertial>
+    <collision>
+      <origin xyz="0 0 0" rpy="0 0 0" />  <!-- might have to adjust height to the clearance -->
+      <geometry>
+        <mesh filename="package://eufs_description/meshes/ads-dv.dae"/>
+      </geometry>
+    </collision>
+  </link>
   <link name="odom_ground_truth">
     <collision>

Commit message: changed car material and set clearance to 0

File: eufs_description/urdf/ads-dv_base.urdf.xacro (robot description, xacro)
@@ -7,5 +7,5 @@
   <xacro:property name="wheel_width" value="0.175" />
   <!-- <xacro:property name="clearance" value="${tire_dia/2.0}" /> -->
-  <xacro:property name="clearance" value="0.15" />
+  <xacro:property name="clearance" value="0.0" />
   <!-- BASE FOOTPRINT -->
   <link name="base_footprint">
@@ -27,5 +27,5 @@
     </inertial>
     <collision>
-      <origin xyz="0 0 0" rpy="0 0 0" />  <!-- might have to adjest height to the clearance -->
+      <origin xyz="0 0 ${clearance}" rpy="0 0 0" />  <!-- height is the clearance -->
       <geometry>
         <mesh filename="package://eufs_description/meshes/ads-dv.dae"/>

File: eufs_description/urdf/eufs_base.gazebo.xacro (robot description, xacro)
@@ -28,6 +28,6 @@
   </gazebo>
   <!-- No Ackermann steering plugin -->
-  <gazebo reference="base_footprint">
+  <!-- <gazebo reference="base_footprint">
     <material>Gazebo/Green</material>
-  </gazebo>
+  </gazebo> -->
 </robot>

Commit message: Created a new link for the chassis because the starting link (base_footprint) should no have inertia

File: eufs_description/urdf/ads-dv_base.urdf.xacro (robot description, xacro)
@@ -8,57 +8,45 @@
   </xacro:include>
   <xacro:macro name="eufs_base" params="name publish_bf hq">
-  <!-- Robot mechanical and motor parameters -->
-  <xacro:property name="PI" value="3.1415926535897931"/>
-  <xacro:property name="wheel_width" value="0.175" />
-  <!-- <xacro:property name="clearance" value="${tire_dia/2.0}" /> -->
-  <xacro:property name="clearance" value="0.0" />
-  <xacro:property name="base_mass" value="140"/>
-  <xacro:property name="base_x" value="0"/>
-  <xacro:property name="base_y" value="0"/>
-  <xacro:property name="base_z" value="0.1"/>
-  <!-- BASE FOOTPRINT -->
-  <link name="base_footprint">
-    <visual>
-      <origin xyz="0 0 ${clearance}" rpy="0 0 0" />  <!-- height is the clearance -->
+    <!-- Robot mechanical and motor parameters -->
+    <xacro:property name="PI" value="3.1415926535897931"/>
+    <xacro:property name="wheel_width" value="0.175" />
+  <!--   <xacro:property name="clearance" value="${tire_diameter/2.0}" />-->
+    <xacro:property name="clearance" value="0.0" />
+    <!--  These are for the position of the center of mass  -->
+    <xacro:property name="base_mass" value="140"/>
+    <!-- BASE FOOTPRINT -->
+    <link name="base_footprint"/>
+    <joint name="chassis_joint" type="fixed">
+      <parent link="base_footprint"/>
+      <child link="chassis"/>
+      <origin xyz="0 0 ${clearance}"
+              rpy="0 0 0"/>
+      <axis xyz="1 0 0"/>
+    </joint>
+    <link name="chassis">
+      <visual>
+        <origin xyz="0 0 ${clearance}" rpy="0 0 0" />
         <geometry>
           <mesh filename="package://eufs_description/meshes/ads-dv.dae"/>
         </geometry>
-    </visual>
-    <inertial>
-      <origin xyz="${base_x} ${base_y} ${base_z}" rpy="0 0 0" />
-      <mass value="${base_mass}" />
-      <inertia
-          ixx="16.3"
-          ixy="0"
-          ixz="0"
-          iyy="33.6"
-          iyz="0"
-          izz="47.9" />
-    </inertial>
-    <collision>
-      <origin xyz="0 0 ${clearance}" rpy="0 0 0" />  <!-- height is the clearance -->
-      <geometry>
-        <mesh filename="package://eufs_description/meshes/ads-dv.dae"/>
-      </geometry>
-    </collision>
-  </link>
-  <link name="odom_ground_truth">
-    <collision>
-      <geometry>
-        <box size="0.1 0.1 0.1"/>
-      </geometry>
-    </collision>
-    <inertial>
-      <mass value="1e-5" />
-      <origin xyz="0 0 0" rpy="0 0 0"/>
-      <inertia ixx="1e-6" ixy="0" ixz="0" iyy="1e-6" iyz="0" izz="1e-6" />
-    </inertial>
-  </link>
-  <joint name="odom_ground_truth_joint" type="fixed">
-    <axis xyz="0 0 0" />
-    <origin xyz="0 0 0" rpy="0 0 0"/>
-    <parent link="base_footprint"/>
-    <child link="odom_ground_truth"/>
-  </joint>
+      </visual>
+      <inertial>
+        <origin xyz="0 0 ${clearance}" rpy="0 0 0" />
+        <mass value="${base_mass}" />
+        <inertia
+            ixx="16.3"
+            ixy="0"
+            ixz="0"
+            iyy="33.6"
+            iyz="0"
+            izz="47.9" />
+      </inertial>
+      <collision>
+        <origin xyz="0 0 ${clearance}" rpy="0 0 0" />  <!-- height is the clearance -->
+        <geometry>
+          <mesh filename="package://eufs_description/meshes/ads-dv.dae"/>
+        </geometry>
+      </collision>
+    </link>
   </xacro:macro>
 </robot>
