Commit message: Moved the camera and lidar They are now in the correct positions. I also made them visible even if perception is simulated, but just do not start the plugin for them when that is the case.

File: eufs_description/robots/ads-dv/robot.urdf.xacro (robot description, xacro)
@@ -51,12 +51,9 @@
         <origin xyz="0.0 0.0 0.4" rpy="0 0 0"/>
     </xacro:sensor_gps>
-    <!-- Simulate raw perception sensors only if we're not using the abstracted perception simulation -->
-    <xacro:unless value="$(arg simulate_perception)">
-        <xacro:VLP-16R parent="base_footprint" name="velodyne" topic="/velodyne_points" hz="10" samples="800">
-            <origin xyz="1.58 0.0 -0.1" rpy="0 ${1*M_PI/180.0} 0"/>
-        </xacro:VLP-16R>
-        <xacro:zed_camera parent="base_footprint" prefix="zed">
-            <origin xyz="0.1 0.0 0.52" rpy="0 0 0"/>
-        </xacro:zed_camera>
-    </xacro:unless>
+    <xacro:VLP-16R parent="base_footprint" name="velodyne" topic="/velodyne_points" hz="10" samples="800" active="$(arg simulate_perception)">
+        <origin xyz="1.58 0.0 -0.1" rpy="0 ${1*M_PI/180.0} 0"/>
+    </xacro:VLP-16R>
+    <xacro:zed_camera parent="base_footprint" prefix="zed" active="$(arg simulate_perception)">
+        <origin xyz="0.1 0.0 0.52" rpy="0 0 0"/>
+    </xacro:zed_camera>
 </robot>

File: eufs_description/robots/eufs/robot.urdf.xacro (robot description, xacro)
@@ -1,4 +1,17 @@
 <?xml version="1.0"?>
 <robot name="eufs" xmlns:xacro="http://www.ros.org/wiki/xacro">
+    <!-- ***************** -->
+    <!-- Config parameters -->
+    <!-- ***************** -->
+    <!--  Load the config file  -->
+    <xacro:property name="config" value="${load_yaml('$(arg config_file)')}"/>
+    <!-- ***************** -->
+    <!-- Global parameters -->
+    <!-- ***************** -->
+    <xacro:property name="PI" value="3.1415926535897931"/>
+    <!-- If the gazebo_ros_race_car_model should publish the ground truth tf -->
+    <xacro:arg name="publish_tf" default="false"/>
+    <!-- If the perception stack should be simulated or if sensors should be used -->
+    <xacro:arg name="simulate_perception" default="true"/>
     <!-- ***************** -->
     <!-- Imported elements -->
@@ -14,19 +27,8 @@
     <xacro:include filename="$(find eufs_description)/sensors/all_sensors.urdf.xacro" />
     <!--  Include the plugins  -->
-    <xacro:arg name="publish_tf" default="false"/>
-    <xacro:arg name="simulate_perception" default="true"/>
     <xacro:include filename="$(find eufs_description)/urdf/eufs_plugins.gazebo.xacro">
         <xacro:arg name="publish_tf" value="$(arg publish_tf)"/>
         <xacro:arg name="simulate_perception" value="$(arg simulate_perception)"/>
     </xacro:include>
-    <!-- ***************** -->
-    <!-- Config parameters -->
-    <!-- ***************** -->
-    <!--  Load the config file  -->
-    <xacro:property name="config" value="${load_yaml('$(arg config_file)')}"/>
-    <!-- ***************** -->
-    <!-- Global parameters -->
-    <!-- ***************** -->
-    <xacro:property name="PI" value="3.1415926535897931"/>
     <!-- *************** -->
     <!-- Robots Elements -->
@@ -51,12 +53,9 @@
         <origin xyz="0.0 0.0 0.4" rpy="0 0 0"/>
     </xacro:sensor_gps>
-    <!-- Simulate raw perception sensors only if we're not using the abstracted perception simulation -->
-    <xacro:unless value="$(arg simulate_perception)">
-        <xacro:VLP-16R parent="base_footprint" name="velodyne" topic="/velodyne_points" hz="10" samples="800">
-            <origin xyz="1.58 0.0 -0.1" rpy="0 ${1*M_PI/180.0} 0"/>
-        </xacro:VLP-16R>
-        <xacro:zed_camera parent="base_footprint" prefix="zed">
-            <origin xyz="0.1 0.0 0.52" rpy="0 0 0"/>
-        </xacro:zed_camera>
-    </xacro:unless>
+    <xacro:VLP-16R parent="base_footprint" name="velodyne" topic="/velodyne_points" hz="10" samples="800" active="$(arg simulate_perception)">
+        <origin xyz="-0.15 0.0 0.79" rpy="0 ${1*M_PI/180.0} 0"/>
+    </xacro:VLP-16R>
+    <xacro:zed_camera parent="base_footprint" prefix="zed" active="$(arg simulate_perception)">
+        <origin xyz="-0.08 0.0 0.76" rpy="0 0 0"/>
+    </xacro:zed_camera>
 </robot>

File: eufs_description/robots/wheelchair/robot.urdf.xacro (robot description, xacro)
@@ -46,12 +46,9 @@
         <origin xyz="0.0 0.0 1.095" rpy="0 0 0"/>
     </xacro:sensor_gps>
-    <!-- Simulate raw perception sensors only if we're not using the abstracted perception simulation -->
-    <xacro:unless value="$(arg simulate_perception)">
-        <xacro:VLP-16R parent="base_footprint" name="velodyne" topic="/velodyne_points" hz="10" samples="800">
-            <origin xyz="0.54 0.0 0.13" rpy="0 ${1*M_PI/180.0} 0"/>
-        </xacro:VLP-16R>
-        <xacro:zed_camera parent="base_footprint" prefix="zed">
-            <origin xyz="0.175 -0.01 0.785" rpy="0 0 0"/>
-        </xacro:zed_camera>
-    </xacro:unless>
+    <xacro:VLP-16R parent="base_footprint" name="velodyne" topic="/velodyne_points" hz="10" samples="800" active="$(arg simulate_perception)">
+        <origin xyz="0.54 0.0 0.13" rpy="0 ${1*M_PI/180.0} 0"/>
+    </xacro:VLP-16R>
+    <xacro:zed_camera parent="base_footprint" prefix="zed" active="$(arg simulate_perception)">
+        <origin xyz="0.175 -0.01 0.785" rpy="0 0 0"/>
+    </xacro:zed_camera>
 </robot>

File: eufs_description/sensors/VLP-16R.urdf.xacro (robot description, xacro)
@@ -2,5 +2,5 @@
 <robot xmlns:xacro="http://www.ros.org/wiki/xacro" name="VLP-16">
   <xacro:property name="M_PI" value="3.1415926535897931" />
-  <xacro:macro name="VLP-16R" params="*origin parent:=base_footprint name:=velodyne topic:=/velodyne_points hz:=6 lasers:=5 samples:=1200 collision_range:=0.3 min_range:=0.6 max_range:=130.0 noise:=0.008 min_angle:=-2 max_angle:=2">
+  <xacro:macro name="VLP-16R" params="*origin parent:=base_footprint name:=velodyne active topic:=/velodyne_points hz:=6 lasers:=5 samples:=1200 collision_range:=0.3 min_range:=0.6 max_range:=130.0 noise:=0.008 min_angle:=-2 max_angle:=2">
     <joint name="${name}_base_mount_joint" type="fixed">
       <xacro:insert_block name="origin" />
@@ -51,45 +51,48 @@
       </visual>
     </link>
-    <!-- Gazebo requires the velodyne_gazebo_plugins package -->
-    <gazebo reference="${name}">
-      <sensor type="ray" name="${name}-VLP16">
-        <pose>0 0 0 0 0 0</pose>
-        <visualize>false</visualize>
-        <update_rate>${hz}</update_rate>
-        <ray>
-          <scan>
-            <horizontal>
-              <samples>${samples}</samples>
-              <resolution>1</resolution>
-              <min_angle>${min_angle}</min_angle>
-              <max_angle>${max_angle}</max_angle>
-            </horizontal>
-            <vertical>
-              <samples>${lasers}</samples>
-              <resolution>1</resolution>
-              <min_angle>-${7.0*M_PI/180.0}</min_angle>
-              <max_angle> ${1.0*M_PI/180.0}</max_angle>
-            </vertical>
-          </scan>
-          <range>
-            <min>${collision_range}</min>
-            <max>${max_range+1}</max>
-            <resolution>0.001</resolution>
-          </range>
-          <noise>
-            <type>gaussian</type>
-            <mean>0.0</mean>
-            <stddev>0.0</stddev>
-          </noise>
-        </ray>
-        <plugin name="gazebo_ros_laser_controller" filename="libgazebo_ros_velodyne_laser.so">
-          <topicName>${topic}</topicName>
-          <frameName>${name}</frameName>
-          <min_range>${min_range}</min_range>
-          <max_range>${max_range}</max_range>
-          <gaussianNoise>${noise}</gaussianNoise>
-        </plugin>
-      </sensor>
-    </gazebo>
+    <!-- Simulate raw perception sensors only if we're not using the abstracted perception simulation -->
+    <xacro:unless value="${active}">
+      <!-- Gazebo requires the velodyne_gazebo_plugins package -->
+      <gazebo reference="${name}">
+        <sensor type="ray" name="${name}-VLP16">
+          <pose>0 0 0 0 0 0</pose>
+          <visualize>false</visualize>
+          <update_rate>${hz}</update_rate>
+          <ray>
+            <scan>
+              <horizontal>
+                <samples>${samples}</samples>
+                <resolution>1</resolution>
+                <min_angle>${min_angle}</min_angle>
+                <max_angle>${max_angle}</max_angle>
+              </horizontal>
+              <vertical>
+                <samples>${lasers}</samples>
+                <resolution>1</resolution>
+                <min_angle>-${7.0*M_PI/180.0}</min_angle>
+                <max_angle> ${1.0*M_PI/180.0}</max_angle>
+              </vertical>
+            </scan>
+            <range>
+              <min>${collision_range}</min>
+              <max>${max_range+1}</max>
+              <resolution>0.001</resolution>
+            </range>
+            <noise>
+              <type>gaussian</type>
+              <mean>0.0</mean>
+              <stddev>0.0</stddev>
+            </noise>
+          </ray>
+          <plugin name="gazebo_ros_laser_controller" filename="libgazebo_ros_velodyne_laser.so">
+            <topicName>${topic}</topicName>
+            <frameName>${name}</frameName>
+            <min_range>${min_range}</min_range>
+            <max_range>${max_range}</max_range>
+            <gaussianNoise>${noise}</gaussianNoise>
+          </plugin>
+        </sensor>
+      </gazebo>
+    </xacro:unless>
   </xacro:macro>
 </robot>

File: eufs_description/sensors/gps.urdf.xacro (robot description, xacro)
@@ -17,9 +17,6 @@
             <visual>
                 <origin rpy="0 0 0" xyz="0 0 0"/>
-                <material name="gps_color">
-                    <color rgba="1 1 1 1"/>
-                </material>
                 <geometry>
-                    <mesh filename="package://eufs_description/meshes/antenna_3GO16.stl" scale="1.0 1.0 1.0"/>
+                    <box size="0.001 0.001 0.001"/>
                 </geometry>
             </visual>
@@ -27,7 +24,22 @@
                 <origin rpy="0 0 0" xyz="0 0 0"/>
                 <geometry>
-                    <mesh filename="package://eufs_description/meshes/antenna_3GO16.stl" scale="1.0 1.0 1.0"/>
+                    <box size=".001 .001 .001"/>
                 </geometry>
             </collision>
+            <!--            <visual>-->
+<!--                <origin rpy="0 0 0" xyz="0 0 0"/>-->
+<!--                <material name="gps_color">-->
+<!--                    <color rgba="1 1 1 1"/>-->
+<!--                </material>-->
+<!--                <geometry>-->
+<!--                    <mesh filename="package://eufs_description/meshes/antenna_3GO16.stl" scale="1.0 1.0 1.0"/>-->
+<!--                </geometry>-->
+<!--            </visual>-->
+<!--            <collision>-->
+<!--                <origin rpy="0 0 0" xyz="0 0 0"/>-->
+<!--                <geometry>-->
+<!--                    <mesh filename="package://eufs_description/meshes/antenna_3GO16.stl" scale="1.0 1.0 1.0"/>-->
+<!--                </geometry>-->
+<!--            </collision>-->
         </link>
         <gazebo reference="${prefix}_base_link">

File: eufs_description/sensors/zed.urdf.xacro (robot description, xacro)
@@ -2,5 +2,5 @@
 <robot name="zed_camera"
   xmlns:xacro="http://www.ros.org/wiki/xacro">
-  <xacro:macro name="zed_camera" params="prefix parent *origin">
+  <xacro:macro name="zed_camera" params="prefix parent *origin active">
     <joint name="${prefix}_base_joint" type="fixed">
       <axis xyz="1 0 0"/>
@@ -52,98 +52,101 @@
       <origin xyz="0 0.06 0" rpy="-${0.5*pi} 0 -${0.5*pi}" />
     </joint>
-    <gazebo reference="${prefix}_left_camera_optical">
-      <sensor type="multicamera" name="stereo_camera">
-        <!-- see MultiSenseSLPlugin.h for available modes -->
-        <update_rate>60.0</update_rate>
-        <camera name="${prefix}_left">
-          <pose>0 0.06 0 0 0 0</pose>
-          <horizontal_fov>1.91986</horizontal_fov>
-          <image>
-            <width>1280</width>
-            <height>720</height>
-            <format>B8G8R8</format>
-          </image>
-          <clip>
-            <near>0.5</near>
-            <far>20</far>
-          </clip>
-          <noise>
-            <type>gaussian</type>
-            <mean>0.0</mean>
-            <stddev>0.007</stddev>
-          </noise>
-        </camera>
-        <camera name="${prefix}_right">
-          <pose>0 -0.12 0 0 0 0</pose>
-          <horizontal_fov>1.91986</horizontal_fov>
-          <image>
-            <width>1280</width>
-            <height>720</height>
-            <format>B8G8R8</format>
-          </image>
-          <clip>
-            <near>0.5</near>
-            <far>20</far>
-          </clip>
-          <noise>
-            <type>gaussian</type>
-            <mean>0.0</mean>
-            <stddev>0.007</stddev>
-          </noise>
-        </camera>
-        <plugin name="stereo_camera_controller" filename="libgazebo_ros_multicamera.so">
-          <alwaysOn>true</alwaysOn>
-          <updateRate>60.0</updateRate>
-          <leftCamera>${prefix}_left</leftCamera>
-          <rightCamera>${prefix}_right</rightCamera>
-          <cameraName>${prefix}</cameraName>
-          <imageTopicName>image_rect_color</imageTopicName>
-          <cameraInfoTopicName>camera_info</cameraInfoTopicName>
-          <frameName>${prefix}_left_camera_optical</frameName>
-          <hackBaseline>0.120</hackBaseline>
-          <distortionK1>0.0</distortionK1>
-          <distortionK2>0.0</distortionK2>
-          <distortionK3>0.0</distortionK3>
-          <distortionT1>0.0</distortionT1>
-          <distortionT2>0.0</distortionT2>
-        </plugin>
-      </sensor>
-      <!-- Depth simulation -->
-      <sensor name="stereo_depth" type="depth">
-        <always_on>true</always_on>
-        <update_rate>60.0</update_rate>
-        <camera>
-          <horizontal_fov>1.91986</horizontal_fov>
-          <image>
-            <width>1280</width>
-            <height>720</height>
-            <format>B8G8R8</format>
-          </image>
-          <clip>
-            <near>0.5</near>
-            <far>20.0</far>
-          </clip>
-        </camera>
-        <plugin filename="libgazebo_ros_openni_kinect.so" name="${prefix}_controller">
-          <cameraName>${prefix}</cameraName>
-          <alwaysOn>true</alwaysOn>
-          <updateRate>60.0</updateRate>
-          <imageTopicName>dont_use</imageTopicName>
-          <depthImageTopicName>depth/depth_registered</depthImageTopicName>
-          <pointCloudTopicName>point_cloud/cloud_registered</pointCloudTopicName>
-          <cameraInfoTopicName>rgb/camera_info</cameraInfoTopicName>
-          <depthImageCameraInfoTopicName>depth/camera_info</depthImageCameraInfoTopicName>
-          <frameName>${prefix}_depth_camera</frameName>
-          <baseline>0.12</baseline>
-          <distortion_k1>0.0</distortion_k1>
-          <distortion_k2>0.0</distortion_k2>
-          <distortion_k3>0.0</distortion_k3>
-          <distortion_t1>0.0</distortion_t1>
-          <distortion_t2>0.0</distortion_t2>
-          <pointCloudCutoff>0.5</pointCloudCutoff>
-          <pointCloudCutoffMax>20.0</pointCloudCutoffMax>
-        </plugin>
-      </sensor>
-    </gazebo>
+    <!-- Simulate raw perception sensors only if we're not using the abstracted perception simulation -->
+    <xacro:unless value="${active}">
+      <gazebo reference="${prefix}_left_camera_optical">
+        <sensor type="multicamera" name="stereo_camera">
+          <!-- see MultiSenseSLPlugin.h for available modes -->
+          <update_rate>60.0</update_rate>
+          <camera name="${prefix}_left">
+            <pose>0 0.06 0 0 0 0</pose>
+            <horizontal_fov>1.91986</horizontal_fov>
+            <image>
+              <width>1280</width>
+              <height>720</height>
+              <format>B8G8R8</format>
+            </image>
+            <clip>
+              <near>0.5</near>
+              <far>20</far>
+            </clip>
+            <noise>
+              <type>gaussian</type>
+              <mean>0.0</mean>
+              <stddev>0.007</stddev>
+            </noise>
+          </camera>
+          <camera name="${prefix}_right">
+            <pose>0 -0.12 0 0 0 0</pose>
+            <horizontal_fov>1.91986</horizontal_fov>
+            <image>
+              <width>1280</width>
+              <height>720</height>
+              <format>B8G8R8</format>
+            </image>
+            <clip>
+              <near>0.5</near>
+              <far>20</far>
+            </clip>
+            <noise>
+              <type>gaussian</type>
+              <mean>0.0</mean>
+              <stddev>0.007</stddev>
+            </noise>
+          </camera>
+          <plugin name="stereo_camera_controller" filename="libgazebo_ros_multicamera.so">
+            <alwaysOn>true</alwaysOn>
+            <updateRate>60.0</updateRate>
+            <leftCamera>${prefix}_left</leftCamera>
+            <rightCamera>${prefix}_right</rightCamera>
+            <cameraName>${prefix}</cameraName>
+            <imageTopicName>image_rect_color</imageTopicName>
+            <cameraInfoTopicName>camera_info</cameraInfoTopicName>
+            <frameName>${prefix}_left_camera_optical</frameName>
+            <hackBaseline>0.120</hackBaseline>
+            <distortionK1>0.0</distortionK1>
+            <distortionK2>0.0</distortionK2>
+            <distortionK3>0.0</distortionK3>
+            <distortionT1>0.0</distortionT1>
+            <distortionT2>0.0</distortionT2>
+          </plugin>
+        </sensor>
+        <!-- Depth simulation -->
+        <sensor name="stereo_depth" type="depth">
+          <always_on>true</always_on>
+          <update_rate>60.0</update_rate>
+          <camera>
+            <horizontal_fov>1.91986</horizontal_fov>
+            <image>
+              <width>1280</width>
+              <height>720</height>
+              <format>B8G8R8</format>
+            </image>
+            <clip>
+              <near>0.5</near>
+              <far>20.0</far>
+            </clip>
+          </camera>
+          <plugin filename="libgazebo_ros_openni_kinect.so" name="${prefix}_controller">
+            <cameraName>${prefix}</cameraName>
+            <alwaysOn>true</alwaysOn>
+            <updateRate>60.0</updateRate>
+            <imageTopicName>dont_use</imageTopicName>
+            <depthImageTopicName>depth/depth_registered</depthImageTopicName>
+            <pointCloudTopicName>point_cloud/cloud_registered</pointCloudTopicName>
+            <cameraInfoTopicName>rgb/camera_info</cameraInfoTopicName>
+            <depthImageCameraInfoTopicName>depth/camera_info</depthImageCameraInfoTopicName>
+            <frameName>${prefix}_depth_camera</frameName>
+            <baseline>0.12</baseline>
+            <distortion_k1>0.0</distortion_k1>
+            <distortion_k2>0.0</distortion_k2>
+            <distortion_k3>0.0</distortion_k3>
+            <distortion_t1>0.0</distortion_t1>
+            <distortion_t2>0.0</distortion_t2>
+            <pointCloudCutoff>0.5</pointCloudCutoff>
+            <pointCloudCutoffMax>20.0</pointCloudCutoffMax>
+          </plugin>
+        </sensor>
+      </gazebo>
+    </xacro:unless>
   </xacro:macro>
 </robot>
