Commit message: Replaces package:// with file://

File: eufs_description/robots/ads-dv/robot.urdf.xacro (robot description, xacro)
@@ -33,5 +33,5 @@
     <!-- *************** -->
     <!-- Chassis of the car -->
-    <xacro:eufs_base chassis_mesh="package://eufs_description/meshes/ads-dv.dae"/>
+    <xacro:eufs_base chassis_mesh="file://ads-dv.dae"/>
     <!-- Wheels -->
     <xacro:wheels chassis_width="0.98" wheelbase="1.530"></xacro:wheels>

File: eufs_description/robots/eufs/robot.urdf.xacro (robot description, xacro)
@@ -35,5 +35,5 @@
     <!-- *************** -->
     <!-- Chassis of the car -->
-    <xacro:eufs_base chassis_mesh="package://eufs_description/meshes/sisu-20d.dae"/>
+    <xacro:eufs_base chassis_mesh="file://sisu-20d.dae"/>
     <!-- Wheels -->
     <xacro:wheels chassis_width="1.6" wheelbase="1.580"></xacro:wheels>

File: eufs_description/robots/wheelchair/robot.urdf.xacro (robot description, xacro)
@@ -34,5 +34,5 @@
     <!-- Chassis of the wheelchair -->
     <!--  NOTE: This is not the chassis of the wheelchair because at the time there is no mesh for it  -->
-    <xacro:eufs_base chassis_mesh="package://eufs_description/meshes/ads-dv.dae"/>
+    <xacro:eufs_base chassis_mesh="file://ads-dv.dae"/>
     <!-- Wheels -->
     <xacro:wheels chassis_width="1" wheelbase="1.530"></xacro:wheels>

File: eufs_description/sensors/VLP-16.urdf.xacro (robot description, xacro)
@@ -18,10 +18,10 @@
       <visual>
         <geometry>
-          <mesh filename="package://eufs_description/meshes/VLP16_base_1.dae" />
+          <mesh filename="file://VLP16_base_1.dae" />
         </geometry>
       </visual>
       <visual>
         <geometry>
-          <mesh filename="package://eufs_description/meshes/VLP16_base_2.dae" />
+          <mesh filename="file://VLP16_base_2.dae" />
         </geometry>
       </visual>
@@ -47,5 +47,5 @@
         <origin xyz="0 0 -0.0377" />
         <geometry>
-          <mesh filename="package://eufs_description/meshes/VLP16_scan.dae" />
+          <mesh filename="file://VLP16_scan.dae" />
         </geometry>
       </visual>

File: eufs_description/sensors/VLP-16R.urdf.xacro (robot description, xacro)
@@ -18,10 +18,10 @@
       <visual>
         <geometry>
-          <mesh filename="package://eufs_description/meshes/VLP16_base_1.dae" />
+          <mesh filename="file://VLP16_base_1.dae" />
         </geometry>
       </visual>
       <visual>
         <geometry>
-          <mesh filename="package://eufs_description/meshes/VLP16_base_2.dae" />
+          <mesh filename="file://VLP16_base_2.dae" />
         </geometry>
       </visual>
@@ -47,5 +47,5 @@
         <origin xyz="0 0 -0.0377" />
         <geometry>
-          <mesh filename="package://eufs_description/meshes/VLP16_scan.dae" />
+          <mesh filename="file://VLP16_scan.dae" />
         </geometry>
       </visual>

File: eufs_description/sensors/gps.urdf.xacro (robot description, xacro)
@@ -33,5 +33,5 @@
 <!--                </material>-->
 <!--                <geometry>-->
-<!--                    <mesh filename="package://eufs_description/meshes/antenna_3GO16.stl" scale="1.0 1.0 1.0"/>-->
+<!--                    <mesh filename="file://antenna_3GO16.stl" scale="1.0 1.0 1.0"/>-->
 <!--                </geometry>-->
 <!--            </visual>-->
@@ -39,5 +39,5 @@
 <!--                <origin rpy="0 0 0" xyz="0 0 0"/>-->
 <!--                <geometry>-->
-<!--                    <mesh filename="package://eufs_description/meshes/antenna_3GO16.stl" scale="1.0 1.0 1.0"/>-->
+<!--                    <mesh filename="file://antenna_3GO16.stl" scale="1.0 1.0 1.0"/>-->
 <!--                </geometry>-->
 <!--            </collision>-->

File: eufs_description/sensors/gps_with_mast.urdf.xacro (robot description, xacro)
@@ -56,5 +56,5 @@
 				</material>
 				<geometry>
-					<mesh filename="package://eufs_description/meshes/antenna_3GO16.stl" scale="1.0 1.0 1.0"/>
+					<mesh filename="file://antenna_3GO16.stl" scale="1.0 1.0 1.0"/>
 				</geometry>
 			</visual>

File: eufs_description/sensors/hokuyo_utm30lx.urdf.xacro (robot description, xacro)
@@ -15,5 +15,5 @@
 				<origin rpy="0 0 0" xyz="0 0 0"/>
 				<geometry>
-					<mesh filename="package://eufs_description/meshes/hokuyo_utm_30lx.dae"/>
+					<mesh filename="file://hokuyo_utm_30lx.dae"/>
 				</geometry>
 			</visual>

File: eufs_description/sensors/kinect.urdf.xacro (robot description, xacro)
@@ -42,5 +42,5 @@
         <origin rpy="0 0 ${M_PI/2}" xyz="0 0 0"/>
         <geometry>
-          <mesh filename="package://eufs_description/meshes/kinect.dae"/>
+          <mesh filename="file://kinect.dae"/>
         </geometry>
       </visual>

File: eufs_description/sensors/kinectv2.urdf.xacro (robot description, xacro)
@@ -53,8 +53,8 @@
       <geometry>
         <xacro:if value="${base}">
-          <mesh filename="package://eufs_description/meshes/kinectv2.dae"/>
+          <mesh filename="file://kinectv2.dae"/>
         </xacro:if>
         <xacro:unless value="${base}">
-          <mesh filename="package://eufs_description/meshes/kinectv2_nobase.dae"/>
+          <mesh filename="file://kinectv2_nobase.dae"/>
         </xacro:unless>
       </geometry>

File: eufs_description/sensors/pointgrey_bumblebee2.urdf.xacro (robot description, xacro)
@@ -70,5 +70,5 @@
         <origin xyz="0 0 0" rpy="-1.5707 0 -1.5707"/>
         <geometry>
-          <mesh filename="package://eufs_description/meshes/pointgrey_bumblebee2.dae"/>
+          <mesh filename="file://pointgrey_bumblebee2.dae"/>
         </geometry>
       </visual>

File: eufs_description/sensors/zed.urdf.xacro (robot description, xacro)
@@ -13,5 +13,5 @@
         <origin xyz="0 0 0" rpy="0 0 0"/>
         <geometry>
-          <mesh filename="package://eufs_description/meshes/zed.dae" />
+          <mesh filename="file://zed.dae" />
         </geometry>
         <material name="light_grey">

File: eufs_description/urdf/wheels.urdf.xacro (robot description, xacro)
@@ -34,5 +34,5 @@
           <origin xyz="0 0 0" rpy="${degrees_90} 0 0"/>
           <geometry>
-            <mesh filename="package://eufs_description/meshes/wheel_${lr_prefix}.dae"/>
+            <mesh filename="file://wheel_${lr_prefix}.dae"/>
           </geometry>
           <material name="tire_mat"/>

Commit message: Fixed mesh path finding

File: eufs_description/robots/ads-dv/robot.urdf.xacro (robot description, xacro)
@@ -33,5 +33,5 @@
     <!-- *************** -->
     <!-- Chassis of the car -->
-    <xacro:eufs_base chassis_mesh="file://ads-dv.dae"/>
+    <xacro:eufs_base chassis_mesh="file:///$(find eufs_description)/meshes/ads-dv.dae"/>
     <!-- Wheels -->
     <xacro:wheels chassis_width="0.98" wheelbase="1.530"></xacro:wheels>

File: eufs_description/robots/eufs/robot.urdf.xacro (robot description, xacro)
@@ -35,5 +35,5 @@
     <!-- *************** -->
     <!-- Chassis of the car -->
-    <xacro:eufs_base chassis_mesh="file://sisu-20d.dae"/>
+    <xacro:eufs_base chassis_mesh="file:///$(find eufs_description)/meshes/sisu-20d.dae"/>
     <!-- Wheels -->
     <xacro:wheels chassis_width="1.6" wheelbase="1.580"></xacro:wheels>

File: eufs_description/robots/wheelchair/robot.urdf.xacro (robot description, xacro)
@@ -34,5 +34,5 @@
     <!-- Chassis of the wheelchair -->
     <!--  NOTE: This is not the chassis of the wheelchair because at the time there is no mesh for it  -->
-    <xacro:eufs_base chassis_mesh="file://ads-dv.dae"/>
+    <xacro:eufs_base chassis_mesh="file:///$(find eufs_description)/meshes/ads-dv.dae"/>
     <!-- Wheels -->
     <xacro:wheels chassis_width="1" wheelbase="1.530"></xacro:wheels>

File: eufs_description/sensors/VLP-16.urdf.xacro (robot description, xacro)
@@ -18,10 +18,10 @@
       <visual>
         <geometry>
-          <mesh filename="file://VLP16_base_1.dae" />
+          <mesh filename="file:///$(find eufs_description)/meshes/VLP16_base_1.dae" />
         </geometry>
       </visual>
       <visual>
         <geometry>
-          <mesh filename="file://VLP16_base_2.dae" />
+          <mesh filename="file:///$(find eufs_description)/meshes/VLP16_base_2.dae" />
         </geometry>
       </visual>
@@ -47,5 +47,5 @@
         <origin xyz="0 0 -0.0377" />
         <geometry>
-          <mesh filename="file://VLP16_scan.dae" />
+          <mesh filename="file:///$(find eufs_description)/meshes/VLP16_scan.dae" />
         </geometry>
       </visual>

File: eufs_description/sensors/VLP-16R.urdf.xacro (robot description, xacro)
@@ -18,10 +18,10 @@
       <visual>
         <geometry>
-          <mesh filename="file://VLP16_base_1.dae" />
+          <mesh filename="file:///$(find eufs_description)/meshes/VLP16_base_1.dae" />
         </geometry>
       </visual>
       <visual>
         <geometry>
-          <mesh filename="file://VLP16_base_2.dae" />
+          <mesh filename="file:///$(find eufs_description)/meshes/VLP16_base_2.dae" />
         </geometry>
       </visual>
@@ -47,5 +47,5 @@
         <origin xyz="0 0 -0.0377" />
         <geometry>
-          <mesh filename="file://VLP16_scan.dae" />
+          <mesh filename="file:///$(find eufs_description)/meshes/VLP16_scan.dae" />
         </geometry>
       </visual>

File: eufs_description/sensors/gps.urdf.xacro (robot description, xacro)
@@ -33,5 +33,5 @@
 <!--                </material>-->
 <!--                <geometry>-->
-<!--                    <mesh filename="file://antenna_3GO16.stl" scale="1.0 1.0 1.0"/>-->
+<!--                    <mesh filename="file:///$(find eufs_description)/meshes/antenna_3GO16.stl" scale="1.0 1.0 1.0"/>-->
 <!--                </geometry>-->
 <!--            </visual>-->
@@ -39,5 +39,5 @@
 <!--                <origin rpy="0 0 0" xyz="0 0 0"/>-->
 <!--                <geometry>-->
-<!--                    <mesh filename="file://antenna_3GO16.stl" scale="1.0 1.0 1.0"/>-->
+<!--                    <mesh filename="file:///$(find eufs_description)/meshes/antenna_3GO16.stl" scale="1.0 1.0 1.0"/>-->
 <!--                </geometry>-->
 <!--            </collision>-->

File: eufs_description/sensors/gps_with_mast.urdf.xacro (robot description, xacro)
@@ -56,5 +56,5 @@
 				</material>
 				<geometry>
-					<mesh filename="file://antenna_3GO16.stl" scale="1.0 1.0 1.0"/>
+					<mesh filename="file:///$(find eufs_description)/meshes/antenna_3GO16.stl" scale="1.0 1.0 1.0"/>
 				</geometry>
 			</visual>

File: eufs_description/sensors/hokuyo_utm30lx.urdf.xacro (robot description, xacro)
@@ -15,5 +15,5 @@
 				<origin rpy="0 0 0" xyz="0 0 0"/>
 				<geometry>
-					<mesh filename="file://hokuyo_utm_30lx.dae"/>
+					<mesh filename="file:///$(find eufs_description)/meshes/hokuyo_utm_30lx.dae"/>
 				</geometry>
 			</visual>

File: eufs_description/sensors/kinect.urdf.xacro (robot description, xacro)
@@ -42,5 +42,5 @@
         <origin rpy="0 0 ${M_PI/2}" xyz="0 0 0"/>
         <geometry>
-          <mesh filename="file://kinect.dae"/>
+          <mesh filename="file:///$(find eufs_description)/meshes/kinect.dae"/>
         </geometry>
       </visual>

File: eufs_description/sensors/kinectv2.urdf.xacro (robot description, xacro)
@@ -53,8 +53,8 @@
       <geometry>
         <xacro:if value="${base}">
-          <mesh filename="file://kinectv2.dae"/>
+          <mesh filename="file:///$(find eufs_description)/meshes/kinectv2.dae"/>
         </xacro:if>
         <xacro:unless value="${base}">
-          <mesh filename="file://kinectv2_nobase.dae"/>
+          <mesh filename="file:///$(find eufs_description)/meshes/kinectv2_nobase.dae"/>
         </xacro:unless>
       </geometry>

File: eufs_description/sensors/pointgrey_bumblebee2.urdf.xacro (robot description, xacro)
@@ -70,5 +70,5 @@
         <origin xyz="0 0 0" rpy="-1.5707 0 -1.5707"/>
         <geometry>
-          <mesh filename="file://pointgrey_bumblebee2.dae"/>
+          <mesh filename="file:///$(find eufs_description)/meshes/pointgrey_bumblebee2.dae"/>
         </geometry>
       </visual>

File: eufs_description/sensors/zed.urdf.xacro (robot description, xacro)
@@ -13,5 +13,5 @@
         <origin xyz="0 0 0" rpy="0 0 0"/>
         <geometry>
-          <mesh filename="file://zed.dae" />
+          <mesh filename="file:///$(find eufs_description)/meshes/zed.dae" />
         </geometry>
         <material name="light_grey">

File: eufs_description/urdf/wheels.urdf.xacro (robot description, xacro)
@@ -34,5 +34,5 @@
           <origin xyz="0 0 0" rpy="${degrees_90} 0 0"/>
           <geometry>
-            <mesh filename="file://wheel_${lr_prefix}.dae"/>
+            <mesh filename="file:///$(find eufs_description)/meshes/wheel_${lr_prefix}.dae"/>
           </geometry>
           <material name="tire_mat"/>

Commit message: Fixed file paths

File: eufs_description/robots/ads-dv/robot.urdf.xacro (robot description, xacro)
@@ -33,5 +33,5 @@
     <!-- *************** -->
     <!-- Chassis of the car -->
-    <xacro:eufs_base chassis_mesh="file:///$(find eufs_description)/meshes/ads-dv.dae"/>
+    <xacro:eufs_base chassis_mesh="file://$(find eufs_description)/meshes/ads-dv.dae"/>
     <!-- Wheels -->
     <xacro:wheels chassis_width="0.98" wheelbase="1.530"></xacro:wheels>

File: eufs_description/robots/eufs/robot.urdf.xacro (robot description, xacro)
@@ -35,5 +35,5 @@
     <!-- *************** -->
     <!-- Chassis of the car -->
-    <xacro:eufs_base chassis_mesh="file:///$(find eufs_description)/meshes/sisu-20d.dae"/>
+    <xacro:eufs_base chassis_mesh="file://$(find eufs_description)/meshes/sisu-20d.dae"/>
     <!-- Wheels -->
     <xacro:wheels chassis_width="1.6" wheelbase="1.580"></xacro:wheels>

File: eufs_description/sensors/VLP-16.urdf.xacro (robot description, xacro)
@@ -18,10 +18,10 @@
       <visual>
         <geometry>
-          <mesh filename="file:///$(find eufs_description)/meshes/VLP16_base_1.dae" />
+          <mesh filename="file://$(find eufs_description)/meshes/VLP16_base_1.dae" />
         </geometry>
       </visual>
       <visual>
         <geometry>
-          <mesh filename="file:///$(find eufs_description)/meshes/VLP16_base_2.dae" />
+          <mesh filename="file://$(find eufs_description)/meshes/VLP16_base_2.dae" />
         </geometry>
       </visual>
@@ -47,5 +47,5 @@
         <origin xyz="0 0 -0.0377" />
         <geometry>
-          <mesh filename="file:///$(find eufs_description)/meshes/VLP16_scan.dae" />
+          <mesh filename="file://$(find eufs_description)/meshes/VLP16_scan.dae" />
         </geometry>
       </visual>

File: eufs_description/sensors/VLP-16R.urdf.xacro (robot description, xacro)
@@ -18,10 +18,10 @@
       <visual>
         <geometry>
-          <mesh filename="file:///$(find eufs_description)/meshes/VLP16_base_1.dae" />
+          <mesh filename="file://$(find eufs_description)/meshes/VLP16_base_1.dae" />
         </geometry>
       </visual>
       <visual>
         <geometry>
-          <mesh filename="file:///$(find eufs_description)/meshes/VLP16_base_2.dae" />
+          <mesh filename="file://$(find eufs_description)/meshes/VLP16_base_2.dae" />
         </geometry>
       </visual>
@@ -47,5 +47,5 @@
         <origin xyz="0 0 -0.0377" />
         <geometry>
-          <mesh filename="file:///$(find eufs_description)/meshes/VLP16_scan.dae" />
+          <mesh filename="file://$(find eufs_description)/meshes/VLP16_scan.dae" />
         </geometry>
       </visual>

File: eufs_description/sensors/gps.urdf.xacro (robot description, xacro)
@@ -33,5 +33,5 @@
 <!--                </material>-->
 <!--                <geometry>-->
-<!--                    <mesh filename="file:///$(find eufs_description)/meshes/antenna_3GO16.stl" scale="1.0 1.0 1.0"/>-->
+<!--                    <mesh filename="file://$(find eufs_description)/meshes/antenna_3GO16.stl" scale="1.0 1.0 1.0"/>-->
 <!--                </geometry>-->
 <!--            </visual>-->
@@ -39,5 +39,5 @@
 <!--                <origin rpy="0 0 0" xyz="0 0 0"/>-->
 <!--                <geometry>-->
-<!--                    <mesh filename="file:///$(find eufs_description)/meshes/antenna_3GO16.stl" scale="1.0 1.0 1.0"/>-->
+<!--                    <mesh filename="file://$(find eufs_description)/meshes/antenna_3GO16.stl" scale="1.0 1.0 1.0"/>-->
 <!--                </geometry>-->
 <!--            </collision>-->

File: eufs_description/sensors/gps_with_mast.urdf.xacro (robot description, xacro)
@@ -56,5 +56,5 @@
 				</material>
 				<geometry>
-					<mesh filename="file:///$(find eufs_description)/meshes/antenna_3GO16.stl" scale="1.0 1.0 1.0"/>
+					<mesh filename="file://$(find eufs_description)/meshes/antenna_3GO16.stl" scale="1.0 1.0 1.0"/>
 				</geometry>
 			</visual>

File: eufs_description/sensors/hokuyo_utm30lx.urdf.xacro (robot description, xacro)
@@ -15,5 +15,5 @@
 				<origin rpy="0 0 0" xyz="0 0 0"/>
 				<geometry>
-					<mesh filename="file:///$(find eufs_description)/meshes/hokuyo_utm_30lx.dae"/>
+					<mesh filename="file://$(find eufs_description)/meshes/hokuyo_utm_30lx.dae"/>
 				</geometry>
 			</visual>

File: eufs_description/sensors/kinect.urdf.xacro (robot description, xacro)
@@ -42,5 +42,5 @@
         <origin rpy="0 0 ${M_PI/2}" xyz="0 0 0"/>
         <geometry>
-          <mesh filename="file:///$(find eufs_description)/meshes/kinect.dae"/>
+          <mesh filename="file://$(find eufs_description)/meshes/kinect.dae"/>
         </geometry>
       </visual>

File: eufs_description/sensors/kinectv2.urdf.xacro (robot description, xacro)
@@ -53,8 +53,8 @@
       <geometry>
         <xacro:if value="${base}">
-          <mesh filename="file:///$(find eufs_description)/meshes/kinectv2.dae"/>
+          <mesh filename="file://$(find eufs_description)/meshes/kinectv2.dae"/>
         </xacro:if>
         <xacro:unless value="${base}">
-          <mesh filename="file:///$(find eufs_description)/meshes/kinectv2_nobase.dae"/>
+          <mesh filename="file://$(find eufs_description)/meshes/kinectv2_nobase.dae"/>
         </xacro:unless>
       </geometry>

File: eufs_description/sensors/pointgrey_bumblebee2.urdf.xacro (robot description, xacro)
@@ -70,5 +70,5 @@
         <origin xyz="0 0 0" rpy="-1.5707 0 -1.5707"/>
         <geometry>
-          <mesh filename="file:///$(find eufs_description)/meshes/pointgrey_bumblebee2.dae"/>
+          <mesh filename="file://$(find eufs_description)/meshes/pointgrey_bumblebee2.dae"/>
         </geometry>
       </visual>

File: eufs_description/sensors/zed.urdf.xacro (robot description, xacro)
@@ -13,5 +13,5 @@
         <origin xyz="0 0 0" rpy="0 0 0"/>
         <geometry>
-          <mesh filename="file:///$(find eufs_description)/meshes/zed.dae" />
+          <mesh filename="file://$(find eufs_description)/meshes/zed.dae" />
         </geometry>
         <material name="light_grey">

File: eufs_description/urdf/wheels.urdf.xacro (robot description, xacro)
@@ -34,5 +34,5 @@
           <origin xyz="0 0 0" rpy="${degrees_90} 0 0"/>
           <geometry>
-            <mesh filename="file:///$(find eufs_description)/meshes/wheel_${lr_prefix}.dae"/>
+            <mesh filename="file://$(find eufs_description)/meshes/wheel_${lr_prefix}.dae"/>
           </geometry>
           <material name="tire_mat"/>

Commit message: Add noise to imu

File: eufs_description/robots/ads-dv/robot.urdf.xacro (robot description, xacro)
@@ -44,9 +44,9 @@
     LIDAR: 1.700 0.0 -0.150
     STEREO CAM: -0.110 0.0 0.800 -->
-    <!-- TODO: Add sensors back -->
-<!--
     <xacro:sensor_imu parent="base_footprint" prefix="imu">
         <origin xyz="0.0 0.0 0.0" rpy="0 0 0"/>
     </xacro:sensor_imu>
+    <!-- TODO: Add sensors back -->
+<!--
     <xacro:sensor_gps parent="base_footprint" prefix="gps">
         <origin xyz="0.0 0.0 0.4" rpy="0 0 0"/>

File: eufs_description/sensors/imu.urdf.xacro (robot description, xacro)
@@ -1,5 +1,5 @@
 <?xml version="1.0"?>
 <robot name="sensor_imu" xmlns:xacro="http://www.ros.org/wiki/xacro">
-    <xacro:macro name="sensor_imu" params="prefix parent *origin">
+    <xacro:macro name="sensor_imu" params="prefix parent *origin noise:=0.08">
         <joint name="${prefix}_base_joint" type="fixed">
             <axis xyz="1 0 0"/>
@@ -34,13 +34,52 @@
                 <visualize>true</visualize>
                 <topic>__default_topic__</topic>
+                <imu>
+                    <angular_velocity>
+                        <x>
+                            <noise type="gaussian">
+                                <mean>0.0</mean>
+                                <stddev>${noise}</stddev>
+                            </noise>
+                        </x>
+                        <y>
+                            <noise type="gaussian">
+                                <mean>0.0</mean>
+                                <stddev>${noise}</stddev>
+                            </noise>
+                        </y>
+                        <z>
+                            <noise type="gaussian">
+                                <mean>0.0</mean>
+                                <stddev>${noise}</stddev>
+                            </noise>
+                        </z>
+                    </angular_velocity>
+                    <linear_acceleration>
+                        <x>
+                            <noise type="gaussian">
+                                <mean>0.0</mean>
+                                <stddev>${noise}</stddev>
+                            </noise>
+                        </x>
+                        <y>
+                            <noise type="gaussian">
+                                <mean>0.0</mean>
+                                <stddev>${noise}</stddev>
+                            </noise>
+                        </y>
+                        <z>
+                            <noise type="gaussian">
+                                <mean>0.0</mean>
+                                <stddev>${noise}</stddev>
+                            </noise>
+                        </z>
+                    </linear_acceleration>
+                </imu>
                 <plugin filename="libgazebo_ros_imu_sensor.so" name="${prefix}">
-                    <topicName>${prefix}</topicName>
-                    <bodyName>${prefix}_base_link</bodyName>
-                    <updateRateHZ>1000.0</updateRateHZ>
-                    <gaussianNoise>0.0</gaussianNoise>
-                    <xyzOffset>0 0 0</xyzOffset>
-                    <rpyOffset>0 0 0</rpyOffset>
-                    <frameName>${prefix}_base_link</frameName>
-                    <initialOrientationAsReference>false</initialOrientationAsReference>
+                    <ros>
+                        <remapping>~/out:=${prefix}</remapping>
+                    </ros>
+                    <frame_name>${prefix}_base_link</frame_name>
+                    <initial_orientation_as_reference>false</initial_orientation_as_reference>
                 </plugin>
                 <pose>0 0 0 0 0 0</pose>
