Commit message: Add IMU sensor to simulation

File: eufs_description/robots/eufs/robot.urdf.xacro (robot description, xacro)
@@ -40,9 +40,9 @@
     LIDAR: 1.700 0.0 -0.150
     STEREO CAM: -0.110 0.0 0.800 -->
-    <!-- TODO: Add sensors back -->
-<!--
     <xacro:sensor_imu parent="base_footprint" prefix="imu">
         <origin xyz="0.0 0.0 0.0" rpy="0 0 0"/>
     </xacro:sensor_imu>
+    <!-- TODO: Add sensors back -->
+<!--
     <xacro:sensor_gps parent="base_footprint" prefix="gps">
         <origin xyz="0.0 0.0 0.4" rpy="0 0 0"/>

File: eufs_description/sensors/imu.urdf.xacro (robot description, xacro)
@@ -1,41 +1,50 @@
 <?xml version="1.0"?>
 <robot name="sensor_imu" xmlns:xacro="http://www.ros.org/wiki/xacro">
-	<xacro:macro name="sensor_imu" params="prefix parent *origin">
-		<joint name="${prefix}_base_joint" type="fixed">
-			<axis xyz="1 0 0"/>
-			<xacro:insert_block name="origin"/>
-			<parent link="${parent}"/>
-			<child link="${prefix}_base_link"/>
-		</joint>
-		<link name="${prefix}_base_link">
-			<inertial>
-				<mass value="0.001"/>
-				<origin rpy="0 0 0" xyz="0 0 0"/>
-				<inertia ixx="0.0001" ixy="0" ixz="0" iyy="0.000001" iyz="0" izz="0.0001"/>
-			</inertial>
-			<visual>
-				<origin rpy="0 0 0" xyz="0 0 0"/>
-				<geometry>
-					<box size="0.001 0.001 0.001"/>
-				</geometry>
-			</visual>
-			<collision>
-				<origin rpy="0 0 0" xyz="0 0 0"/>
-				<geometry>
-					<box size=".001 .001 .001"/>
-				</geometry>
-			</collision>
-		</link>
-		<gazebo>
-            <plugin filename="libhector_gazebo_ros_imu.so" name="${prefix}_controller">
-				<alwaysOn>true</alwaysOn>
-				<bodyName>${prefix}_base_link</bodyName>
-				<topicName>${prefix}</topicName>
-				<serviceName>${prefix}_service</serviceName>
-				<gaussianNoise>0.00</gaussianNoise>
-				<updateRate>1000.0</updateRate>
-                <accelOffset>0.0 0.0 -9.81</accelOffset>
-			</plugin>
-		</gazebo>
-	</xacro:macro>
+    <xacro:macro name="sensor_imu" params="prefix parent *origin">
+        <joint name="${prefix}_base_joint" type="fixed">
+            <axis xyz="1 0 0"/>
+            <xacro:insert_block name="origin"/>
+            <parent link="${parent}"/>
+            <child link="${prefix}_base_link"/>
+        </joint>
+        <link name="${prefix}_base_link">
+            <inertial>
+                <mass value="0.001"/>
+                <origin rpy="0 0 0" xyz="0 0 0"/>
+                <inertia ixx="0.0001" ixy="0" ixz="0" iyy="0.000001" iyz="0" izz="0.0001"/>
+            </inertial>
+            <visual>
+                <origin rpy="0 0 0" xyz="0 0 0"/>
+                <geometry>
+                    <box size="0.001 0.001 0.001"/>
+                </geometry>
+            </visual>
+            <collision>
+                <origin rpy="0 0 0" xyz="0 0 0"/>
+                <geometry>
+                    <box size=".001 .001 .001"/>
+                </geometry>
+            </collision>
+        </link>
+        <gazebo reference="${prefix}_base_link">
+            <gravity>true</gravity>
+            <sensor name="imu_sensor" type="imu">
+                <always_on>true</always_on>
+                <update_rate>1000</update_rate>
+                <visualize>true</visualize>
+                <topic>__default_topic__</topic>
+                <plugin filename="libgazebo_ros_imu_sensor.so" name="${prefix}">
+                    <topicName>${prefix}</topicName>
+                    <bodyName>${prefix}_base_link</bodyName>
+                    <updateRateHZ>1000.0</updateRateHZ>
+                    <gaussianNoise>0.0</gaussianNoise>
+                    <xyzOffset>0 0 0</xyzOffset>
+                    <rpyOffset>0 0 0</rpyOffset>
+                    <frameName>${prefix}_base_link</frameName>
+                    <initialOrientationAsReference>false</initialOrientationAsReference>
+                </plugin>
+                <pose>0 0 0 0 0 0</pose>
+            </sensor>
+        </gazebo>
+    </xacro:macro>
 </robot>

Commit message: Update lidar params

File: eufs_description/robots/eufs/robot.urdf.xacro (robot description, xacro)
@@ -46,5 +46,5 @@
         <origin xyz="0.0 0.0 0.4" rpy="0 0 0"/>
     </xacro:sensor_gps>
-    <xacro:VLP-16R parent="base_footprint" name="velodyne" topic="/velodyne_points" hz="10" samples="800" active="$(arg simulate_perception)">
+    <xacro:VLP-16R parent="base_footprint" name="velodyne" topic="/velodyne_points" hz="10" active="$(arg simulate_perception)">
         <origin xyz="-0.15 0.0 0.79" rpy="0 ${1*M_PI/180.0} 0"/>
     </xacro:VLP-16R>

File: eufs_description/sensors/VLP-16R.urdf.xacro (robot description, xacro)
@@ -2,5 +2,5 @@
 <robot xmlns:xacro="http://www.ros.org/wiki/xacro" name="VLP-16">
   <xacro:property name="M_PI" value="3.1415926535897931" />
-  <xacro:macro name="VLP-16R" params="*origin parent:=base_footprint name:=velodyne active topic:=/velodyne_points hz:=6 lasers:=5 samples:=1200 min_range:=0.6 max_range:=130.0 noise:=0.008 min_angle:=-2 max_angle:=2">
+  <xacro:macro name="VLP-16R" params="*origin parent:=base_footprint name:=velodyne active topic:=/velodyne_points hz:=10 lasers:=40 hsamples:=350 min_range:=0.2 max_range:=100.0 noise:=0.008 min_angle:=-2 max_angle:=2">
     <joint name="${name}_base_mount_joint" type="fixed">
       <xacro:insert_block name="origin" />
@@ -63,5 +63,5 @@
             <scan>
               <horizontal>
-                <samples>${samples}</samples>
+                <samples>${hsamples}</samples>
                 <resolution>1.0</resolution>
                 <min_angle>${min_angle}</min_angle>
@@ -71,6 +71,6 @@
                 <samples>${lasers}</samples>
                 <resolution>1.0</resolution>
-                <min_angle>-${7.0*M_PI/180.0}</min_angle>
-                <max_angle> ${1.0*M_PI/180.0}</max_angle>
+                <min_angle>-${15.0*M_PI/180.0}</min_angle>
+                <max_angle> ${15.0*M_PI/180.0}</max_angle>
               </vertical>
             </scan>
