Commit message: remove the wacky rotations from the zed depth frame

File: eufs_sensors/urdf/zed.urdf.xacro (robot description, xacro)
@@ -50,5 +50,5 @@
       <parent link="${prefix}_camera_center"/>
       <child link="${prefix}_depth_camera_frame"/>
-      <origin xyz="0 0.06 0" rpy="-${0.5*pi} 0 -${0.5*pi}" />
+      <origin xyz="0 0.06 0" rpy="0 0 0" />
     </joint>
     <!-- Simulate raw perception sensors only if we're not using the abstracted perception simulation -->
