Commit message: Updated lidar name to VLC-32C

File: eufs_sensors/urdf/VLP-32C.urdf.xacro (robot description, xacro)
@@ -1,6 +1,6 @@
 <?xml version="1.0"?>
-<robot xmlns:xacro="http://www.ros.org/wiki/xacro" name="VLP-16">
+<robot xmlns:xacro="http://www.ros.org/wiki/xacro" name="VLP-32">
   <xacro:property name="M_PI" value="3.1415926535897931" />
-  <xacro:macro name="VLP-16R" params="*origin parent:=base_footprint name:=velodyne active topic:=/velodyne_points hz:=10 lasers:=40 samples:=600 min_range:=0.2 max_range:=200.0 noise:=0.01 min_angle:=-1.5707963 max_angle:=1.5707963">
+  <xacro:macro name="VLP-32C" params="*origin parent:=base_footprint name:=velodyne active topic:=/velodyne_points hz:=10 lasers:=40 samples:=600 min_range:=0.2 max_range:=200.0 noise:=0.01 min_angle:=-1.5707963 max_angle:=1.5707963">
     <joint name="${name}_base_mount_joint" type="fixed">
       <xacro:insert_block name="origin" />
