Commit message: Remove robots urdf file

File: eufs_racecar/robots/ads-dv/robot.urdf.xacro (robot description, xacro)
@@ -47,8 +47,8 @@
     </xacro:sensor_gps>
     <xacro:VLP-16R parent="base_footprint" name="velodyne" topic="/velodyne_points" hz="10" samples="800" active="$(arg simulate_perception)">
-        <origin xyz="1.58 0.0 -0.1" rpy="0 ${1*M_PI/180.0} 0"/>
+	<origin xyz="0.59 0.0 0.51" rpy="0 ${10*M_PI/180.0} 0"/>
     </xacro:VLP-16R>
     <xacro:zed_camera parent="base_footprint" prefix="zed" active="$(arg simulate_perception)">
-        <origin xyz="0.1 0.0 0.52" rpy="0 0 0"/>
+	<origin xyz="0.12 0.0 0.76" rpy="0 ${10.15*M_PI/180.0} 0"/>
     </xacro:zed_camera>
 </robot>

File: eufs_sensors/urdf/all_sensors.urdf.xacro (robot description, xacro)
@@ -4,16 +4,8 @@
   <!-- GPS -->
   <xacro:include filename="$(find eufs_sensors)/urdf/gps.urdf.xacro"/>
-  <!-- Hokuyo utm30lx -->
-  <xacro:include filename="$(find eufs_sensors)/urdf/hokuyo_utm30lx.urdf.xacro"/>
   <!-- Velodyne VLP-16R -->
   <xacro:include filename="$(find eufs_sensors)/urdf/VLP-16R.urdf.xacro"/>
   <!-- Imu -->
   <xacro:include filename="$(find eufs_sensors)/urdf/imu.urdf.xacro"/>
-  <!-- Kinect -->
-  <xacro:include filename="$(find eufs_sensors)/urdf/kinect.urdf.xacro"/>
-  <!-- KinectV2 -->
-  <xacro:include filename="$(find eufs_sensors)/urdf/kinectv2.urdf.xacro"/>
-  <!-- Pointgrey Bumblebee -->
-  <xacro:include filename="$(find eufs_sensors)/urdf/pointgrey_bumblebee2.urdf.xacro"/>
   <!-- ZED Stereo camera -->
   <xacro:include filename="$(find eufs_sensors)/urdf/zed.urdf.xacro"/>

Commit message: Fix ads dv urdf

File: eufs_racecar/robots/ads-dv/robot.urdf.xacro (robot description, xacro)
@@ -29,26 +29,26 @@
     <!-- *************** -->
     <!-- Chassis of the car -->
-    <xacro:eufs_base chassis_mesh="file://$(find eufs_racecar)/meshes/ads-dv.dae"/>
+    <xacro:eufs_base chassis_mesh="file://$(find eufs_racecar)/meshes/ads_dv_chassis.dae"/>
     <!-- Wheels -->
-    <xacro:wheels chassis_width="0.98" wheelbase="1.530" />
+    <xacro:wheels chassis_width="1.15" wheelbase="1.532"/>
     <!-- *********************************************** -->
     <!--                 MAIN SENSORS                    -->
     <!-- *********************************************** -->
     <!--     LOCATIONS: (XYZ)
-    IMU: 0.0 0.0 0.170
-    GPS: -0.110 0.0 0.9
-    LIDAR: 1.700 0.0 -0.150
-    STEREO CAM: -0.110 0.0 0.800 -->
-    <xacro:sensor_imu parent="base_footprint" prefix="imu">
+    IMU: 0.0 0.0 0.0
+    GPS: 0.463 0.0679 0.224
+    LIDAR: 0.243 0.0 0.324
+    STEREO CAM: 0.334 0.0 0.295 -->
+    <xacro:sensor_imu parent="chassis" prefix="imu">
         <origin xyz="0.0 0.0 0.0" rpy="0 0 0"/>
     </xacro:sensor_imu>
-    <xacro:sensor_gps parent="base_footprint" prefix="gps">
-        <origin xyz="0.0 0.0 0.4" rpy="0 0 0"/>
+    <xacro:sensor_gps parent="chassis" prefix="gps">
+        <origin xyz="0.463 0.06792 0.224" rpy="0 0 0"/>
     </xacro:sensor_gps>
-    <xacro:VLP-16R parent="base_footprint" name="velodyne" topic="/velodyne_points" hz="10" samples="800" active="$(arg simulate_perception)">
-	<origin xyz="0.59 0.0 0.51" rpy="0 ${10*M_PI/180.0} 0"/>
+    <xacro:VLP-16R parent="chassis" name="velodyne" topic="/velodyne_points" hz="10" samples="800" active="$(arg simulate_perception)">
+	    <origin xyz="0.243 0.0 0.324" rpy="0 ${6.1*M_PI/180.0} 0"/>
     </xacro:VLP-16R>
-    <xacro:zed_camera parent="base_footprint" prefix="zed" active="$(arg simulate_perception)">
-	<origin xyz="0.12 0.0 0.76" rpy="0 ${10.15*M_PI/180.0} 0"/>
+    <xacro:zed_camera parent="chassis" prefix="zed" active="$(arg simulate_perception)">
+	    <origin xyz="0.334 0.0 0.295" rpy="0 ${10.15*M_PI/180.0} 0"/>
     </xacro:zed_camera>
 </robot>

File: eufs_racecar/robots/eufs/robot.urdf.xacro (robot description, xacro)
@@ -31,5 +31,5 @@
     <xacro:eufs_base chassis_mesh="file://$(find eufs_racecar)/meshes/sisu-20d.dae"/>
     <!-- Wheels -->
-    <xacro:wheels chassis_width="1.6" wheelbase="1.580" />
+    <xacro:wheels chassis_width="1.6" wheelbase="1.580"/>
     <!-- *********************************************** -->
     <!--                 MAIN SENSORS                    -->

Commit message: Simulate IMU in Zed Camera

File: eufs_racecar/robots/ads-dv/robot.urdf.xacro (robot description, xacro)
@@ -40,5 +40,5 @@
     LIDAR: 0.243 0.0 0.324
     STEREO CAM: 0.334 0.0 0.295 -->
-    <xacro:sensor_imu parent="chassis" prefix="imu">
+    <xacro:sensor_imu parent="chassis" prefix="imu" topic_prefix="">
         <origin xyz="0.0 0.0 0.0" rpy="0 0 0"/>
     </xacro:sensor_imu>
@@ -52,3 +52,6 @@
 	    <origin xyz="0.334 0.0 0.295" rpy="0 ${10.15*M_PI/180.0} 0"/>
     </xacro:zed_camera>
+    <xacro:sensor_imu parent="chassis" prefix="zed_imu" topic_prefix="/camera">
+        <origin xyz="0.334 0.0 0.295" rpy="0 ${10.15*M_PI/180.0} 0"/>
+    </xacro:sensor_imu>
 </robot>

File: eufs_racecar/robots/eufs/robot.urdf.xacro (robot description, xacro)
@@ -40,5 +40,5 @@
     LIDAR: 1.700 0.0 -0.150
     STEREO CAM: -0.110 0.0 0.800 -->
-    <xacro:sensor_imu parent="chassis" prefix="imu">
+    <xacro:sensor_imu parent="chassis" prefix="sbg_imu" topic_prefix="">
         <origin xyz="0.0 0.0 0.0" rpy="0 0 0"/>
     </xacro:sensor_imu>
@@ -52,3 +52,6 @@
         <origin xyz="-0.08 0.0 0.76" rpy="0 0 0"/>
     </xacro:zed_camera>
+    <xacro:sensor_imu parent="chassis" prefix="zed_imu" topic_prefix="/camera">
+        <origin xyz="-0.08 0.0 0.76" rpy="0 0 0"/>
+    </xacro:sensor_imu>
 </robot>

File: eufs_sensors/urdf/all_sensors.urdf.xacro (robot description, xacro)
@@ -6,5 +6,5 @@
   <!-- Velodyne VLP-16R -->
   <xacro:include filename="$(find eufs_sensors)/urdf/VLP-16R.urdf.xacro"/>
-  <!-- Imu -->
+  <!--IMU -->
   <xacro:include filename="$(find eufs_sensors)/urdf/imu.urdf.xacro"/>
   <!-- ZED Stereo camera -->

File: eufs_sensors/urdf/imu.urdf.xacro (robot description, xacro)
@@ -1,5 +1,5 @@
 <?xml version="1.0"?>
 <robot name="sensor_imu" xmlns:xacro="http://www.ros.org/wiki/xacro">
-    <xacro:macro name="sensor_imu" params="prefix parent *origin noise:=0.08">
+    <xacro:macro name="sensor_imu" params="prefix parent topic_prefix *origin noise:=0.08">
         <joint name="${prefix}_base_joint" type="fixed">
             <axis xyz="1 0 0"/>
@@ -29,9 +29,9 @@
         <gazebo reference="${prefix}_base_link">
             <gravity>true</gravity>
-            <sensor name="imu_sensor" type="imu">
+            <sensor name="{prefix}_sensor" type="imu">
                 <always_on>true</always_on>
                 <update_rate>1000</update_rate>
                 <visualize>true</visualize>
-                <topic>__default_topic__</topic>
+                <topic>imu/data</topic>
                 <imu>
                     <angular_velocity>
@@ -78,5 +78,5 @@
                 <plugin filename="libgazebo_ros_imu_sensor.so" name="${prefix}">
                     <ros>
-                        <remapping>~/out:=${prefix}</remapping>
+                        <remapping>~/out:=${topic_prefix}/imu/data</remapping>
                     </ros>
                     <frame_name>${prefix}_base_link</frame_name>
