Commit message: updated wheel mesh

File: eufs_racecar/urdf/wheels.urdf.xacro (robot description, xacro)
@@ -8,5 +8,5 @@
     <xacro:property name="degrees_90" value="1.5708"/>
     <xacro:property name="wheel_mass" value="10.0"/>
-    <xacro:property name="wheel_diameter" value="0.505"/>
+    <xacro:property name="wheel_diameter" value="0.4064"/>
     <xacro:property name="wheel_width" value="0.2"/>
     <xacro:property name="wheel_friction_mu1" value="2"/>
@@ -14,4 +14,7 @@
     <xacro:property name="wheel_friction_kp" value="1e8"/>
     <xacro:property name="steering_hinge_mass" value="1"/>
+    <material name="black">
+        <color rgba="0 0 0 1"/>
+    </material>
     <!-- ***************** -->
     <!-- Wheel description -->
@@ -34,7 +37,8 @@
           <origin xyz="0 0 0" rpy="${degrees_90} 0 0"/>
           <geometry>
-            <mesh filename="file://$(find eufs_racecar)/meshes/wheel_${lr_prefix}.dae"/>
+            <cylinder radius="${wheel_diameter / 2}" length="${wheel_width}"/>
+            <!-- <mesh filename="file://$(find eufs_racecar)/meshes/wheel_${lr_prefix}.dae"/> -->
           </geometry>
-          <material name="tire_mat"/>
+          <material name="black"/>
         </visual>
         <collision>
