Commit message: correct wheel dims for more accurate speeds

File: eufs_racecar/urdf/chassis_base.urdf.xacro (robot description, xacro)
@@ -2,5 +2,5 @@
 <robot name="chassis_base" xmlns:xacro="http://www.ros.org/wiki/xacro">
   <xacro:macro name="chassis_base" params="chassis_mesh">
-    <xacro:property name="wheel_diameter" value="0.505"/>
+    <xacro:property name="wheel_diameter" value="0.4064"/>
     <!-- BASE FOOTPRINT -->
     <link name="base_footprint"/>

Commit message: variable base frame

File: eufs_racecar/urdf/chassis_base.urdf.xacro (robot description, xacro)
@@ -1,10 +1,10 @@
 <?xml version="1.0"?>
 <robot name="chassis_base" xmlns:xacro="http://www.ros.org/wiki/xacro">
-  <xacro:macro name="chassis_base" params="chassis_mesh">
+  <xacro:macro name="chassis_base" params="chassis_mesh base_frame">
     <xacro:property name="wheel_diameter" value="0.4064"/>
     <!-- BASE FOOTPRINT -->
-    <link name="base_footprint"/>
+    <link name="${base_frame}"/>
     <joint name="chassis_joint" type="fixed">
-      <parent link="base_footprint"/>
+      <parent link="${base_frame}"/>
       <child link="chassis"/>
       <origin xyz="0 0 ${wheel_diameter/2}"

File: eufs_racecar/urdf/robot.urdf.xacro (robot description, xacro)
@@ -6,4 +6,6 @@
     <!--  Load the config file  -->
     <xacro:property name="config" value="${load_yaml('$(arg vehicle_config)')}"/>
+    <!--  Get the parameters  -->
+    <xacro:arg name="base_frame" default="base_link"/>
     <!-- Simulate sensors or not? -->
     <xacro:arg name="enable_camera" default="false"/>
@@ -43,5 +45,5 @@
     <!-- *************** -->
     <!-- Chassis of the car -->
-    <xacro:chassis_base chassis_mesh="file://$(find eufs_racecar)/meshes/lando.dae"/>
+    <xacro:chassis_base chassis_mesh="file://$(find eufs_racecar)/meshes/lando.dae" base_frame="$(arg base_frame)"/>
     <!-- Wheels -->
     <xacro:wheels chassis_width="1.6" wheelbase="1.580"/>
