Commit message: reduce lidar scan range and density - save memory

File: eufs_racecar/urdf/VLP-32C.urdf.xacro (robot description, xacro)
@@ -2,5 +2,5 @@
 <robot name="VLP-32C_LiDAR" xmlns:xacro="http://www.ros.org/wiki/xacro">
   <xacro:property name="M_PI" value="3.1415926535897931" />
-  <xacro:macro name="VLP-32C_LiDAR" params="*origin parent prefix lidar_active scan_active hz:=10 lasers:=40 samples:=600 min_range:=0.2 max_range:=200.0 noise:=0.01 min_angle:=-1.5707963 max_angle:=1.5707963">
+  <xacro:macro name="VLP-32C_LiDAR" params="*origin parent prefix lidar_active scan_active hz:=10 lasers:=40 samples:=400 min_range:=0.2 max_range:=100.0 noise:=0.01 min_angle:=-1.5707963 max_angle:=1.5707963">
     <joint name="${prefix}_base_mount_joint" type="fixed">
       <xacro:insert_block name="origin" />

Commit message: more accurate sensors

File: eufs_racecar/urdf/VLP-32C.urdf.xacro (robot description, xacro)
@@ -2,5 +2,5 @@
 <robot name="VLP-32C_LiDAR" xmlns:xacro="http://www.ros.org/wiki/xacro">
   <xacro:property name="M_PI" value="3.1415926535897931" />
-  <xacro:macro name="VLP-32C_LiDAR" params="*origin parent prefix lidar_active scan_active hz:=10 lasers:=40 samples:=400 min_range:=0.2 max_range:=100.0 noise:=0.01 min_angle:=-1.5707963 max_angle:=1.5707963">
+  <xacro:macro name="VLP-32C_LiDAR" params="*origin parent prefix lidar_active scan_active hz:=10 lasers:=32 samples:=400 min_range:=0.2 max_range:=100.0 noise:=0.01 min_angle:=-1.5707963 max_angle:=1.5707963">
     <joint name="${prefix}_base_mount_joint" type="fixed">
       <xacro:insert_block name="origin" />
