Commit message: Fix base_footprint

File: eufs_racecar/robots/eufs/robot.urdf.xacro (robot description, xacro)
@@ -40,14 +40,14 @@
     LIDAR: 1.700 0.0 -0.150
     STEREO CAM: -0.110 0.0 0.800 -->
-    <xacro:sensor_imu parent="base_footprint" prefix="imu">
+    <xacro:sensor_imu parent="chassis" prefix="imu">
         <origin xyz="0.0 0.0 0.0" rpy="0 0 0"/>
     </xacro:sensor_imu>
-    <xacro:sensor_gps parent="base_footprint" prefix="gps">
+    <xacro:sensor_gps parent="chassis" prefix="gps">
         <origin xyz="0.0 0.0 0.4" rpy="0 0 0"/>
     </xacro:sensor_gps>
-    <xacro:VLP-16R parent="base_footprint" name="velodyne" topic="/velodyne_points" hz="10" active="$(arg simulate_perception)">
+    <xacro:VLP-16R parent="chassis" name="velodyne" topic="/velodyne_points" hz="10" active="$(arg simulate_perception)">
         <origin xyz="-0.15 0.0 0.79" rpy="0 ${1*M_PI/180.0} 0"/>
     </xacro:VLP-16R>
-    <xacro:zed_camera parent="base_footprint" prefix="zed" active="$(arg simulate_perception)">
+    <xacro:zed_camera parent="chassis" prefix="zed" active="$(arg simulate_perception)">
         <origin xyz="-0.08 0.0 0.76" rpy="0 0 0"/>
     </xacro:zed_camera>

File: eufs_racecar/urdf/eufs_base.urdf.xacro (robot description, xacro)
@@ -2,4 +2,5 @@
 <robot name="eufs" xmlns:xacro="http://www.ros.org/wiki/xacro">
   <xacro:macro name="eufs_base" params="chassis_mesh">
+    <xacro:property name="wheel_diameter" value="0.505"/>
     <!-- BASE FOOTPRINT -->
     <link name="base_footprint"/>
@@ -7,5 +8,5 @@
       <parent link="base_footprint"/>
       <child link="chassis"/>
-      <origin xyz="0 0 0"
+      <origin xyz="0 0 ${wheel_diameter/2}"
               rpy="0 0 0"/>
       <axis xyz="1 0 0"/>

File: eufs_racecar/urdf/wheels.urdf.xacro (robot description, xacro)
@@ -56,5 +56,5 @@
     <!-- Front and rear wheel descriptions -->
     <!-- ********************************* -->
-    <!-- Description of how a front wheel is connected to the base_footprint -->
+    <!-- Description of how a front wheel is connected to the chassis -->
     <xacro:macro name="front_wheel"
                  params="lr_prefix lr_reflect">
@@ -64,5 +64,5 @@
                      0"
                 rpy="0 0 0"/>
-        <parent link="base_footprint"/>
+        <parent link="chassis"/>
         <child link="${lr_prefix}_steering_hinge"/>
         <axis xyz="0 0 1"/>
@@ -92,5 +92,5 @@
       <xacro:wheel lr_prefix="${lr_prefix}" fr_prefix="front"/>
     </xacro:macro>
-    <!-- Description of how a rear wheel is connected to the base_footprint -->
+    <!-- Description of how a rear wheel is connected to the chassis -->
     <xacro:macro name="rear_wheel"
                  params="lr_prefix lr_reflect">
@@ -100,5 +100,5 @@
                      0"
                 rpy="0 0 0"/>
-        <parent link="base_footprint"/>
+        <parent link="chassis"/>
         <child link="${lr_prefix}_rear_wheel"/>
         <axis xyz="0 1 0"/>

Commit message: Updated config kinematics values

File: eufs_racecar/robots/eufs/robot.urdf.xacro (robot description, xacro)
@@ -35,23 +35,28 @@
     <!--                 MAIN SENSORS                    -->
     <!-- *********************************************** -->
-    <!--     LOCATIONS: (XYZ)
+    <!--     LOCATIONS: (XYZ) - original values
     IMU: 0.0 0.0 0.170
     GPS: -0.110 0.0 0.9
     LIDAR: 1.700 0.0 -0.150
     STEREO CAM: -0.110 0.0 0.800 -->
+    <!--     LOCATIONS: (XYZ) - new values measured on 24/01/23
+    IMU: 0.0 0.0 0.0
+    GPS: 1.220 0.0 0.530
+    LIDAR: 1.590 0.0 0.130
+    STEREO CAM: 0.370 0.0 0.900 -->
     <xacro:sensor_imu parent="chassis" prefix="sbg_imu" topic_prefix="">
         <origin xyz="0.0 0.0 0.0" rpy="0 0 0"/>
     </xacro:sensor_imu>
     <xacro:sensor_gps parent="chassis" prefix="gps">
-        <origin xyz="0.0 0.0 0.4" rpy="0 0 0"/>
+        <origin xyz="1.220 0.0 0.530" rpy="0 0 0"/>
     </xacro:sensor_gps>
     <xacro:VLP-16R parent="chassis" name="velodyne" topic="/velodyne_points" hz="10" active="$(arg simulate_perception)">
-        <origin xyz="-0.15 0.0 0.79" rpy="0 ${1*M_PI/180.0} 0"/>
+        <origin xyz="1.590 0.0 0.130" rpy="0 ${1*M_PI/180.0} 0"/>
     </xacro:VLP-16R>
     <xacro:zed_camera parent="chassis" prefix="zed" active="$(arg simulate_perception)">
-        <origin xyz="-0.08 0.0 0.76" rpy="0 0 0"/>
+        <origin xyz="0.0 0.0 0.0" rpy="0 0 0"/>
     </xacro:zed_camera>
     <xacro:sensor_imu parent="chassis" prefix="zed_imu" topic_prefix="/camera">
-        <origin xyz="-0.08 0.0 0.76" rpy="0 0 0"/>
+        <origin xyz="0.0 0.0 0.0" rpy="0 0 0"/>
     </xacro:sensor_imu>
 </robot>

Commit message: Updated location of sensors

File: eufs_racecar/robots/eufs/robot.urdf.xacro (robot description, xacro)
@@ -55,5 +55,5 @@
     </xacro:VLP-16R>
     <xacro:zed_camera parent="chassis" prefix="zed" active="$(arg simulate_perception)">
-        <origin xyz="0.0 0.0 0.0" rpy="0 0 0"/>
+        <origin xyz="0.370 0.0 0.900" rpy="0 0 0"/>
     </xacro:zed_camera>
     <xacro:sensor_imu parent="chassis" prefix="zed_imu" topic_prefix="/camera">

Commit message: velodyne positioning and sensor param adjustments

File: eufs_racecar/robots/eufs/robot.urdf.xacro (robot description, xacro)
@@ -52,5 +52,5 @@
     </xacro:sensor_gps>
     <xacro:VLP-16R parent="chassis" name="velodyne" topic="/velodyne_points" hz="10" active="$(arg simulate_perception)">
-        <origin xyz="1.590 0.0 0.130" rpy="0 ${1*M_PI/180.0} 0"/>
+        <origin xyz="1.590 0.0 -0.15" rpy="0 0 0"/>
     </xacro:VLP-16R>
     <xacro:zed_camera parent="chassis" prefix="zed" active="$(arg simulate_perception)">

File: eufs_sensors/urdf/VLP-32C.urdf.xacro (robot description, xacro)
@@ -2,5 +2,5 @@
 <robot xmlns:xacro="http://www.ros.org/wiki/xacro" name="VLP-16">
   <xacro:property name="M_PI" value="3.1415926535897931" />
-  <xacro:macro name="VLP-16R" params="*origin parent:=base_footprint name:=velodyne active topic:=/velodyne_points hz:=100 lasers:=32 samples:=350 min_range:=0.2 max_range:=200.0 noise:=0.008 min_angle:=-1.5707963 max_angle:=1.5707963">
+  <xacro:macro name="VLP-16R" params="*origin parent:=base_footprint name:=velodyne active topic:=/velodyne_points hz:=10 lasers:=40 samples:=600 min_range:=0.2 max_range:=200.0 noise:=0.01 min_angle:=-1.5707963 max_angle:=1.5707963">
     <joint name="${name}_base_mount_joint" type="fixed">
       <xacro:insert_block name="origin" />
@@ -71,5 +71,5 @@
                 <samples>${lasers}</samples>
                 <resolution>1.0</resolution>
-                <min_angle>-${15.0*M_PI/180.0}</min_angle>
+                <min_angle>-${10.0*M_PI/180.0}</min_angle>
                 <max_angle> ${15.0*M_PI/180.0}</max_angle>
               </vertical>

Commit message: Updated camera location

File: eufs_racecar/robots/eufs/robot.urdf.xacro (robot description, xacro)
@@ -44,5 +44,5 @@
     GPS: 1.220 0.0 0.530
     LIDAR: 1.590 0.0 0.130
-    STEREO CAM: 0.370 0.0 0.900 -->
+    STEREO CAM: -0.370 0.0 0.900 -->
     <xacro:sensor_imu parent="chassis" prefix="sbg_imu" topic_prefix="">
         <origin xyz="0.0 0.0 0.0" rpy="0 0 0"/>
@@ -55,5 +55,5 @@
     </xacro:VLP-16R>
     <xacro:zed_camera parent="chassis" prefix="zed" active="$(arg simulate_perception)">
-        <origin xyz="0.370 0.0 0.900" rpy="0 0 0"/>
+        <origin xyz="-0.370 0.0 0.900" rpy="0 0 0"/>
     </xacro:zed_camera>
     <xacro:sensor_imu parent="chassis" prefix="zed_imu" topic_prefix="/camera">

Commit message: Changed robot name to qev3

File: eufs_racecar/robots/eufs/robot.urdf.xacro (robot description, xacro)
@@ -14,8 +14,4 @@
     <!-- If the perception stack should be simulated or if sensors should be used -->
     <xacro:arg name="simulate_perception" default="true"/>
-    <!-- If the camera should be simulated or if sensors should be removed -->
-    <xacro:arg name="simulate_camera" default="true"/>
-    <!-- If the lidar should be simulated or if sensors should be removed -->
-    <xacro:arg name="simulate_lidar" default="false"/>
     <!-- ***************** -->
     <!-- Imported elements -->
@@ -33,5 +29,5 @@
     <!-- *************** -->
     <!-- Chassis of the car -->
-    <xacro:eufs_base chassis_mesh="file://$(find eufs_racecar)/meshes/lando.dae"/>
+    <xacro:eufs_base chassis_mesh="file://$(find eufs_racecar)/meshes/sisu-20d.dae"/>
     <!-- Wheels -->
     <xacro:wheels chassis_width="1.6" wheelbase="1.580"/>
@@ -39,29 +35,23 @@
     <!--                 MAIN SENSORS                    -->
     <!-- *********************************************** -->
-    <!--     LOCATIONS: (XYZ) - original values
+    <!--     LOCATIONS: (XYZ)
     IMU: 0.0 0.0 0.170
     GPS: -0.110 0.0 0.9
     LIDAR: 1.700 0.0 -0.150
     STEREO CAM: -0.110 0.0 0.800 -->
-    <!--     LOCATIONS: (XYZ) - new values measured on 24/01/23
-    IMU: 0.0 0.0 0.0
-    GPS: 1.220 0.0 0.530
-    LIDAR: 1.590 0.0 0.130
-    STEREO CAM: -0.370 0.0 0.900 -->
     <xacro:sensor_imu parent="chassis" prefix="sbg_imu" topic_prefix="">
         <origin xyz="0.0 0.0 0.0" rpy="0 0 0"/>
     </xacro:sensor_imu>
     <xacro:sensor_gps parent="chassis" prefix="gps">
-        <origin xyz="1.220 0.0 0.530" rpy="0 0 0"/>
+        <origin xyz="0.0 0.0 0.4" rpy="0 0 0"/>
     </xacro:sensor_gps>
-<!--  <xacro:VLP-16R parent="chassis" name="velodyne" topic="/velodyne_points" hz="10" active= $(arg simulate_perception) -->
-    <xacro:VLP-16R parent="chassis" name="velodyne" topic="/velodyne_points" hz="10" active="$(arg simulate_lidar)">
-        <origin xyz="1.590 0.0 -0.15" rpy="0 0 0"/>
+    <xacro:VLP-16R parent="chassis" name="velodyne" topic="/velodyne_points" hz="10" active="$(arg simulate_perception)">
+        <origin xyz="-0.15 0.0 0.79" rpy="0 ${1*M_PI/180.0} 0"/>
     </xacro:VLP-16R>
-    <xacro:zed_camera parent="chassis" prefix="zed" active="$(arg simulate_camera)">
-        <origin xyz="-0.370 0.0 0.900" rpy="0 0 0"/>
+    <xacro:zed_camera parent="chassis" prefix="zed" active="$(arg simulate_perception)">
+        <origin xyz="-0.08 0.0 0.76" rpy="0 0 0"/>
     </xacro:zed_camera>
     <xacro:sensor_imu parent="chassis" prefix="zed_imu" topic_prefix="/camera">
-        <origin xyz="0.0 0.0 0.0" rpy="0 0 0"/>
+        <origin xyz="-0.08 0.0 0.76" rpy="0 0 0"/>
     </xacro:sensor_imu>
 </robot>

File: eufs_racecar/robots/qev3/robot.urdf.xacro (robot description, xacro)
@@ -1,4 +1,4 @@
 <?xml version="1.0"?>
-<robot name="eufs" xmlns:xacro="http://www.ros.org/wiki/xacro">
+<robot name="qev3" xmlns:xacro="http://www.ros.org/wiki/xacro">
     <!-- ***************** -->
     <!-- Config parameters -->
@@ -14,4 +14,8 @@
     <!-- If the perception stack should be simulated or if sensors should be used -->
     <xacro:arg name="simulate_perception" default="true"/>
+    <!-- If the camera should be simulated or if sensors should be removed -->
+    <xacro:arg name="simulate_camera" default="true"/>
+    <!-- If the lidar should be simulated or if sensors should be removed -->
+    <xacro:arg name="simulate_lidar" default="false"/>
     <!-- ***************** -->
     <!-- Imported elements -->
@@ -29,5 +33,5 @@
     <!-- *************** -->
     <!-- Chassis of the car -->
-    <xacro:eufs_base chassis_mesh="file://$(find eufs_racecar)/meshes/sisu-20d.dae"/>
+    <xacro:eufs_base chassis_mesh="file://$(find eufs_racecar)/meshes/lando.dae"/>
     <!-- Wheels -->
     <xacro:wheels chassis_width="1.6" wheelbase="1.580"/>
@@ -35,23 +39,29 @@
     <!--                 MAIN SENSORS                    -->
     <!-- *********************************************** -->
-    <!--     LOCATIONS: (XYZ)
+    <!--     LOCATIONS: (XYZ) - original values
     IMU: 0.0 0.0 0.170
     GPS: -0.110 0.0 0.9
     LIDAR: 1.700 0.0 -0.150
     STEREO CAM: -0.110 0.0 0.800 -->
+    <!--     LOCATIONS: (XYZ) - new values measured on 24/01/23
+    IMU: 0.0 0.0 0.0
+    GPS: 1.220 0.0 0.530
+    LIDAR: 1.590 0.0 0.130
+    STEREO CAM: -0.370 0.0 0.900 -->
     <xacro:sensor_imu parent="chassis" prefix="sbg_imu" topic_prefix="">
         <origin xyz="0.0 0.0 0.0" rpy="0 0 0"/>
     </xacro:sensor_imu>
     <xacro:sensor_gps parent="chassis" prefix="gps">
-        <origin xyz="0.0 0.0 0.4" rpy="0 0 0"/>
+        <origin xyz="1.220 0.0 0.530" rpy="0 0 0"/>
     </xacro:sensor_gps>
-    <xacro:VLP-16R parent="chassis" name="velodyne" topic="/velodyne_points" hz="10" active="$(arg simulate_perception)">
-        <origin xyz="-0.15 0.0 0.79" rpy="0 ${1*M_PI/180.0} 0"/>
+<!--  <xacro:VLP-16R parent="chassis" name="velodyne" topic="/velodyne_points" hz="10" active= $(arg simulate_perception) -->
+    <xacro:VLP-16R parent="chassis" name="velodyne" topic="/velodyne_points" hz="10" active="$(arg simulate_lidar)">
+        <origin xyz="1.590 0.0 -0.15" rpy="0 0 0"/>
     </xacro:VLP-16R>
-    <xacro:zed_camera parent="chassis" prefix="zed" active="$(arg simulate_perception)">
-        <origin xyz="-0.08 0.0 0.76" rpy="0 0 0"/>
+    <xacro:zed_camera parent="chassis" prefix="zed" active="$(arg simulate_camera)">
+        <origin xyz="-0.370 0.0 0.900" rpy="0 0 0"/>
     </xacro:zed_camera>
     <xacro:sensor_imu parent="chassis" prefix="zed_imu" topic_prefix="/camera">
-        <origin xyz="-0.08 0.0 0.76" rpy="0 0 0"/>
+        <origin xyz="0.0 0.0 0.0" rpy="0 0 0"/>
     </xacro:sensor_imu>
 </robot>
