Commit message: fix eufs_sensor files, change eufs_racecar robots folder to racecars

File: eufs_racecar/racecars/qev3/robot.urdf.xacro (robot description, xacro)
@@ -6,12 +6,12 @@
     <!--  Load the config file  -->
     <xacro:property name="config" value="${load_yaml('$(arg config_file)')}"/>
+    <!-- If the camera should be simulated or if sensors should be removed -->
+    <xacro:arg name="simulate_camera" default="true"/>
+    <!-- If the lidar should be simulated or if sensors should be removed -->
+    <xacro:arg name="simulate_lidar" default="false"/>
     <!-- ***************** -->
     <!-- Global parameters -->
     <!-- ***************** -->
     <xacro:property name="PI" value="3.1415926535897931"/>
-    <!-- If the camera should be simulated or if sensors should be removed -->
-    <xacro:arg name="simulate_camera" default="true"/>
-    <!-- If the lidar should be simulated or if sensors should be removed -->
-    <xacro:arg name="simulate_lidar" default="false"/>
     <!-- ***************** -->
     <!-- Imported elements -->
@@ -20,5 +20,5 @@
     <xacro:include filename="$(find eufs_racecar)/urdf/wheels.urdf.xacro"/>
     <!-- Import EUFS base element with the chassis -->
-    <xacro:include filename="$(find eufs_racecar)/urdf/eufs_base.urdf.xacro" />
+    <xacro:include filename="$(find eufs_racecar)/urdf/chassis_base.urdf.xacro" />
     <!-- Import all available sensors -->
     <!-- GPS -->
@@ -36,5 +36,5 @@
     <!-- *************** -->
     <!-- Chassis of the car -->
-    <xacro:eufs_base chassis_mesh="file://$(find eufs_racecar)/meshes/lando.dae"/>
+    <xacro:chassis_base chassis_mesh="file://$(find eufs_racecar)/meshes/lando.dae"/>
     <!-- Wheels -->
     <xacro:wheels chassis_width="1.6" wheelbase="1.580"/>

File: eufs_racecar/urdf/SBG_GPS.urdf.xacro (robot description, xacro)
@@ -33,5 +33,5 @@
 <!--            </material>-->
 <!--            <geometry>-->
-<!--                <mesh filename="file://$(find eufs_sensors)/meshes/antenna_3GO16.stl" scale="1.0 1.0 1.0"/>-->
+<!--                <mesh filename="file://$(find eufs_racecar)/meshes/antenna_3GO16.stl" scale="1.0 1.0 1.0"/>-->
 <!--            </geometry>-->
 <!--        </visual>-->
@@ -39,5 +39,5 @@
 <!--            <origin rpy="0 0 0" xyz="0 0 0"/>-->
 <!--            <geometry>-->
-<!--                <mesh filename="file://$(find eufs_sensors)/meshes/antenna_3GO16.stl" scale="1.0 1.0 1.0"/>-->
+<!--                <mesh filename="file://$(find eufs_racecar)/meshes/antenna_3GO16.stl" scale="1.0 1.0 1.0"/>-->
 <!--            </geometry>-->
 <!--        </collision>-->

File: eufs_racecar/urdf/VLP-32C.urdf.xacro (robot description, xacro)
@@ -18,10 +18,10 @@
       <visual>
         <geometry>
-          <mesh filename="file://$(find eufs_sensors)/meshes/VLP16_base_1.dae" />
+          <mesh filename="file://$(find eufs_racecar)/meshes/VLP16_base_1.dae" />
         </geometry>
       </visual>
       <visual>
         <geometry>
-          <mesh filename="file://$(find eufs_sensors)/meshes/VLP16_base_2.dae" />
+          <mesh filename="file://$(find eufs_racecar)/meshes/VLP16_base_2.dae" />
         </geometry>
       </visual>
@@ -47,5 +47,5 @@
         <origin xyz="0 0 -0.0377" />
         <geometry>
-          <mesh filename="file://$(find eufs_sensors)/meshes/VLP16_scan.dae" />
+          <mesh filename="file://$(find eufs_racecar)/meshes/VLP16_scan.dae" />
         </geometry>
       </visual>

File: eufs_racecar/urdf/ZED2i.urdf.xacro (robot description, xacro)
@@ -13,5 +13,5 @@
         <origin xyz="0 0 0" rpy="0 0 0"/>
         <geometry>
-          <mesh filename="file://$(find eufs_sensors)/meshes/zed.dae" />
+          <mesh filename="file://$(find eufs_racecar)/meshes/zed.dae" />
         </geometry>
         <material name="light_grey">

File: eufs_racecar/urdf/chassis_base.urdf.xacro (robot description, xacro)
@@ -1,5 +1,5 @@
 <?xml version="1.0"?>
-<robot name="eufs" xmlns:xacro="http://www.ros.org/wiki/xacro">
-  <xacro:macro name="eufs_base" params="chassis_mesh">
+<robot name="chassis_base" xmlns:xacro="http://www.ros.org/wiki/xacro">
+  <xacro:macro name="chassis_base" params="chassis_mesh">
     <xacro:property name="wheel_diameter" value="0.505"/>
     <!-- BASE FOOTPRINT -->
