Commit message: plugin consolidation. naming better, remove overhead

File: eufs_plugins/urdf/eufs_plugins.gazebo.xacro (robot description, xacro)
@@ -44,5 +44,5 @@
       <lidarYViewDistance>15</lidarYViewDistance>
       <lidarMinViewDistance>1</lidarMinViewDistance>
-      <cameraFOV>2.09</cameraFOV><!--120 degrees-->
+      <cameraFOV>1.91986</cameraFOV><!--110 degrees-->
       <cameraMinViewDistance>0.5</cameraMinViewDistance>
       <lidarFOV>3.141593</lidarFOV><!-- 180 degrees-->

File: eufs_racecar/robots/qev3/robot.urdf.xacro (robot description, xacro)
@@ -10,8 +10,4 @@
     <!-- ***************** -->
     <xacro:property name="PI" value="3.1415926535897931"/>
-    <!-- If the gazebo_ros_race_car_model should publish the ground truth tf -->
-    <xacro:arg name="publish_tf" default="false"/>
-    <!-- If the perception stack should be simulated or if sensors should be used -->
-    <xacro:arg name="simulate_perception" default="true"/>
     <!-- If the camera should be simulated or if sensors should be removed -->
     <xacro:arg name="simulate_camera" default="true"/>
@@ -25,8 +21,15 @@
     <!-- Import EUFS base element with the chassis -->
     <xacro:include filename="$(find eufs_racecar)/urdf/eufs_base.urdf.xacro" />
-    <!-- Import all available sensors -->
-    <xacro:include filename="$(find eufs_sensors)/urdf/all_sensors.urdf.xacro" />
     <!--  Include the plugins  -->
     <xacro:include filename="$(find eufs_plugins)/urdf/eufs_plugins.gazebo.xacro" />
+    <!-- Import all available sensors -->
+    <!-- GPS -->
+    <xacro:include filename="$(find eufs_sensors)/urdf/SBG_GPS.urdf.xacro"/>
+    <!--IMU -->
+    <xacro:include filename="$(find eufs_sensors)/urdf/SBG_IMU.urdf.xacro"/>
+    <!-- Velodyne VLP-32C -->
+    <xacro:include filename="$(find eufs_sensors)/urdf/VLP-32C.urdf.xacro"/>
+    <!-- ZED Stereo camera -->
+    <xacro:include filename="$(find eufs_sensors)/urdf/ZED2i.urdf.xacro"/>
     <!-- *************** -->
     <!-- Robots Elements -->
@@ -49,18 +52,15 @@
     LIDAR: 1.590 0.0 0.130
     STEREO CAM: -0.370 0.0 0.900 -->
-    <xacro:sensor_imu parent="chassis" prefix="sbg_imu" topic_prefix="">
+    <xacro:SBG_IMU_sensor parent="chassis" prefix="imu">
         <origin xyz="0.0 0.0 0.0" rpy="0 0 0"/>
-    </xacro:sensor_imu>
-    <xacro:sensor_gps parent="chassis" prefix="gps">
+    </xacro:SBG_IMU_sensor>
+    <xacro:SBG_GPS_sensor parent="chassis" prefix="sbg">
         <origin xyz="1.220 0.0 0.530" rpy="0 0 0"/>
-    </xacro:sensor_gps>
-    <xacro:VLP-32C parent="chassis" name="velodyne" topic="/velodyne_points" hz="10" active="$(arg simulate_lidar)">
+    </xacro:SBG_GPS_sensor>
+    <xacro:VLP-32C_LiDAR parent="chassis" prefix="velodyne" hz="10" active="$(arg simulate_lidar)">
         <origin xyz="1.590 0.0 -0.15" rpy="0 0 0"/>
-    </xacro:VLP-32C>
-    <xacro:zed_camera parent="chassis" prefix="zed" active="$(arg simulate_camera)">
+    </xacro:VLP-32C_LiDAR>
+    <xacro:ZED2i_camera parent="chassis" prefix="zed2i" active="$(arg simulate_camera)">
         <origin xyz="-0.370 0.0 0.900" rpy="0 0 0"/>
-    </xacro:zed_camera>
-    <!-- <xacro:sensor_imu parent="chassis" prefix="zed_imu" topic_prefix="/camera"> -->
-        <!-- <origin xyz="0.0 0.0 0.0" rpy="0 0 0"/> -->
-    <!-- </xacro:sensor_imu> -->
+    </xacro:ZED2i_camera>
 </robot>

File: eufs_sensors/urdf/SBG_GPS.urdf.xacro (robot description, xacro)
@@ -1,5 +1,5 @@
 <?xml version="1.0"?>
-<robot name="sensor_gps" xmlns:xacro="http://www.ros.org/wiki/xacro">
-    <xacro:macro name="sensor_gps" params="prefix parent *origin">
+<robot name="SBG_GPS_sensor" xmlns:xacro="http://www.ros.org/wiki/xacro">
+    <xacro:macro name="SBG_GPS_sensor" params="prefix parent *origin">
         <!-- ANTENNA GPS -->
         <joint name="${prefix}_joint" type="fixed">
@@ -81,9 +81,8 @@
                     </velocity_sensing>
                 </gps>
-                <plugin name="${prefix}_controller" filename="libgazebo_ros_gps_sensor.so">
+                <plugin name="gps_controller" filename="libgazebo_ros_gps_sensor.so">
                     <ros>
-                        <!--remapping gps to nav_sat for QEV3 imu -->
-                        <!-- <remapping>~/out:=${prefix}</remapping> (original code) -->
                         <remapping>~/out:=/imu/nav_sat_fix</remapping>
+                        <remapping>~/vel:=/imu/gps_vel</remapping>
                     </ros>
                     <frame_name>${prefix}_base_link</frame_name>

File: eufs_sensors/urdf/SBG_IMU.urdf.xacro (robot description, xacro)
@@ -1,5 +1,5 @@
 <?xml version="1.0"?>
-<robot name="sensor_imu" xmlns:xacro="http://www.ros.org/wiki/xacro">
-    <xacro:macro name="sensor_imu" params="prefix parent topic_prefix *origin noise:=0.08">
+<robot name="SBG_IMU_sensor" xmlns:xacro="http://www.ros.org/wiki/xacro">
+    <xacro:macro name="SBG_IMU_sensor" params="prefix parent *origin noise:=0.08">
         <joint name="${prefix}_base_joint" type="fixed">
             <axis xyz="1 0 0"/>
@@ -78,5 +78,5 @@
                 <plugin filename="libgazebo_ros_imu_sensor.so" name="${prefix}">
                     <ros>
-                        <remapping>~/out:=${topic_prefix}/imu/data</remapping>
+                        <remapping>~/out:=/imu/data</remapping>
                     </ros>
                     <frame_name>${prefix}_base_link</frame_name>

File: eufs_sensors/urdf/VLP-32C.urdf.xacro (robot description, xacro)
@@ -1,12 +1,12 @@
 <?xml version="1.0"?>
-<robot xmlns:xacro="http://www.ros.org/wiki/xacro" name="VLP-32">
+<robot name="VLP-32C_LiDAR" xmlns:xacro="http://www.ros.org/wiki/xacro">
   <xacro:property name="M_PI" value="3.1415926535897931" />
-  <xacro:macro name="VLP-32C" params="*origin parent:=base_footprint name:=velodyne active topic:=/velodyne_points hz:=10 lasers:=40 samples:=600 min_range:=0.2 max_range:=200.0 noise:=0.01 min_angle:=-1.5707963 max_angle:=1.5707963">
-    <joint name="${name}_base_mount_joint" type="fixed">
+  <xacro:macro name="VLP-32C_LiDAR" params="*origin parent prefix active hz:=10 lasers:=40 samples:=600 min_range:=0.2 max_range:=200.0 noise:=0.01 min_angle:=-1.5707963 max_angle:=1.5707963">
+    <joint name="${prefix}_base_mount_joint" type="fixed">
       <xacro:insert_block name="origin" />
       <parent link="${parent}"/>
-      <child link="${name}_base_link"/>
+      <child link="${prefix}_base_link"/>
     </joint>
-    <link name="${name}_base_link">
+    <link name="${prefix}_base_link">
       <inertial>
         <mass value="0.83"/>
@@ -33,10 +33,10 @@
       </collision>
     </link>
-    <joint name="${name}_base_scan_joint" type="fixed" >
+    <joint name="${prefix}_base_scan_joint" type="fixed" >
       <origin xyz="0 0 0.0377" rpy="0 0 0" />
-      <parent link="${name}_base_link" />
-      <child link="${name}"/>
+      <parent link="${prefix}_base_link" />
+      <child link="${prefix}"/>
     </joint>
-    <link name="${name}">
+    <link name="${prefix}">
       <inertial>
         <mass value="0.01"/>
@@ -54,6 +54,6 @@
     <xacro:unless value="${active}">
       <!-- Gazebo requires the velodyne_gazebo_plugins package -->
-      <gazebo reference="${name}">
-        <sensor type="ray" name="${name}-VLP16">
+      <gazebo reference="${prefix}">
+        <sensor type="ray" name="${prefix}-VLP16">
           <always_on>true</always_on>
           <pose>0 0 0 0 0 0</pose>
@@ -88,7 +88,7 @@
           <plugin name="gazebo_ros_laser_controller" filename="libgazebo_ros_ray_sensor.so">
             <ros>
-              <remapping>~/out:=${topic}</remapping>
+              <remapping>~/out:=/velodyne_points</remapping>
             </ros>
-            <frame_name>${name}</frame_name>
+            <frame_name>${prefix}</frame_name>
             <radiation_type>infrared</radiation_type>
             <output_type>sensor_msgs/PointCloud2</output_type>

File: eufs_sensors/urdf/ZED2i.urdf.xacro (robot description, xacro)
@@ -1,6 +1,6 @@
 <?xml version="1.0"?>
-<robot name="zed_camera"
+<robot name="ZED2i_camera"
   xmlns:xacro="http://www.ros.org/wiki/xacro">
-  <xacro:macro name="zed_camera" params="prefix parent *origin active">
+  <xacro:macro name="ZED2i_camera" params="prefix parent *origin active">
     <joint name="${prefix}_base_joint" type="fixed">
       <axis xyz="1 0 0"/>
@@ -55,6 +55,5 @@
     <xacro:unless value="${active}">
       <gazebo reference="${prefix}_left_camera_optical_frame">
-        <sensor type="multicamera" name="stereo_camera">
-          <!-- see MultiSenseSLPlugin.h for available modes -->
+        <!-- <sensor type="multicamera" name="stereo_camera">
           <always_on>true</always_on>
           <update_rate>60.0</update_rate>
@@ -109,5 +108,5 @@
             <triggered>false</triggered>
           </plugin>
-        </sensor>
+        </sensor> -->
         <!-- Depth simulation -->
         <sensor name="stereo_depth" type="depth">
@@ -126,17 +125,20 @@
             <clip>
               <near>0.5</near>
-              <far>20.0</far>
+              <far>15.0</far>
             </clip>
           </camera>
-          <plugin name="${prefix}_controller" filename="libgazebo_ros_camera.so">
+          <plugin name="zed_controller" filename="libgazebo_ros_camera.so">
             <ros>
-              <parameter name="update_rate" type="double">30.0</parameter>
-              <remapping>/zed/depth/camera_info:=/zed2i/zed_node/depth/camera_info</remapping>
-              <remapping>/zed/depth/image_raw:=/zed2i/zed_node/depth/depth_registered</remapping>
+              <!-- <parameter name="update_rate" type="double">30.0</parameter> -->
+              <remapping>/zed2i/depth/camera_info:=/zed2i/zed_node/depth/camera_info</remapping>
+              <remapping>/zed2i/depth/image_raw:=/zed2i/zed_node/depth/depth_registered</remapping>
+              <remapping>/zed2i/image_raw:=/zed2i/zed_node/rgb/image_rect_color</remapping>
+              <remapping>/zed2i/camera_info:=/zed2i/zed_node/rgb/camera_info</remapping>
+              <remapping>/zed2i/points:=/zed2i/zed_node/point_cloud/cloud_registered</remapping>
             </ros>
             <camera_name>${prefix}</camera_name>
             <frame_name>${prefix}_depth_camera_frame</frame_name>
             <hack_baseline>0.120</hack_baseline>
-            <max_depth>20.0</max_depth>
+            <max_depth>15.0</max_depth>
             <min_depth>0.1</min_depth>
           </plugin>

Commit message: split sim slam and laser scanner into options. nearly broke the sim a few times lol i hate these launch files

File: eufs_plugins/urdf/eufs_plugins.gazebo.xacro (robot description, xacro)
@@ -2,5 +2,6 @@
 <robot xmlns:xacro="http://www.ros.org/wiki/xacro">
   <xacro:arg name="publish_tf" default="false"/>
-  <xacro:arg name="simulate_perception" default="false"/>
+  <xacro:arg name="sim_perception" default="true"/>
+  <xacro:arg name="sim_slam" default="true"/>
   <xacro:arg name="command_mode" default="velocity"/>
   <xacro:arg name="pub_ground_truth" default="true"/>
@@ -61,6 +62,6 @@
       <SLAMLocalRangeY>10</SLAMLocalRangeY>
       <publishGroundTruth>$(arg pub_ground_truth)</publishGroundTruth>
-      <simulatePerception>$(arg simulate_perception)</simulatePerception>
-      <simulateSLAM>$(arg simulate_perception)</simulateSLAM>
+      <simulatePerception>$(arg sim_perception)</simulatePerception>
+      <simulateSLAM>$(arg sim_slam)</simulateSLAM>
     </plugin>
   </gazebo>

File: eufs_racecar/racecars/qev3/robot.urdf.xacro (robot description, xacro)
@@ -6,8 +6,8 @@
     <!--  Load the config file  -->
     <xacro:property name="config" value="${load_yaml('$(arg config_file)')}"/>
-    <!-- If the camera should be simulated or if sensors should be removed -->
-    <xacro:arg name="simulate_camera" default="true"/>
-    <!-- If the lidar should be simulated or if sensors should be removed -->
-    <xacro:arg name="simulate_lidar" default="false"/>
+    <!-- Simulate sensors or not? -->
+    <xacro:arg name="enable_camera" default="false"/>
+    <xacro:arg name="enable_lidar" default="false"/>
+    <xacro:arg name="enable_laserscan" default="false"/>
     <!-- ***************** -->
     <!-- Global parameters -->
@@ -58,8 +58,8 @@
         <origin xyz="1.220 0.0 0.530" rpy="0 0 0"/>
     </xacro:SBG_GPS_sensor>
-    <xacro:VLP-32C_LiDAR parent="chassis" prefix="velodyne" hz="10" active="$(arg simulate_lidar)">
+    <xacro:VLP-32C_LiDAR parent="chassis" prefix="velodyne" hz="10" lidar_active="$(arg enable_lidar)" scan_active="$(arg enable_laserscan)">
         <origin xyz="1.590 0.0 -0.15" rpy="0 0 0"/>
     </xacro:VLP-32C_LiDAR>
-    <xacro:ZED2i_camera parent="chassis" prefix="zed2i" active="$(arg simulate_camera)">
+    <xacro:ZED2i_camera parent="chassis" prefix="zed2i" active="$(arg enable_camera)">
         <origin xyz="-0.370 0.0 0.900" rpy="0 0 0"/>
     </xacro:ZED2i_camera>

File: eufs_racecar/urdf/VLP-32C.urdf.xacro (robot description, xacro)
@@ -2,5 +2,5 @@
 <robot name="VLP-32C_LiDAR" xmlns:xacro="http://www.ros.org/wiki/xacro">
   <xacro:property name="M_PI" value="3.1415926535897931" />
-  <xacro:macro name="VLP-32C_LiDAR" params="*origin parent prefix active hz:=10 lasers:=40 samples:=600 min_range:=0.2 max_range:=200.0 noise:=0.01 min_angle:=-1.5707963 max_angle:=1.5707963">
+  <xacro:macro name="VLP-32C_LiDAR" params="*origin parent prefix lidar_active scan_active hz:=10 lasers:=40 samples:=600 min_range:=0.2 max_range:=200.0 noise:=0.01 min_angle:=-1.5707963 max_angle:=1.5707963">
     <joint name="${prefix}_base_mount_joint" type="fixed">
       <xacro:insert_block name="origin" />
@@ -51,8 +51,7 @@
       </visual>
     </link>
-    <!-- Simulate raw perception sensors only if we're not using the abstracted perception simulation -->
-    <xacro:unless value="${active}">
-      <!-- Gazebo requires the velodyne_gazebo_plugins package -->
-      <gazebo reference="${prefix}">
+    <gazebo reference="${prefix}">
+      <!-- Enable simulated Velodyne LiDAR -->
+      <xacro:if value="${lidar_active}">
         <sensor type="ray" name="${prefix}-vlp32">
           <always_on>true</always_on>
@@ -86,5 +85,5 @@
             </noise>
           </ray>
-          <plugin name="gazebo_ros_laser_controller" filename="libgazebo_ros_ray_sensor.so">
+          <plugin name="ros_lidar_plugin" filename="libgazebo_ros_ray_sensor.so">
             <ros>
               <remapping>~/out:=/velodyne_points</remapping>
@@ -95,4 +94,7 @@
           </plugin>
         </sensor>
+      </xacro:if>
+      <!-- Enable simulated laser scanner -->
+      <xacro:if value="${scan_active}">
         <sensor type="ray" name="${prefix}-laserscan">
           <always_on>true</always_on>
@@ -126,5 +128,5 @@
             </noise>
           </ray>
-          <plugin name="gazebo_ros_laserscan_controller" filename="libgazebo_ros_ray_sensor.so">
+          <plugin name="ros_laserscan_plugin" filename="libgazebo_ros_ray_sensor.so">
             <ros>
               <remapping>~/out:=/scan</remapping>
@@ -135,6 +137,6 @@
           </plugin>
         </sensor>
-      </gazebo>
-    </xacro:unless>
+      </xacro:if>
+    </gazebo>
   </xacro:macro>
 </robot>

File: eufs_racecar/urdf/ZED2i.urdf.xacro (robot description, xacro)
@@ -52,62 +52,8 @@
       <origin xyz="0 0.06 0" rpy="0 0 0" />
     </joint>
-    <!-- Simulate raw perception sensors only if we're not using the abstracted perception simulation -->
-    <xacro:unless value="${active}">
+    <!-- Enable simulated ZED2i Camera  -->
+    <xacro:if value="${active}">
       <gazebo reference="${prefix}_left_camera_optical_frame">
-        <!-- <sensor type="multicamera" name="stereo_camera">
-          <always_on>true</always_on>
-          <update_rate>60.0</update_rate>
-          <visualize>true</visualize>
-          <camera name="${prefix}_left">
-            <pose>0 0.0 0 0 0 0</pose>
-            <horizontal_fov>1.91986</horizontal_fov>
-            <image>
-              <width>640</width>
-              <height>320</height>
-              <format>B8G8R8</format>
-            </image>
-            <clip>
-              <near>0.5</near>
-              <far>20</far>
-            </clip>
-            <noise>
-              <type>gaussian</type>
-              <mean>0.0</mean>
-              <stddev>0.007</stddev>
-            </noise>
-          </camera>
-          <camera name="${prefix}_right">
-            <pose>0 -0.12 0 0 0 0</pose>
-            <horizontal_fov>1.91986</horizontal_fov>
-            <image>
-              <width>640</width>
-              <height>320</height>
-              <format>B8G8R8</format>
-            </image>
-            <clip>
-              <near>0.5</near>
-              <far>20</far>
-            </clip>
-            <noise>
-              <type>gaussian</type>
-              <mean>0.0</mean>
-              <stddev>0.007</stddev>
-            </noise>
-          </camera>
-          <plugin name="stereo_camera_controller" filename="libgazebo_ros_camera.so">
-            <ros>
-              <parameter name="update_rate" type="double">30.0</parameter>
-              <remapping>/zed/zed_left/camera_info:=/zed2i/zed_node/rgb/camera_info</remapping>
-              <remapping>/zed/zed_left/image_raw:=/zed2i/zed_node/rgb/image_rect_color</remapping>
-              <remapping>/zed/zed_right/camera_info:=/zed2i/zed_node/right/camera_info</remapping>
-              <remapping>/zed/zed_right/image_raw:=/zed2i/zed_node/right/image_rect_color</remapping>
-            </ros>
-            <camera_name>${prefix}</camera_name>
-            <frame_name>${prefix}_left_camera_optical_frame</frame_name>
-            <hack_baseline>0.120</hack_baseline>
-            <triggered>false</triggered>
-          </plugin>
-        </sensor> -->
-        <!-- Depth simulation -->
+        <!-- Depth and Mono cam simulation -->
         <sensor name="stereo_depth" type="depth">
           <always_on>true</always_on>
@@ -128,5 +74,5 @@
             </clip>
           </camera>
-          <plugin name="zed_controller" filename="libgazebo_ros_camera.so">
+          <plugin name="ros_camera_plugin" filename="libgazebo_ros_camera.so">
             <ros>
               <!-- <parameter name="update_rate" type="double">30.0</parameter> -->
@@ -145,5 +91,5 @@
         </sensor>
       </gazebo>
-    </xacro:unless>
+    </xacro:if>
   </xacro:macro>
 </robot>

Commit message: tidied up params names and initialising

File: eufs_plugins/urdf/eufs_plugins.gazebo.xacro (robot description, xacro)
@@ -3,24 +3,24 @@
   <gazebo>
     <plugin name="race_car" filename="libgazebo_ros_race_car.so">
-      <pubGroundTruth>$(arg pub_ground_truth)</pubGroundTruth>
-      <pubTransform>$(arg publish_tf)</pubTransform>
+      <publishGroundTruth>$(arg publish_ground_truth)</publishGroundTruth>
+      <publishTransform>$(arg publish_transform)</publishTransform>
       <commandMode>$(arg command_mode)</commandMode>
-      <yamlConfig>$(arg config_file)</yamlConfig>
+      <vehicleConfig>$(arg vehicle_config)</vehicleConfig>
       <noiseConfig>$(arg noise_config)</noiseConfig>
       <vehicleModel>$(arg vehicle_model)</vehicleModel>
-      <simulateSLAM>$(arg sim_slam)</simulateSLAM>
+      <simulateSLAM>$(arg simulate_slam)</simulateSLAM>
     </plugin>
   </gazebo>
   <gazebo>
     <plugin name="cone_detection" filename="libgazebo_ros_cone_detection.so">
-      <publishGroundTruth>$(arg pub_ground_truth)</publishGroundTruth>
-      <simulatePerception>$(arg sim_perception)</simulatePerception>
-      <simulateSLAM>$(arg sim_slam)</simulateSLAM>
+      <publishGroundTruth>$(arg publish_ground_truth)</publishGroundTruth>
+      <simulatePerception>$(arg simulate_perception)</simulatePerception>
+      <simulateSLAM>$(arg simulate_slam)</simulateSLAM>
     </plugin>
   </gazebo>
   <gazebo>
     <plugin name="sbg_driver" filename="libgazebo_ros_sbg_driver.so">
-      <noise_config>$(arg noise_config)</noise_config>
-      <pubGroundTruth>$(arg pub_ground_truth)</pubGroundTruth>
+      <noiseConfig>$(arg noise_config)</noiseConfig>
+      <publishGroundTruth>$(arg publish_ground_truth)</publishGroundTruth>
     </plugin>
   </gazebo>

File: eufs_racecar/racecars/qev3/robot.urdf.xacro (robot description, xacro)
@@ -5,5 +5,5 @@
     <!-- ***************** -->
     <!--  Load the config file  -->
-    <xacro:property name="config" value="${load_yaml('$(arg config_file)')}"/>
+    <xacro:property name="config" value="${load_yaml('$(arg vehicle_config)')}"/>
     <!-- Simulate sensors or not? -->
     <xacro:arg name="enable_camera" default="false"/>
